File: KiCAD files/FLASH2/FLASH2.sch (KiCad schematic (older format))
At the start: 15 parts, among them J1 card addr, J2 Power Bus, J3 Signal Bus, J4 IDE connector, U1 74LS04, U2 74LS85, U3 74LS245, U4 74LS245

Commit message: Update FLASH2.sch
Parts:
- added C3, C4: 10nF, symbol Device:C
Connections:
- net +5V: now also C3.1, C4.1
- net GND: now also C3.2, C4.2
Other:
- moved on the sheet: C1, C2, J1, J2, J3, J4, R1, R2, R3, R4, R6, U1A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

Commit message: Update FLASH2.sch
Connections:
- net +5V: no longer J4.20 (Pin_20), J4.42 (Pin_42)
- net GND: no longer J4.19 (Pin_19), J4.22 (Pin_22), J4.24 (Pin_24), J4.26 (Pin_26), J4.30 (Pin_30), J4.40 (Pin_40), J4.43 (Pin_43), J4.44 (Pin_44)
- net fd07: now reaches J4.3 (Pin_3), U4.11 (B7)
- net fd06: now reaches J4.5 (Pin_5), U4.12 (B6)
- no-connect marks 45 -> 55
Other:
- moved on the sheet: C2
Changed lines of the file:
@@
 EESchema Schematic File Version 4
+LIBS:FLASH2-cache
 EELAYER 30 0
 EELAYER END
@@
 L power:GND #PWR017
 U 1 1 5EDFD85C
-P 10200 5200
-F 0 "#PWR017" H 10200 4950 50  0001 C CNN
-F 1 "GND" H 10205 5027 50  0000 C CNN
-F 2 "" H 10200 5200 50  0001 C CNN
-F 3 "" H 10200 5200 50  0001 C CNN
-	1    10200 5200
-	1    0    0    -1
-$EndComp
-Wire Wire Line
-	9950 4550 10200 4550
+P 10200 2750
+F 0 "#PWR017" H 10200 2500 50  0001 C CNN
+F 1 "GND" H 10205 2577 50  0000 C CNN
+F 2 "" H 10200 2750 50  0001 C CNN
+F 3 "" H 10200 2750 50  0001 C CNN
+	1    10200 2750
+	1    0    0    -1
+$EndComp
 NoConn ~ 9950 3950
 NoConn ~ 9950 4150
 NoConn ~ 9950 4250
-Wire Wire Line
-	9950 4050 10200 4050
-Wire Wire Line
-	10200 4050 10200 4550
-Wire Wire Line
-	9950 3650 10200 3650
-Wire Wire Line
-	10200 3650 10200 3750
-Connection ~ 10200 4050
-Wire Wire Line
-	9950 3750 10200 3750
-Connection ~ 10200 3750
-Wire Wire Line
-	10200 3750 10200 3850
-Wire Wire Line
-	9950 3850 10200 3850
-Connection ~ 10200 3850
-Wire Wire Line
-	10200 3850 10200 4050
 Text Label 9950 4350 0    50   ~ 0
 fa02
@@
 L Device:C C2
 U 1 1 5F59C5F0
-P 10600 3700
-F 0 "C2" H 10400 3750 50  0000 C CNN
-F 1 "10nF" H 10400 3650 50  0000 C CNN
-F 2 "" H 10638 3550 50  0001 C CNN
-F 3 "~" H 10600 3700 50  0001 C CNN
-	1    10600 3700
+P 9300 4950
+F 0 "C2" H 9100 5000 50  0000 C CNN
+F 1 "10nF" H 9100 4900 50  0000 C CNN
+F 2 "" H 9338 4800 50  0001 C CNN
+F 3 "~" H 9300 4950 50  0001 C CNN
+	1    9300 4950
 	1    0    0    -1
 $EndComp
@@
 	1    9650 3650
 	1    0    0    -1
-$EndComp
-Wire Wire Line
-	9950 4750 10200 4750
-Wire Wire Line
-	10200 4750 10200 4550
-Connection ~ 10200 4550
-$Comp
-L power:+5V #PWR016
-U 1 1 5F5CC642
-P 9950 4650
-F 0 "#PWR016" H 9950 4500 50  0001 C CNN
-F 1 "+5V" V 9965 4778 50  0000 L CNN
-F 2 "" H 9950 4650 50  0001 C CNN
-F 3 "" H 9950 4650 50  0001 C CNN
-	1    9950 4650
-	0    1    1    0
 $EndComp
 $Comp
@@
 	0    1    1    0
 $EndComp
-$Comp
-L power:+5V #PWR013
-U 1 1 5F5E3373
-P 10600 3400
-F 0 "#PWR013" H 10600 3250 50  0001 C CNN
-F 1 "+5V" H 10615 3528 50  0000 L CNN
-F 2 "" H 10600 3400 50  0001 C CNN
-F 3 "" H 10600 3400 50  0001 C CNN
-	1    10600 3400
-	1    0    0    -1
-$EndComp
-Connection ~ 10200 4750
 Text Label 9450 3850 2    50   ~ 0
 frd
@@
 	3950 5600 3650 5600
 Wire Wire Line
-	9950 3550 10600 3550
-Wire Wire Line
-	10600 3400 10600 3550
-Connection ~ 10600 3550
+	9300 4650 9300 4800
 $Comp
 L power:GND #PWR014
 U 1 1 5F6B4BAE
-P 10600 3850
-F 0 "#PWR014" H 10600 3600 50  0001 C CNN
-F 1 "GND" H 10605 3677 50  0000 C CNN
-F 2 "" H 10600 3850 50  0001 C CNN
-F 3 "" H 10600 3850 50  0001 C CNN
-	1    10600 3850
+P 9300 5100
+F 0 "#PWR014" H 9300 4850 50  0001 C CNN
+F 1 "GND" H 9305 4927 50  0000 C CNN
+F 2 "" H 9300 5100 50  0001 C CNN
+F 3 "" H 9300 5100 50  0001 C CNN
+	1    9300 5100
 	1    0    0    -1
 $EndComp
@@
 L power:+5V #PWR011
 U 1 1 5F6B634B
-P 9450 4650
-F 0 "#PWR011" H 9450 4500 50  0001 C CNN
-F 1 "+5V" V 9465 4778 50  0000 L CNN
-F 2 "" H 9450 4650 50  0001 C CNN
-F 3 "" H 9450 4650 50  0001 C CNN
-	1    9450 4650
+P 9150 4650
+F 0 "#PWR011" H 9150 4500 50  0001 C CNN
+F 1 "+5V" V 9165 4778 50  0000 L CNN
+F 2 "" H 9150 4650 50  0001 C CNN
+F 3 "" H 9150 4650 50  0001 C CNN
+	1    9150 4650
 	0    -1   -1   0
 $EndComp
 Wire Wire Line
-	10200 3650 10200 2650
-Wire Wire Line
 	10200 2650 9950 2650
-Connection ~ 10200 3650
 $Comp
 L 74xx:74LS245 U3
@@
 Connection ~ 5550 4850
 $Comp
-L power:GND #PWR024
-U 1 1 5FF07438
-P 9450 4750
-F 0 "#PWR024" H 9450 4500 50  0001 C CNN
-F 1 "GND" V 9455 4577 50  0000 C CNN
-F 2 "" H 9450 4750 50  0001 C CNN
-F 3 "" H 9450 4750 50  0001 C CNN
-	1    9450 4750
-	0    1    1    0
-$EndComp
-$Comp
-L power:GND #PWR023
-U 1 1 5FF0DA3B
-P 9450 3550
-F 0 "#PWR023" H 9450 3300 50  0001 C CNN
-F 1 "GND" V 9455 3377 50  0000 C CNN
-F 2 "" H 9450 3550 50  0001 C CNN
-F 3 "" H 9450 3550 50  0001 C CNN
-	1    9450 3550
-	0    1    1    0
-$EndComp
-Wire Wire Line
-	10200 4750 10200 5200
-$Comp
 L Device:C C3
 U 1 1 5FE1CE6E
@@
 	8550 5600 5550 5600
 Connection ~ 5550 5600
+Wire Wire Line
+	10200 2650 10200 2750
+NoConn ~ 9950 3550
+NoConn ~ 9950 3650
+NoConn ~ 9950 3750
+NoConn ~ 9950 3850
+NoConn ~ 9950 4050
+NoConn ~ 9950 4550
+NoConn ~ 9950 4650
+NoConn ~ 9950 4750
+NoConn ~ 9450 4750
+NoConn ~ 9450 3550
+Wire Wire Line
+	9150 4650 9300 4650
+Wire Wire Line
+	9450 4650 9300 4650
+Connection ~ 9300 4650
+Text Label 9450 2850 2    50   ~ 0
+fd06
+Text Label 9450 2750 2    50   ~ 0
+fd07
 $EndSCHEMATC
