File: KiCAD files/USARTv2/USARTv2.sch (KiCad schematic (older format))
At the start: 26 parts, among them J1 Card addr, J2 Power Bus, J3 Signal Buss, J4 RS232, Q1 BC328, Q2 BC328, U1 74LS00, U2 74LS85, U5 MAX232

Commit message: home
Parts:
- removed D1, D2: LED, symbol Device:LED
- removed J1: Card addr, symbol Connector_Generic:Conn_02x04_Odd_Even
- removed Q1, Q2: BC328, Package_TO_SOT_THT:TO-92_Inline, symbol Transistor_BJT:BC328
- removed R1, R2, R3, R4: 10k, symbol Device:R
- removed R5, R7: 180, symbol Device:R
- removed R6, R9: 3k3, symbol Device:R
- removed U1: 74LS00, symbol 74xx:74LS00
- removed U2: 74LS85, symbol 74xx:74LS85
- added C?: 22nF, symbol Device:C
- added D?: TX 0, symbol Device:LED
- added D?: RX 0, symbol Device:LED
- added D?: TX 1, symbol Device:LED
- added D?: RX 1, symbol Device:LED
- added J?: RS232, symbol Connector:DB9_Male
- added R? (x4): 270, symbol Device:R
- added U? (x7): SN74LS07, symbol 74xx:SN74LS07
- added U?: ATmega328P-PU, Package_DIP:DIP-28_W7.62mm, symbol MCU_Microchip_ATmega:ATmega328P-PU
Connections:
- net labels added: +5C
- net labels removed: CS0, CS1
- no-connect marks 42 -> 33
Other:
- note removed: "(For future expansion)"
- note removed: "RX"
- note removed: "TX"
- note removed: "lsb"
- note removed: "msb"
- moved on the sheet: A1, C2, C3, C4, C5, C6, C9, J2, J3, J4, U5
