File: KiCAD files/USARTv2/USARTv2.sch (KiCad schematic (older format))
At the start: 25 parts, among them J1 Card addr, J2 Power Bus, J3 Signal Buss, J4 RS232, Q1 BC328, Q2 BC328, U2 74LS85, U5 MAX232

Commit message: office
Parts:
- added U1: 74LS00, symbol 74xx:74LS00
Connections:
- net +5V: now also U1.14 (VCC); no longer U2.3 (Ia=b)
- net GND: now also U1.7 (GND)
- net a00: now also U1.12, U1.13, U1.9; no longer A1.13 (D10)
- net a01: now also A1.13 (D10); no longer A1.14 (D11)
- net iorq: now also U1.1, U1.2; no longer A1.19 (A0)
- net rd: now also A1.14 (D11); no longer A1.15 (D12)
- net wr: now also A1.15 (D12); no longer A1.16 (D13)
- net CS: no longer names the net of U2.6 (Oa=b)
- net CS: now also U1.10, U1.5; no longer A1.20 (A1)
- new net: U1.3, U2.3 (Ia=b)
- new net: U1.11, U1.4
- new net CS0: A1.16 (D13), U1.6
- new net CS1: U1.8
- no-connect marks 39 -> 42
Other:
- note added: "(For future expansion)"
- moved on the sheet: A1, C2, C3, C4, C5, C6, D1, D2, J4, Q1, Q2, R5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

Commit message: home
Parts:
- A1: symbol MCU_Module:Arduino_Nano_v3.x -> USARTv2-rescue:Arduino_Nano_v3.x-MCU_Module
Changed lines of the file:
@@
 EESchema Schematic File Version 4
+LIBS:USARTv2-cache
 EELAYER 30 0
 EELAYER END
@@
 Connection ~ 2250 2650
 $Comp
-L MCU_Module:Arduino_Nano_v3.x A1
+L USARTv2-rescue:Arduino_Nano_v3.x-MCU_Module A1
 U 1 1 60CCDAA2
 P 6450 4750

Commit message: office
Parts:
- removed D1, D2: LED, symbol Device:LED
- removed J1: Card addr, symbol Connector_Generic:Conn_02x04_Odd_Even
- removed Q1, Q2: BC328, Package_TO_SOT_THT:TO-92_Inline, symbol Transistor_BJT:BC328
- removed R1, R2, R3, R4: 10k, symbol Device:R
- removed R5, R7: 180, symbol Device:R
- removed R6, R9: 3k3, symbol Device:R
- removed U1: 74LS00, symbol 74xx:74LS00
- removed U2: 74LS85, symbol 74xx:74LS85
- added D? (x2): RX, symbol Device:LED
- added D? (x2): TX, symbol Device:LED
- added J?: RS232, symbol Connector:DB9_Male
- added R? (x4): 180, symbol Device:R
- added U? (x5): SN74LS07, symbol 74xx:SN74LS07
- added U?: ATmega328P-PU, Package_DIP:DIP-28_W7.62mm, symbol MCU_Microchip_ATmega:ATmega328P-PU
Connections:
- net +5V: now also D?.2 (A), D?.2 (A), D?.2 (A), D?.2 (A)
- net GND: now also J?.5
- net at U5.7 (T2OUT): now also J?.3
- net at U5.8 (R2IN): now also J?.2
- new net: R?.1, U?.2
- new net: R?.1, U?.4
- new net: R?.1, U?.6
- new net: R?.1, U?.8
- new net: D?.1 (K), R?.2 (x4)
- new net: J?.1, J?.4, J?.6
- new net: J?.7, J?.8
- new net: U?.22 (GND), U?.8 (GND)
- no-connect marks 42 -> 38
Other:
- note added: "TTY0"
- note added: "TTY1"
- note removed: "(For future expansion)"
- note removed: "RX"
- note removed: "TX"
- note removed: "lsb"
- note removed: "msb"
