File: KiCAD files/CPU/CPU.kicad_pcb (KiCad board)
At the start: 2 copper layers, 99.7 x 69.8 mm, 29 parts, among them J1 Signal Bus, J2 Power Bus, J3 INT, J4 EXT RESET/INT, J5 Reset, J6 clock rate, Q1 BC328, U1 74LS00, U2 74LS74, U3 Z80CPU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

Commit message: office
Other:
- board text added: "HALT"
- board text added: "INT"
- board text added: "Power on"
- board text added: "RESET"

Commit message: office
Parts:
- J6: value clock rate -> clock selector
- U3: footprint Package_DIP:DIP-40_W15.24mm_Socket_LongPads -> Package_DIP:DIP-40_W25.4mm_Socket_LongPads
- moved J6 15.7 mm to (173.7, 98.6), turned to 0 degrees
- moved C5 1.27 mm to (120.0, 76.2)
- moved C6 1.05 mm to (131.1, 81.5)
Connections:
- J6 pad 2: Net-(J6-Pad2) -> /clk
- J6 pad 5: /clk -> Net-(J6-Pad5)
- U2 pad 11: Net-(J6-Pad2) -> Net-(J6-Pad3)
- U2 pad 5: Net-(J6-Pad2) -> Net-(J6-Pad3)
- U2 pad 9: Net-(J6-Pad3) -> Net-(J6-Pad5)
Routing:
- net +5V: track 251.9 -> 0.00 mm, vias 1 -> 0
- net GND: track 244.7 -> 0.00 mm
- net /reset: track 150.3 -> 0.00 mm
- net /halt: track 118.8 -> 0.00 mm
- net /int: track 103.3 -> 0.00 mm
- net /clk: track 96.1 -> 0.00 mm, vias 1 -> 0
- net /d01: track 86.4 -> 0.00 mm
- net /iorq: track 82.4 -> 0.00 mm
- net /rd: track 71.1 -> 0.00 mm
- net /nmi: track 65.8 -> 0.00 mm
- net /wr: track 65.8 -> 0.00 mm
- net /d05: track 64.9 -> 0.00 mm
- net /busack: track 63.7 -> 0.00 mm
- net /mreq: track 63.4 -> 0.00 mm, vias 1 -> 0
- net /wait: track 62.6 -> 0.00 mm
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- removed copper zone on B.Cu, net GND
Other:
- board text added: "Clock"
- board text added: "f"
- board text added: "f/2"
- board text added: "f/4"

Commit message: office
Parts:
- U3: footprint Package_DIP:DIP-40_W25.4mm_Socket_LongPads -> Package_DIP:DIP-40_W15.24mm_Socket_LongPads
- moved J4 2.54 mm to (188.0, 117.5)
Routing:
- net GND: track 0.00 -> 243.4 mm
- net +5V: track 0.00 -> 233.0 mm
- net /reset: track 0.00 -> 176.9 mm
- net /halt: track 0.00 -> 128.2 mm
- net /int: track 0.00 -> 107.0 mm
- net /clk: track 0.00 -> 103.6 mm
- net /d00: track 0.00 -> 87.0 mm
- net /mreq: track 0.00 -> 86.0 mm
- net /iorq: track 0.00 -> 78.8 mm
- net /d01: track 0.00 -> 74.8 mm
- net /rd: track 0.00 -> 73.6 mm
- net /nmi: track 0.00 -> 67.7 mm
- net /d05: track 0.00 -> 66.0 mm
- net /wr: track 0.00 -> 66.0 mm
- net /busack: track 0.00 -> 63.7 mm
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- added copper zone on B.Cu, net GND
