File: KiCAD files/CPU/CPU.kicad_pcb (KiCad board)
At the start: 2 copper layers, 99.7 x 69.8 mm, 29 parts, among them J1 Signal Bus, J2 Power Bus, J3 INT, J4 EXT RESET/INT, J5 Reset, J6 clock selector, Q1 BC328, U1 74LS00, U2 74LS74, U3 Z80CPU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

Commit message: home
Other:
- board text added: "Grid 25.00mils"
Changed lines of the file:
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@@
   (general
     (thickness 1.6)
-    (drawings 13)
+    (drawings 26)
     (tracks 600)
     (zones 0)
@@
     )
   )
+  (gr_text "Grid 25.00mils" (at 147.955 135.255) (layer F.SilkS)
+    (effects (font (size 1 1) (thickness 0.15)))
+  )
+  (dimension 5.08 (width 0.12) (layer F.SilkS)
+    (gr_text "0.2000 in" (at 192.405 139.7) (layer F.SilkS)
+      (effects (font (size 1 1) (thickness 0.15)))
+    )
+    (feature1 (pts (xy 194.945 127.635) (xy 194.945 139.016421)))
+    (feature2 (pts (xy 189.865 127.635) (xy 189.865 139.016421)))
+    (crossbar (pts (xy 189.865 138.43) (xy 194.945 138.43)))
+    (arrow1a (pts (xy 194.945 138.43) (xy 193.818496 139.016421)))
+    (arrow1b (pts (xy 194.945 138.43) (xy 193.818496 137.843579)))
+    (arrow2a (pts (xy 189.865 138.43) (xy 190.991504 139.016421)))
+    (arrow2b (pts (xy 189.865 138.43) (xy 190.991504 137.843579)))
+  )
+  (dimension 3.048 (width 0.12) (layer F.SilkS)
+    (gr_text "0.1200 in" (at 192.405 137.287) (layer F.SilkS)
+      (effects (font (size 1 1) (thickness 0.15)))
+    )
+    (feature1 (pts (xy 193.929 127.635) (xy 193.929 136.603421)))
+    (feature2 (pts (xy 190.881 127.635) (xy 190.881 136.603421)))
+    (crossbar (pts (xy 190.881 136.017) (xy 193.929 136.017)))
+    (arrow1a (pts (xy 193.929 136.017) (xy 192.802496 136.603421)))
+    (arrow1b (pts (xy 193.929 136.017) (xy 192.802496 135.430579)))
+    (arrow2a (pts (xy 190.881 136.017) (xy 192.007504 136.603421)))
+    (arrow2b (pts (xy 190.881 136.017) (xy 192.007504 135.430579)))
+  )
+  (dimension 5.08 (width 0.12) (layer F.SilkS)
+    (gr_text "0.2000 in" (at 199.39 130.175 90) (layer F.SilkS)
+      (effects (font (size 1 1) (thickness 0.15)))
+    )
+    (feature1 (pts (xy 192.405 127.635) (xy 198.706421 127.635)))
+    (feature2 (pts (xy 192.405 132.715) (xy 198.706421 132.715)))
+    (crossbar (pts (xy 198.12 132.715) (xy 198.12 127.635)))
+    (arrow1a (pts (xy 198.12 127.635) (xy 198.706421 128.761504)))
+    (arrow1b (pts (xy 198.12 127.635) (xy 197.533579 128.761504)))
+    (arrow2a (pts (xy 198.12 132.715) (xy 198.706421 131.588496)))
+    (arrow2b (pts (xy 198.12 132.715) (xy 197.533579 131.588496)))
+  )
+  (dimension 5.08 (width 0.12) (layer F.SilkS)
+    (gr_text "0.2000 in" (at 194.945 134.62) (layer F.SilkS)
+      (effects (font (size 1 1) (thickness 0.15)))
+    )
+    (feature1 (pts (xy 197.485 127.635) (xy 197.485 133.936421)))
+    (feature2 (pts (xy 192.405 127.635) (xy 192.405 133.936421)))
+    (crossbar (pts (xy 192.405 133.35) (xy 197.485 133.35)))
+    (arrow1a (pts (xy 197.485 133.35) (xy 196.358496 133.936421)))
+    (arrow1b (pts (xy 197.485 133.35) (xy 196.358496 132.763579)))
+    (arrow2a (pts (xy 192.405 133.35) (xy 193.531504 133.936421)))
+    (arrow2b (pts (xy 192.405 133.35) (xy 193.531504 132.763579)))
+  )
+  (dimension 5.08 (width 0.12) (layer F.SilkS)
+    (gr_text "0.2000 in" (at 199.39 65.405 90) (layer F.SilkS)
+      (effects (font (size 1 1) (thickness 0.15)))
+    )
+    (feature1 (pts (xy 192.405 62.865) (xy 198.706421 62.865)))
+    (feature2 (pts (xy 192.405 67.945) (xy 198.706421 67.945)))
+    (crossbar (pts (xy 198.12 67.945) (xy 198.12 62.865)))
+    (arrow1a (pts (xy 198.12 62.865) (xy 198.706421 63.991504)))
+    (arrow1b (pts (xy 198.12 62.865) (xy 197.533579 63.991504)))
+    (arrow2a (pts (xy 198.12 67.945) (xy 198.706421 66.818496)))
+    (arrow2b (pts (xy 198.12 67.945) (xy 197.533579 66.818496)))
+  )
+  (dimension 5.08 (width 0.12) (layer F.SilkS)
+    (gr_text "0.2000 in" (at 194.945 60.96) (layer F.SilkS)
+      (effects (font (size 1 1) (thickness 0.15)))
+    )
+    (feature1 (pts (xy 192.405 67.945) (xy 192.405 61.643579)))
+    (feature2 (pts (xy 197.485 67.945) (xy 197.485 61.643579)))
+    (crossbar (pts (xy 197.485 62.23) (xy 192.405 62.23)))
+    (arrow1a (pts (xy 192.405 62.23) (xy 193.531504 61.643579)))
+    (arrow1b (pts (xy 192.405 62.23) (xy 193.531504 62.816421)))
+    (arrow2a (pts (xy 197.485 62.23) (xy 196.358496 61.643579)))
+    (arrow2b (pts (xy 197.485 62.23) (xy 196.358496 62.816421)))
+  )
+  (dimension 99.695 (width 0.12) (layer F.SilkS)
+    (gr_text "3.9250 in" (at 147.6375 57.785) (layer F.SilkS)
+      (effects (font (size 1 1) (thickness 0.15)))
+    )
+    (feature1 (pts (xy 97.79 62.865) (xy 97.79 58.468579)))
+    (feature2 (pts (xy 197.485 62.865) (xy 197.485 58.468579)))
+    (crossbar (pts (xy 197.485 59.055) (xy 97.79 59.055)))
+    (arrow1a (pts (xy 97.79 59.055) (xy 98.916504 58.468579)))
+    (arrow1b (pts (xy 97.79 59.055) (xy 98.916504 59.641421)))
+    (arrow2a (pts (xy 197.485 59.055) (xy 196.358496 58.468579)))
+    (arrow2b (pts (xy 197.485 59.055) (xy 196.358496 59.641421)))
+  )
+  (dimension 69.85 (width 0.12) (layer F.SilkS)
+    (gr_text "2.7500 in" (at 92.71 97.79 90) (layer F.SilkS)
+      (effects (font (size 1 1) (thickness 0.15)))
+    )
+    (feature1 (pts (xy 97.79 62.865) (xy 93.393579 62.865)))
+    (feature2 (pts (xy 97.79 132.715) (xy 93.393579 132.715)))
+    (crossbar (pts (xy 93.98 132.715) (xy 93.98 62.865)))
+    (arrow1a (pts (xy 93.98 62.865) (xy 94.566421 63.991504)))
+    (arrow1b (pts (xy 93.98 62.865) (xy 93.393579 63.991504)))
+    (arrow2a (pts (xy 93.98 132.715) (xy 94.566421 131.588496)))
+    (arrow2b (pts (xy 93.98 132.715) (xy 93.393579 131.588496)))
+  )
+  (dimension 3.175 (width 0.12) (layer F.SilkS)
+    (gr_text "0.1250 in" (at 95.885 131.1275 90) (layer F.SilkS)
+      (effects (font (size 1 1) (thickness 0.15)))
+    )
+    (feature1 (pts (xy 102.235 129.54) (xy 96.568579 129.54)))
+    (feature2 (pts (xy 102.235 132.715) (xy 96.568579 132.715)))
+    (crossbar (pts (xy 97.155 132.715) (xy 97.155 129.54)))
+    (arrow1a (pts (xy 97.155 129.54) (xy 97.741421 130.666504)))
+    (arrow1b (pts (xy 97.155 129.54) (xy 96.568579 130.666504)))
+    (arrow2a (pts (xy 97.155 132.715) (xy 97.741421 131.588496)))
+    (arrow2b (pts (xy 97.155 132.715) (xy 96.568579 131.588496)))
+  )
+  (dimension 4.445 (width 0.12) (layer F.SilkS)
+    (gr_text "0.1750 in" (at 100.0125 134.62) (layer F.SilkS)
+      (effects (font (size 1 1) (thickness 0.15)))
+    )
+    (feature1 (pts (xy 97.79 129.54) (xy 97.79 133.936421)))
+    (feature2 (pts (xy 102.235 129.54) (xy 102.235 133.936421)))
+    (crossbar (pts (xy 102.235 133.35) (xy 97.79 133.35)))
+    (arrow1a (pts (xy 97.79 133.35) (xy 98.916504 132.763579)))
+    (arrow1b (pts (xy 97.79 133.35) (xy 98.916504 133.936421)))
+    (arrow2a (pts (xy 102.235 133.35) (xy 101.108496 132.763579)))
+    (arrow2b (pts (xy 102.235 133.35) (xy 101.108496 133.936421)))
+  )
+  (dimension 3.175 (width 0.12) (layer F.SilkS)
+    (gr_text "0.1250 in" (at 95.885 64.4525 90) (layer F.SilkS)
+      (effects (font (size 1 1) (thickness 0.15)))
+    )
+    (feature1 (pts (xy 102.235 62.865) (xy 96.568579 62.865)))
+    (feature2 (pts (xy 102.235 66.04) (xy 96.568579 66.04)))
+    (crossbar (pts (xy 97.155 66.04) (xy 97.155 62.865)))
+    (arrow1a (pts (xy 97.155 62.865) (xy 97.741421 63.991504)))
+    (arrow1b (pts (xy 97.155 62.865) (xy 96.568579 63.991504)))
+    (arrow2a (pts (xy 97.155 66.04) (xy 97.741421 64.913496)))
+    (arrow2b (pts (xy 97.155 66.04) (xy 96.568579 64.913496)))
+  )
+  (dimension 4.445 (width 0.12) (layer F.SilkS)
+    (gr_text "0.1750 in" (at 100.0125 60.96) (layer F.SilkS)
+      (effects (font (size 1 1) (thickness 0.15)))
+    )
+    (feature1 (pts (xy 97.79 66.04) (xy 97.79 61.643579)))
+    (feature2 (pts (xy 102.235 66.04) (xy 102.235 61.643579)))
+    (crossbar (pts (xy 102.235 62.23) (xy 97.79 62.23)))
+    (arrow1a (pts (xy 97.79 62.23) (xy 98.916504 61.643579)))
+    (arrow1b (pts (xy 97.79 62.23) (xy 98.916504 62.816421)))
+    (arrow2a (pts (xy 102.235 62.23) (xy 101.108496 61.643579)))
+    (arrow2b (pts (xy 102.235 62.23) (xy 101.108496 62.816421)))
+  )
   (gr_text f/4 (at 179.832 103.632) (layer F.SilkS)
