File: KiCAD files/CPU/CPU.sch (KiCad schematic (older format))
At the start: 26 parts, among them J1 Power Bus, J2 Signal Bus, J3 reset button, J4 clock rate, Q1 BC328, U1 74LS00, U3 Z80CPU, U4 74LS74, Y1 4MHz

Commit message: office
Parts:
- added D3: LED, symbol Device:LED
- added R11: 270, symbol Device:R
Connections:
- wire segments 98 -> 99
Other:
- note added: "Power On"
Changed lines of the file:
@@
 EESchema Schematic File Version 4
-LIBS:CPU-cache
 EELAYER 30 0
 EELAYER END
@@
 	1    0    0    -1
 $EndComp
+$Comp
+L Device:LED D3
+U 1 1 60CBC165
+P 3800 1300
+F 0 "D3" V 3850 1450 50  0000 C CNN
+F 1 "LED" V 3750 1450 50  0000 C CNN
+F 2 "" H 3800 1300 50  0001 C CNN
+F 3 "~" H 3800 1300 50  0001 C CNN
+	1    3800 1300
+	0    -1   -1   0
+$EndComp
+Text Notes 3950 1350 0    50   ~ 0
+Power On
+$Comp
+L power:GND #PWR020
+U 1 1 60CBEDD9
+P 3800 1550
+F 0 "#PWR020" H 3800 1300 50  0001 C CNN
+F 1 "GND" H 3805 1377 50  0000 C CNN
+F 2 "" H 3800 1550 50  0001 C CNN
+F 3 "" H 3800 1550 50  0001 C CNN
+	1    3800 1550
+	1    0    0    -1
+$EndComp
+Wire Wire Line
+	3800 1550 3800 1450
+$Comp
+L Device:R R11
+U 1 1 60CC4F5F
+P 3800 1000
+F 0 "R11" H 3870 1046 50  0000 L CNN
+F 1 "270" H 3870 955 50  0000 L CNN
+F 2 "" V 3730 1000 50  0001 C CNN
+F 3 "~" H 3800 1000 50  0001 C CNN
+	1    3800 1000
+	1    0    0    -1
+$EndComp
+$Comp
+L power:+5V #PWR019
+U 1 1 60CC8077
+P 3800 850
+F 0 "#PWR019" H 3800 700 50  0001 C CNN
+F 1 "+5V" H 3815 1023 50  0000 C CNN
+F 2 "" H 3800 850 50  0001 C CNN
+F 3 "" H 3800 850 50  0001 C CNN
+	1    3800 850
+	1    0    0    -1
+$EndComp

Commit message: office
Parts:
- removed J3: reset button, symbol Connector_Generic:Conn_01x02
- added J3: External reset/int, symbol Connector:Conn_01x04_Male
- added J5: RST 7, symbol Connector_Generic:Conn_02x01
- added J6: Reset, symbol Connector_Generic:Conn_02x01
Connections:
- wire segments 99 -> 105
Other:
- moved on the sheet: D2, Q1, R10, R9, U1E, U4C

Commit message: office
Other:
- note added: "Connects to a\npushbutton on\nthe front panel"
Changed lines of the file:
@@
 Wire Wire Line
 	4450 5550 4450 5700
+Text Notes 4400 5400 0    50   ~ 0
+Connects to a\npushbutton on\nthe front panel
+Text Notes 4800 1050 0    50   ~ 0
+Connects to a\npushbutton on\nthe front panel
 $EndSCHEMATC

Commit message: home
Parts:
- removed C4: 10n, symbol Device:C
- removed R5, R6, R7, R8: 8k2, symbol Device:R
- added C? (x3): 10n, symbol Device:C
- added RN?: 4x10k, Resistor_THT:R_Array_SIP5, symbol Device:R_Network04
Connections:
- net +5V: now also C?.1, C?.1, C?.1, RN?.1 (common)
- net GND: now also C?.2, C?.2, C?.2
- net busrq: now also RN?.2 (R1)
- net int: now also RN?.5 (R4)
- net nmi: now also RN?.4 (R3)
- net wait: now also RN?.3 (R2)
Other:
- moved on the sheet: C1, C2, C3, C5, D1, D2, D3, J1, J2, J3, J4, J5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

Commit message: home
Parts:
- removed J3: External reset/int, symbol Connector:Conn_01x04_Male
- added J4: EXT RESET/INT, Connector_PinHeader_2.54mm:PinHeader_2x02_P2.54mm_Vertical, symbol Connector_Generic:Conn_02x02_Odd_Even
- C1, C2, C3: renamed from C?; footprint (none) -> Capacitor_THT:C_Disc_D3.8mm_W2.6mm_P2.50mm
- C4: renamed from C5; footprint (none) -> Capacitor_THT:CP_Radial_D5.0mm_P2.50mm
- C5: renamed from C1; footprint (none) -> Capacitor_THT:C_Disc_D3.8mm_W2.6mm_P2.50mm
- C6: renamed from C2; footprint (none) -> Capacitor_THT:C_Disc_D3.8mm_W2.6mm_P2.50mm
- C7: renamed from C3; footprint (none) -> Capacitor_THT:CP_Radial_D5.0mm_P2.50mm
- D1: renamed from D3; footprint (none) -> LED_THT:LED_D3.0mm
- D3: renamed from D2; footprint (none) -> LED_THT:LED_D3.0mm
- J1: renamed from J2; footprint (none) -> Connector_PinHeader_2.54mm:PinHeader_2x20_P2.54mm_Vertical
- J2: renamed from J1; footprint (none) -> Connector_PinHeader_2.54mm:PinHeader_2x05_P2.54mm_Vertical
- J3: renamed from J5; value RST 7 -> INT; footprint (none) -> Connector_PinHeader_2.54mm:PinHeader_2x01_P2.54mm_Vertical
- J5: renamed from J6; footprint (none) -> Connector_PinHeader_2.54mm:PinHeader_2x01_P2.54mm_Vertical
- J6: renamed from J4; footprint (none) -> Connector_PinHeader_2.54mm:PinHeader_2x03_P2.54mm_Vertical
- R1, R2: footprint (none) -> Resistor_THT:R_Axial_DIN0207_L6.3mm_D2.5mm_P10.16mm_Horizontal
- R3: renamed from R11; footprint (none) -> Resistor_THT:R_Axial_DIN0207_L6.3mm_D2.5mm_P10.16mm_Horizontal
- R4: renamed from R3; footprint (none) -> Resistor_THT:R_Axial_DIN0207_L6.3mm_D2.5mm_P10.16mm_Horizontal
- R5: renamed from R4; footprint (none) -> Resistor_THT:R_Axial_DIN0207_L6.3mm_D2.5mm_P10.16mm_Horizontal
- R6: renamed from R9; value 3.3k -> 270; footprint (none) -> Resistor_THT:R_Axial_DIN0207_L6.3mm_D2.5mm_P10.16mm_Horizontal
- R7: renamed from R10; value 180 -> 3.3k; footprint (none) -> Resistor_THT:R_Axial_DIN0207_L6.3mm_D2.5mm_P10.16mm_Horizontal
- U1: footprint (none) -> Package_DIP:DIP-14_W7.62mm_Socket_LongPads
- U2: renamed from U4; footprint (none) -> Package_DIP:DIP-14_W7.62mm_Socket_LongPads
- U3: footprint (none) -> Package_DIP:DIP-40_W25.4mm_Socket_LongPads
- Y1: footprint (none) -> Crystal:Crystal_HC49-U_Vertical
- gave numbers to parts that had none: 1
- renumbered D1 to D2
Connections:
- net +5V: now also J5.1 (Pin_1), J4.1 (Pin_1)
- net GND: now also J4.3 (Pin_3); no longer J5.1 (Pin_1)
- net int: now also J4.4 (Pin_4)
- net reset: now also J4.2 (Pin_2)

Commit message: office
Parts:
- removed J6: clock rate, Connector_PinHeader_2.54mm:PinHeader_2x03_P2.54mm_Vertical, symbol Connector_Generic:Conn_02x03_Top_Bottom
- added J6: clock selector, Connector_PinHeader_2.54mm:PinHeader_2x03_P2.54mm_Vertical, symbol Connector_Generic:Conn_02x03_Odd_Even
Connections:
- net clk: now also J6.2 (Pin_2), J6.4 (Pin_4), J6.6 (Pin_6)
- net at U1.8, U2.3 (C): now also J6.1 (Pin_1)
- net at U2.11 (C), U2.5 (Q): now also J6.3 (Pin_3)
- net at U2.9 (Q): now also J6.5 (Pin_5)
Changed lines of the file:
@@
 EESchema Schematic File Version 4
-LIBS:CPU-cache
 EELAYER 30 0
 EELAYER END
@@
 	0    -1   -1   0
 $EndComp
-$Comp
-L Connector_Generic:Conn_02x03_Top_Bottom J6
-U 1 1 5E640B5B
-P 7750 2550
-F 0 "J6" H 7800 2867 50  0000 C CNN
-F 1 "clock rate" H 7800 2776 50  0000 C CNN
-F 2 "Connector_PinHeader_2.54mm:PinHeader_2x03_P2.54mm_Vertical" H 7750 2550 50  0001 C CNN
-F 3 "~" H 7750 2550 50  0001 C CNN
-	1    7750 2550
-	1    0    0    -1
-$EndComp
 Wire Wire Line
 	7150 2550 7150 2900
@@
 Text Label 6100 6600 0    50   ~ 0
 int
+$Comp
+L Connector_Generic:Conn_02x03_Odd_Even J6
+U 1 1 60D99554
+P 7750 2550
+F 0 "J6" H 7800 2867 50  0000 C CNN
+F 1 "clock selector" H 7800 2776 50  0000 C CNN
+F 2 "Connector_PinHeader_2.54mm:PinHeader_2x03_P2.54mm_Vertical" H 7750 2550 50  0001 C CNN
+F 3 "~" H 7750 2550 50  0001 C CNN
+	1    7750 2550
+	1    0    0    -1
+$EndComp
 $EndSCHEMATC

Commit message: office
Parts:
- R3, R6: value 270 -> 270R
- R4: value 100 -> 100R
- R5: value 10k -> 1k
Changed lines of the file:
@@
 P 7300 1750
 F 0 "R5" H 7370 1796 50  0000 L CNN
-F 1 "10k" H 7370 1705 50  0000 L CNN
+F 1 "1k" H 7370 1705 50  0000 L CNN
 F 2 "Resistor_THT:R_Axial_DIN0207_L6.3mm_D2.5mm_P10.16mm_Horizontal" V 7230 1750 50  0001 C CNN
 F 3 "~" H 7300 1750 50  0001 C CNN
@@
 P 7050 1500
 F 0 "R4" V 7257 1500 50  0000 C CNN
-F 1 "100" V 7166 1500 50  0000 C CNN
+F 1 "100R" V 7166 1500 50  0000 C CNN
 F 2 "Resistor_THT:R_Axial_DIN0207_L6.3mm_D2.5mm_P10.16mm_Horizontal" V 6980 1500 50  0001 C CNN
 F 3 "~" H 7050 1500 50  0001 C CNN
@@
 P 7850 5050
 F 0 "R6" H 7920 5096 50  0000 L CNN
-F 1 "270" H 7920 5005 50  0000 L CNN
+F 1 "270R" H 7920 5005 50  0000 L CNN
 F 2 "Resistor_THT:R_Axial_DIN0207_L6.3mm_D2.5mm_P10.16mm_Horizontal" V 7780 5050 50  0001 C CNN
 F 3 "~" H 7850 5050 50  0001 C CNN
@@
 P 6500 4900
 F 0 "R3" H 6570 4946 50  0000 L CNN
-F 1 "270" H 6570 4855 50  0000 L CNN
+F 1 "270R" H 6570 4855 50  0000 L CNN
 F 2 "Resistor_THT:R_Axial_DIN0207_L6.3mm_D2.5mm_P10.16mm_Horizontal" V 6430 4900 50  0001 C CNN
 F 3 "~" H 6500 4900 50  0001 C CNN
