File: KiCAD files/FLASHv2/FLASHv2.sch (KiCad schematic (older format))
At the start: 17 parts, among them J1 card addr, J2 Power Bus, J3 Signal Bus, J4 IDE connector, U1 74LS04, U2 74LS85, U3 74LS245, U4 74LS245

Commit message: A
Connections:
- net GND: now also U3.16 (B2), U3.17 (B1), U3.18 (B0), U3.2 (A0), U3.3 (A1), U3.4 (A2)
- no-connect marks 55 -> 49
Changed lines of the file:
@@
 Text Label 5850 4150 2    50   ~ 0
 wr
-NoConn ~ 5850 3850
-NoConn ~ 5850 3950
-NoConn ~ 5850 4050
-NoConn ~ 6850 3850
-NoConn ~ 6850 3950
-NoConn ~ 6850 4050
 Wire Wire Line
 	7100 2450 5550 2450
@@
 Text Label 9450 2750 2    50   ~ 0
 fd07
+Wire Wire Line
+	5850 3850 5850 3950
+Wire Wire Line
+	5850 4050 5850 3950
+Connection ~ 5850 3950
+Wire Wire Line
+	6850 3850 6850 3950
+Wire Wire Line
+	6850 3950 6850 4050
+Connection ~ 6850 3950
+$Comp
+L power:GND #PWR?
+U 1 1 6088510C
+P 6850 3950
+F 0 "#PWR?" H 6850 3700 50  0001 C CNN
+F 1 "GND" V 6950 3850 50  0000 C CNN
+F 2 "" H 6850 3950 50  0001 C CNN
+F 3 "" H 6850 3950 50  0001 C CNN
+	1    6850 3950
+	0    -1   1    0
+$EndComp
+$Comp
+L power:GND #PWR?
+U 1 1 6088AC73
+P 5850 3950
+F 0 "#PWR?" H 5850 3700 50  0001 C CNN
+F 1 "GND" V 5900 3750 50  0000 C CNN
+F 2 "" H 5850 3950 50  0001 C CNN
+F 3 "" H 5850 3950 50  0001 C CNN
+	1    5850 3950
+	0    1    1    0
+$EndComp
 $EndSCHEMATC

Commit message: office
Parts:
- removed R1, R2, R3, R4: 10k, symbol Device:R
- added RN1: 4x10k, Resistor_THT:R_Array_SIP5, symbol Device:R_Network04
Connections:
- net +5V: now also RN1.1 (common)
- net GND: no longer U3.16 (B2), U3.17 (B1), U3.18 (B0)
- net at J1.2 (Pin_2), U2.1 (B3): now also RN1.2 (R1)
- net at J1.6 (Pin_6), U2.11 (B1): now also RN1.4 (R3)
- net at J1.4 (Pin_4), U2.14 (B2): now also RN1.3 (R2)
- net at J1.8 (Pin_8), U2.9 (B0): now also RN1.5 (R4)
- no-connect marks 49 -> 52
Changed lines of the file:
@@
 EESchema Schematic File Version 4
-LIBS:FLASHv2-cache
 EELAYER 30 0
 EELAYER END
@@
 $EndComp
 Wire Wire Line
-	2650 4800 1850 4800
-Wire Wire Line
-	1750 4900 2050 4900
-Wire Wire Line
-	2650 5000 2250 5000
-Wire Wire Line
-	1750 5100 2450 5100
-Wire Wire Line
 	1250 4800 1250 4900
 Wire Wire Line
@@
 Connection ~ 3650 4800
 $Comp
-L Device:R R1
-U 1 1 5E8F1A02
-P 1850 4500
-F 0 "R1" V 1950 4600 50  0000 C CNN
-F 1 "10k" V 1950 4450 50  0000 C CNN
-F 2 "" V 1780 4500 50  0001 C CNN
-F 3 "~" H 1850 4500 50  0001 C CNN
-	1    1850 4500
-	1    0    0    -1
-$EndComp
-$Comp
-L Device:R R2
-U 1 1 5E8F954C
-P 2050 4500
-F 0 "R2" V 2150 4600 50  0000 C CNN
-F 1 "10k" V 2150 4450 50  0000 C CNN
-F 2 "" V 1980 4500 50  0001 C CNN
-F 3 "~" H 2050 4500 50  0001 C CNN
-	1    2050 4500
-	1    0    0    -1
-$EndComp
-$Comp
-L Device:R R3
-U 1 1 5E8FB1E6
-P 2250 4500
-F 0 "R3" V 2350 4600 50  0000 C CNN
-F 1 "10k" V 2350 4450 50  0000 C CNN
-F 2 "" V 2180 4500 50  0001 C CNN
-F 3 "~" H 2250 4500 50  0001 C CNN
-	1    2250 4500
-	1    0    0    -1
-$EndComp
-$Comp
-L Device:R R4
-U 1 1 5E8FCDB9
-P 2450 4500
-F 0 "R4" V 2550 4600 50  0000 C CNN
-F 1 "10k" V 2550 4450 50  0000 C CNN
-F 2 "" V 2380 4500 50  0001 C CNN
-F 3 "~" H 2450 4500 50  0001 C CNN
-	1    2450 4500
-	1    0    0    -1
-$EndComp
-Wire Wire Line
-	1850 4650 1850 4800
-Connection ~ 1850 4800
-Wire Wire Line
-	1850 4800 1750 4800
-Wire Wire Line
-	2050 4650 2050 4900
-Connection ~ 2050 4900
-Wire Wire Line
-	2050 4900 2650 4900
-Wire Wire Line
-	2250 4650 2250 5000
-Connection ~ 2250 5000
-Wire Wire Line
-	2250 5000 1750 5000
-Wire Wire Line
-	2450 4650 2450 5100
-Connection ~ 2450 5100
-Wire Wire Line
-	2450 5100 2650 5100
-Wire Wire Line
-	1850 4350 1850 4250
-Wire Wire Line
-	1850 4250 2050 4250
-Wire Wire Line
-	2450 4250 2450 4350
-Wire Wire Line
-	2250 4350 2250 4250
-Connection ~ 2250 4250
-Wire Wire Line
-	2250 4250 2450 4250
-Wire Wire Line
-	2050 4350 2050 4250
-Connection ~ 2050 4250
-$Comp
 L power:+5V #PWR02
 U 1 1 5E914060
-P 2050 4100
-F 0 "#PWR02" H 2050 3950 50  0001 C CNN
-F 1 "+5V" H 2065 4273 50  0000 C CNN
-F 2 "" H 2050 4100 50  0001 C CNN
-F 3 "" H 2050 4100 50  0001 C CNN
-	1    2050 4100
-	1    0    0    -1
-$EndComp
-Wire Wire Line
-	2050 4100 2050 4250
+P 2000 4150
+F 0 "#PWR02" H 2000 4000 50  0001 C CNN
+F 1 "+5V" H 2015 4323 50  0000 C CNN
+F 2 "" H 2000 4150 50  0001 C CNN
+F 3 "" H 2000 4150 50  0001 C CNN
+	1    2000 4150
+	1    0    0    -1
+$EndComp
 $Comp
 L power:GND #PWR01
@@
 NoConn ~ 3650 5400
 NoConn ~ 3650 5500
-Wire Wire Line
-	2050 4250 2250 4250
 Wire Wire Line
 	4900 5150 5100 5150
@@
 Connection ~ 6350 3550
 $Comp
-L power:GND #PWR025
-U 1 1 5FE2A96F
-P 5950 3550
-F 0 "#PWR025" H 5950 3300 50  0001 C CNN
-F 1 "GND" V 5955 3377 50  0000 C CNN
-F 2 "" H 5950 3550 50  0001 C CNN
-F 3 "" H 5950 3550 50  0001 C CNN
-	1    5950 3550
-	0    1    1    0
-$EndComp
-$Comp
 L power:GND #PWR026
 U 1 1 5FE324FA
@@
 Text Label 9450 2750 2    50   ~ 0
 fd07
+$Comp
+L Device:R_Network04 RN1
+U 1 1 60D30812
+P 2200 4450
+F 0 "RN1" H 2388 4496 50  0000 L CNN
+F 1 "4x10k" H 2388 4405 50  0000 L CNN
+F 2 "Resistor_THT:R_Array_SIP5" V 2475 4450 50  0001 C CNN
+F 3 "http://www.vishay.com/docs/31509/csc.pdf" H 2200 4450 50  0001 C CNN
+	1    2200 4450
+	1    0    0    -1
+$EndComp
+Wire Wire Line
+	1750 4800 2000 4800
+Wire Wire Line
+	1750 4900 2100 4900
+Wire Wire Line
+	1750 5000 2200 5000
+Wire Wire Line
+	1750 5100 2300 5100
+Wire Wire Line
+	2000 4150 2000 4250
+Wire Wire Line
+	2000 4650 2000 4800
+Connection ~ 2000 4800
+Wire Wire Line
+	2000 4800 2650 4800
+Wire Wire Line
+	2100 4650 2100 4900
+Connection ~ 2100 4900
+Wire Wire Line
+	2100 4900 2650 4900
+Wire Wire Line
+	2200 4650 2200 5000
+Connection ~ 2200 5000
+Wire Wire Line
+	2200 5000 2650 5000
+Wire Wire Line
+	2300 4650 2300 5100
+Connection ~ 2300 5100
+Wire Wire Line
+	2300 5100 2650 5100
+NoConn ~ 6850 3850
+NoConn ~ 6850 3950
+NoConn ~ 6850 4050
 Wire Wire Line
 	5850 3850 5850 3950
@@
 	5850 4050 5850 3950
 Connection ~ 5850 3950
-Wire Wire Line
-	6850 3850 6850 3950
-Wire Wire Line
-	6850 3950 6850 4050
-Connection ~ 6850 3950
-$Comp
-L power:GND #PWR?
-U 1 1 6088510C
-P 6850 3950
-F 0 "#PWR?" H 6850 3700 50  0001 C CNN
-F 1 "GND" V 6950 3850 50  0000 C CNN
-F 2 "" H 6850 3950 50  0001 C CNN
-F 3 "" H 6850 3950 50  0001 C CNN
-	1    6850 3950
-	0    -1   1    0
-$EndComp
-$Comp
-L power:GND #PWR?
-U 1 1 6088AC73
-P 5850 3950
-F 0 "#PWR?" H 5850 3700 50  0001 C CNN
-F 1 "GND" V 5900 3750 50  0000 C CNN
-F 2 "" H 5850 3950 50  0001 C CNN
-F 3 "" H 5850 3950 50  0001 C CNN
-	1    5850 3950
+$Comp
+L power:GND #PWR0101
+U 1 1 60D4BBB9
+P 5650 4000
+F 0 "#PWR0101" H 5650 3750 50  0001 C CNN
+F 1 "GND" H 5655 3827 50  0000 C CNN
+F 2 "" H 5650 4000 50  0001 C CNN
+F 3 "" H 5650 4000 50  0001 C CNN
+	1    5650 4000
+	1    0    0    -1
+$EndComp
+Wire Wire Line
+	5650 4000 5650 3950
+Wire Wire Line
+	5650 3950 5850 3950
+$Comp
+L power:GND #PWR0102
+U 1 1 60D57F2C
+P 5900 3550
+F 0 "#PWR0102" H 5900 3300 50  0001 C CNN
+F 1 "GND" V 5905 3422 50  0000 R CNN
+F 2 "" H 5900 3550 50  0001 C CNN
+F 3 "" H 5900 3550 50  0001 C CNN
+	1    5900 3550
 	0    1    1    0
 $EndComp
+Wire Wire Line
+	5900 3550 5950 3550
 $EndSCHEMATC

Commit message: home
Parts:
- added C5, C6: 10nF, Capacitor_THT:C_Disc_D3.8mm_W2.6mm_P2.50mm, symbol Device:C
- added unit 3 of U1
- added unit 4 of U1
- added unit 5 of U1
- added unit 6 of U1
- C1: footprint (none) -> Capacitor_THT:CP_Radial_D5.0mm_P2.50mm
- C2, C3, C4: footprint (none) -> Capacitor_THT:C_Disc_D3.8mm_W2.6mm_P2.50mm
- J1: footprint (none) -> Connector_PinHeader_2.54mm:PinHeader_2x04_P2.54mm_Vertical
- J2: footprint (none) -> Connector_PinHeader_2.54mm:PinHeader_2x05_P2.54mm_Vertical
- J3: footprint (none) -> Connector_PinHeader_2.54mm:PinHeader_2x20_P2.54mm_Vertical
- J4: footprint (none) -> Connector_PinHeader_2.00mm:PinHeader_2x22_P2.00mm_Vertical
- R6: footprint (none) -> Resistor_THT:R_Axial_DIN0207_L6.3mm_D2.5mm_P10.16mm_Horizontal
- U1: footprint (none) -> Package_DIP:DIP-14_W7.62mm_Socket_LongPads
- U2: footprint (none) -> Package_DIP:DIP-16_W7.62mm_Socket_LongPads
- U3, U4: footprint (none) -> Package_DIP:DIP-20_W7.62mm_Socket_LongPads
Connections:
- net +5V: now also C5.1, C6.1
- net GND: now also C5.2, C6.2, U1.11, U1.13, U1.5, U1.9
- no-connect marks 52 -> 56
Other:
- moved on the sheet: J3, U1G

Commit message: home
Connections:
- net +5V: now also J4.3 (Pin_3); no longer J4.41 (Pin_41)
- net GND: now also J4.44 (Pin_44); no longer J4.2 (Pin_2)
- net cf_sel: now also J4.7 (Pin_7); no longer J4.37 (Pin_37)
- net fa00: now also J4.9 (Pin_9); no longer J4.35 (Pin_35)
- net fa01: now also J4.11 (Pin_11); no longer J4.33 (Pin_33)
- net fa02: now also J4.10 (Pin_10); no longer J4.36 (Pin_36)
- net fd00: now also J4.27 (Pin_27); no longer J4.17 (Pin_17)
- net fd01: now also J4.29 (Pin_29); no longer J4.15 (Pin_15)
- net fd02: now also J4.31 (Pin_31); no longer J4.13 (Pin_13)
- net fd03: now also J4.33 (Pin_33); no longer J4.11 (Pin_11)
- net fd04: now also J4.35 (Pin_35); no longer J4.9 (Pin_9)
- net fd05: now also J4.37 (Pin_37); no longer J4.7 (Pin_7)
- net fd06: now also J4.39 (Pin_39); no longer J4.5 (Pin_5)
- net fd07: now also J4.41 (Pin_41); no longer J4.3 (Pin_3)
- net frd: now also J4.19 (Pin_19); no longer J4.25 (Pin_25)
- net fwr: now also J4.21 (Pin_21); no longer J4.23 (Pin_23)
- net reset: now also J4.43 (Pin_43); no longer J4.1 (Pin_1)
- net at R6.1: now also J4.8 (Pin_8); no longer J4.38 (Pin_38)
Changed lines of the file:
@@
 L Connector_Generic:Conn_02x22_Odd_Even J4
 U 1 1 5F5B7653
-P 9650 3650
-F 0 "J4" H 9700 4867 50  0000 C CNN
-F 1 "IDE connector" H 9700 4776 50  0000 C CNN
-F 2 "Connector_PinHeader_2.00mm:PinHeader_2x22_P2.00mm_Vertical" H 9650 3650 50  0001 C CNN
-F 3 "~" H 9650 3650 50  0001 C CNN
-	1    9650 3650
-	1    0    0    -1
+P 9650 3750
+F 0 "J4" H 9700 4967 50  0000 C CNN
+F 1 "IDE connector" H 9700 4876 50  0000 C CNN
+F 2 "Connector_PinHeader_2.00mm:PinHeader_2x22_P2.00mm_Vertical" H 9650 3750 50  0001 C CNN
+F 3 "~" H 9650 3750 50  0001 C CNN
+	1    9650 3750
+	1    0    0    1
 $EndComp
 $Comp
