File: KiCAD files/FLASHv2/FLASHv2.kicad_pcb (KiCad board)
At the start: 2 copper layers, 99.7 x 69.8 mm, 16 parts, among them J1 card addr, J2 Power Bus, J3 Signal Bus, J4 IDE connector, U1 74LS04, U2 74LS85, U3 74LS245, U4 74LS245

Commit message: home
Parts:
- moved U2 72.8 mm to (123.2, 130.8), turned to 90 degrees
- moved U1 59.7 mm to (125.1, 104.1), turned to 90 degrees
- moved C4 55.5 mm to (120.7, 69.2), turned to 270 degrees
- moved C5 46.8 mm to (120.7, 82.5), turned to 270 degrees
- moved C2 40.0 mm to (121.3, 95.9), turned to 270 degrees
- moved C6 36.0 mm to (156.8, 130.8)
- moved J4 35.6 mm to (156.8, 79.4)
- moved U4 33.2 mm to (124.8, 90.8), turned to 90 degrees
- moved R6 32.0 mm to (163.2, 69.8), turned to 180 degrees
- moved C3 21.6 mm to (119.4, 122.6), turned to 270 degrees
- moved J1 21.4 mm to (132.7, 117.5), turned to 90 degrees
- moved U3 15.6 mm to (124.8, 77.2), turned to 90 degrees
- moved RN1 13.1 mm to (130.2, 109.9)
- moved C1 3.86 mm to (114.9, 77.5), turned to 90 degrees
Connections:
- J4 pad 1: /reset -> Net-(J4-Pad1)
- J4 pad 10: Net-(J4-Pad10) -> /fa02
- J4 pad 11: /fd03 -> /fa01
- J4 pad 13: /fd02 -> Net-(J4-Pad13)
- J4 pad 15: /fd01 -> Net-(J4-Pad15)
- J4 pad 17: /fd00 -> Net-(J4-Pad17)
- J4 pad 19: Net-(J4-Pad19) -> /frd
- J4 pad 2: GND -> Net-(J4-Pad2)
- J4 pad 21: Net-(J4-Pad21) -> /fwr
- J4 pad 23: /fwr -> Net-(J4-Pad23)
- J4 pad 25: /frd -> Net-(J4-Pad25)
- J4 pad 27: Net-(J4-Pad27) -> /fd00
- J4 pad 29: Net-(J4-Pad29) -> /fd01
- J4 pad 3: /fd07 -> +5V
- J4 pad 31: Net-(J4-Pad31) -> /fd02
- J4 pad 33: /fa01 -> /fd03
- J4 pad 35: /fa00 -> /fd04
- J4 pad 36: /fa02 -> Net-(J4-Pad36)
- J4 pad 37: /cf_sel -> /fd05
- J4 pad 39: Net-(J4-Pad39) -> /fd06
- J4 pad 41: +5V -> /fd07
- J4 pad 43: Net-(J4-Pad43) -> /reset
- J4 pad 44: Net-(J4-Pad44) -> GND
- J4 pad 5: /fd06 -> Net-(J4-Pad5)
- J4 pad 7: /fd05 -> /cf_sel
- J4 pad 9: /fd04 -> /fa00
- R6 pad 1: Net-(J4-Pad38) -> Net-(J4-Pad8)
Routing:
- net GND: track 0.00 -> 236.6 mm
- net +5V: track 0.00 -> 181.9 mm
- net /rd: track 0.00 -> 93.0 mm
- net /cf_sel: track 0.00 -> 70.2 mm
- net /reset: track 0.00 -> 60.8 mm
- net /wr: track 0.00 -> 54.8 mm
- net /d07: track 0.00 -> 50.7 mm
- net /a02: track 0.00 -> 49.4 mm
- net /fd02: track 0.00 -> 49.1 mm
- net /a04: track 0.00 -> 48.8 mm, vias 0 -> 1
- net /fd03: track 0.00 -> 47.8 mm
- net /a05: track 0.00 -> 46.8 mm
- net /fd04: track 0.00 -> 46.5 mm
- net /fd05: track 0.00 -> 45.1 mm
- net /d06: track 0.00 -> 44.5 mm
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- added copper zone on B.Cu, net GND
Other:
- net class Power added: clearance 0.2, trace_width 0.375001, via_dia 0.8, via_drill 0.4
- board text added: "3 2 1 0"
- board text added: "Card Addr"
- board text added: "Compact Flash Card Adapter"
- board text added: "Z80 Modular Computer FLASH Card version 2.0 Design by Kaltchuk, 06/2021"

Commit message: pcb updates
Other:
- net class Default removed
- net class Power removed
