File: KiCAD files/preTTY/preTTY.sch (KiCad schematic (older format))
At the start: 27 parts, among them J1 Power Bus, J2 Signal Buss, J3 TTL/RS232, J4 PORT0 TTL, J5 PORT1 TTL/RS232, J6 DB9, U1 74LS07, U2 ATmega328P-PU, U3 MAX232, Y1 16MHz

Commit message: HOME
Connections:
- net a00: now also U2.28 (PC5)
- no-connect marks 35 -> 34
Changed lines of the file:
@@
 EESchema Schematic File Version 4
+LIBS:preTTY-cache
 EELAYER 30 0
 EELAYER END
@@
 Text Label 3900 5000 2    50   ~ 0
 iorq
-NoConn ~ 3900 5100
 NoConn ~ 5100 3700
 $Comp
@@
 Wire Wire Line
 	8850 5650 9750 5650
+Text Label 3900 5100 2    50   ~ 0
+a00
 $EndSCHEMATC

Commit message: office
Parts:
- removed A1: Arduino_Nano_v3.x, Module:Arduino_Nano, symbol preTTY-rescue:Arduino_Nano_v3.x-MCU_Module-USARTv2-rescue
- added C? (x2): 22pF, symbol Device:C
- added C? (x2): 10nF, symbol Device:C
- added J?: Card addr, symbol Connector_Generic:Conn_02x04_Odd_Even
- added RN?: 4x10k, Resistor_THT:R_Array_SIP5, symbol Device:R_Network04
- added U?: ATmega328P-PU, Package_DIP:DIP-28_W7.62mm, symbol preTTY-rescue:ATmega328P-PU-MCU_Microchip_ATmega
- added U?: 74LS85, symbol 74xx:74LS85
- added U? (x5): 74LS00, symbol 74xx:74LS00
- added Y?: 16MHz, symbol Device:Crystal
Connections:
- net +5V: now also C?.1, C?.1, RN?.1 (common), U?.14 (VCC), U?.16 (VCC), U?.20 (AVCC), U?.7 (VCC)
- net GND: now also C?.2, C?.2, C?.2, C?.2, J?.1 (Pin_1), J?.3 (Pin_3), J?.5 (Pin_5), J?.7 (Pin_7), U?.2 (Ia<b), U?.22 (GND), U?.4 (Ia>b), U?.7 (GND), U?.8 (GND), U?.8 (GND)
- net RX0: now also U?.2 (PD0)
- net TX0: now also U?.3 (PD1)
- net a00: now also U?.12, U?.13, U?.5; no longer U2.28 (PC5)
- net a01: now also U2.24 (PC1), U?.24 (PC1); no longer U2.16 (PB2)
- net a04: now also U?.10 (A0); no longer U2.23 (PC0)
- net a05: now also U?.12 (A1); no longer U2.24 (PC1)
- net a06: now also U?.13 (A2); no longer U2.25 (PC2)
- net a07: now also U?.15 (A3); no longer U2.26 (PC3)
- net d00: now also U?.4 (PD2)
- net d01: now also U?.5 (PD3)
- net d02: now also U?.6 (PD4)
- net d03: now also U?.11 (PD5)
- net d04: now also U?.12 (PD6)
- net d05: now also U?.13 (PD7)
- net d06: now also U?.14 (PB0)
- net d07: now also U?.15 (PB1)
- net iorq: now also U?.1, U?.2; no longer U2.27 (PC4)
- net rd: now also U2.25 (PC2), U?.25 (PC2); no longer U2.17 (PB3)
- net reset: now also U?.1 (~RESET~/PC6)
- net wr: now also U2.26 (PC3), U?.26 (PC3); no longer U2.18 (PB4)
- new net: C?.1, U?.10 (XTAL2/PB7), Y?.2
- new net: C?.1, U?.9 (XTAL1/PB6), Y?.1
- new net: J?.2 (Pin_2), RN?.2 (R1), U?.1 (B3)
- new net: J?.6 (Pin_6), RN?.4 (R3), U?.11 (B1)
- new net: J?.4 (Pin_4), RN?.3 (R2), U?.14 (B2)
- new net: U?.3, U?.3 (Ia=b)
- new net: U?.4, U?.6 (Oa=b), U?.9
- new net: J?.8 (Pin_8), RN?.5 (R4), U?.9 (B0)
- new net: U?.10, U?.11
- new net cs0: U?.23 (PC0), U?.8
- new net cs1: U2.23 (PC0), U?.6
- no-connect marks 34 -> 42
Other:
- moved on the sheet: C1, C2, C3, C4, C5, C6, C7, D1, D2, D3, D4, J1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

Commit message: office
Parts:
- removed C5, C6: 22pF, symbol Device:C
- removed C?: 10nF, symbol Device:C
- removed D3, D4: LED, symbol Device:LED
- removed J3: TTL/RS232, symbol Connector_Generic:Conn_02x03_Odd_Even
- removed J4: PORT0 TTL, symbol Connector_Generic:Conn_02x02_Odd_Even
- removed J5: PORT1 TTL/RS232, symbol Connector_Generic:Conn_02x04_Odd_Even
- removed U2: ATmega328P-PU, Package_DIP:DIP-28_W7.62mm, symbol preTTY-rescue:ATmega328P-PU-MCU_Microchip_ATmega
- removed Y1: 16MHz, symbol Device:Crystal
- added J4: ISP, symbol Connector_Generic:Conn_02x03_Odd_Even
- added J5: TTL/RS232, symbol Connector_Generic:Conn_01x03
- added J6: TTL PORT0, symbol Connector_Generic:Conn_01x03
- added R1: 22k, symbol Device:R
- Y1: renamed from Y?; value 16MHz -> 20MHz
- gave numbers to parts that had none: 8
- renumbered C9 to C10, C10 to C11, C11 to C12, C3 to C4, C4 to C5, C2 to C7, C7 to C8, C8 to C9, J6 to J7, RN1 to RN2, U1 to U2, U3 to U5
Connections:
- net RX1 is gone; now on net GND: U2.9
- net +5V: now also J4.2 (Pin_2), R1.1
- net GND: now also U2.5, J4.6 (Pin_6), J6.3 (Pin_3)
- net RX0: now also J5.2 (Pin_2)
- net RX0RS232: now also J5.3 (Pin_3)
- net RX0TTL: now also J5.1 (Pin_1), J6.2 (Pin_2)
- net TX0: now also J6.1 (Pin_1)
- net a01: now also U1.23 (PC0); no longer U1.24 (PC1)
- net cs0: now also U1.4 (PD2); no longer U1.23 (PC0)
- net d00: now also U1.14 (PB0); no longer U1.4 (PD2)
- net d01: now also U1.15 (PB1); no longer U1.5 (PD3)
- net d02: now also U1.16 (PB2); no longer U1.6 (PD4)
- net d03: now also U1.5 (PD3); no longer U1.11 (PD5)
- net d04: now also U1.6 (PD4); no longer U1.12 (PD6)
- net d05: now also U1.11 (PD5); no longer U1.13 (PD7)
- net d06: now also U1.12 (PD6); no longer U1.14 (PB0)
- net d07: now also U1.13 (PD7); no longer U1.15 (PB1)
- net rd: now also U1.24 (PC1); no longer U1.25 (PC2)
- net reset: now also J4.5 (Pin_5), R1.2
- net wr: now also U1.25 (PC2); no longer U1.26 (PC3)
- net mosi: now reaches U1.17 (PB3)
- net mosi: now also J4.4 (Pin_4)
- net miso: now reaches U1.18 (PB4)
- net miso: now also J4.1 (Pin_1)
- net sck: now reaches U1.19 (PB5)
- net sck: now also J4.3 (Pin_3)
- net RX1RS232: no longer names the net of U5.9 (R2OUT)
- net TX1: no longer names the net of U5.10 (T2IN)
- net TX1: no longer U2.5
- no-connect marks 42 -> 41
Other:
- note removed: "RX1"
- note removed: "TX1"
- moved on the sheet: U2C, U2D, U2E, U2F

Commit message: office
Connections:
- net cs0 renamed CS0
- net cs1 renamed CS1
- net miso renamed MISO
- net mosi renamed MOSI
- net sck renamed SCK
Other:
- moved on the sheet: J4, J5
Changed lines of the file:
@@
 Text Label 9800 2350 2    50   ~ 0
 RX0TTL
-Text Label 8250 2250 2    50   ~ 0
+Text Label 5200 4050 2    50   ~ 0
 RX0TTL
-Text Label 8250 2350 2    50   ~ 0
+Text Label 5200 4150 2    50   ~ 0
 RX0
-Text Label 8250 2450 2    50   ~ 0
+Text Label 5200 4250 2    50   ~ 0
 RX0RS232
 $Comp
@@
 iorq
 Text Label 7300 2950 0    50   ~ 0
-cs0
+CS0
 Text Label 5850 3150 2    50   ~ 0
 a00
@@
 L Connector_Generic:Conn_01x03 J5
 U 1 1 61202836
-P 8450 2350
-F 0 "J5" H 8530 2392 50  0000 L CNN
-F 1 "TTL/RS232" H 8530 2301 50  0000 L CNN
-F 2 "" H 8450 2350 50  0001 C CNN
-F 3 "~" H 8450 2350 50  0001 C CNN
-	1    8450 2350
+P 5400 4150
+F 0 "J5" H 5480 4192 50  0000 L CNN
+F 1 "TTL/RS232" H 5480 4101 50  0000 L CNN
+F 2 "" H 5400 4150 50  0001 C CNN
+F 3 "~" H 5400 4150 50  0001 C CNN
+	1    5400 4150
 	1    0    0    -1
 $EndComp
@@
 d02
 Text Label 1600 4000 2    50   ~ 0
-mosi
+MOSI
 Text Label 1600 4100 2    50   ~ 0
-miso
+MISO
 Text Label 1600 4200 2    50   ~ 0
-sck
+SCK
 Text Label 1600 4600 2    50   ~ 0
 a01
@@
 NoConn ~ 1600 5100
 Text Label 1600 5600 2    50   ~ 0
-cs0
+CS0
 Text Label 1600 5700 2    50   ~ 0
 d03
@@
 L Connector_Generic:Conn_02x03_Odd_Even J4
 U 1 1 61227C0B
-P 4300 4100
-F 0 "J4" H 4350 4417 50  0000 C CNN
-F 1 "ISP" H 4350 4326 50  0000 C CNN
-F 2 "" H 4300 4100 50  0001 C CNN
-F 3 "~" H 4300 4100 50  0001 C CNN
-	1    4300 4100
-	1    0    0    -1
-$EndComp
-Text Label 4100 4000 2    50   ~ 0
-miso
-Text Label 4100 4100 2    50   ~ 0
-sck
-Text Label 4100 4200 2    50   ~ 0
+P 3700 4150
+F 0 "J4" H 3750 4467 50  0000 C CNN
+F 1 "ISP" H 3750 4376 50  0000 C CNN
+F 2 "" H 3700 4150 50  0001 C CNN
+F 3 "~" H 3700 4150 50  0001 C CNN
+	1    3700 4150
+	1    0    0    -1
+$EndComp
+Text Label 3500 4050 2    50   ~ 0
+MISO
+Text Label 3500 4150 2    50   ~ 0
+SCK
+Text Label 3500 4250 2    50   ~ 0
 reset
-Text Label 4600 4100 0    50   ~ 0
-mosi
+Text Label 4000 4150 0    50   ~ 0
+MOSI
 $Comp
 L power:+5V #PWR024
 U 1 1 6122E66E
-P 4600 4000
-F 0 "#PWR024" H 4600 3850 50  0001 C CNN
-F 1 "+5V" H 4615 4173 50  0000 C CNN
-F 2 "" H 4600 4000 50  0001 C CNN
-F 3 "" H 4600 4000 50  0001 C CNN
-	1    4600 4000
+P 4000 4050
+F 0 "#PWR024" H 4000 3900 50  0001 C CNN
+F 1 "+5V" H 4015 4223 50  0000 C CNN
+F 2 "" H 4000 4050 50  0001 C CNN
+F 3 "" H 4000 4050 50  0001 C CNN
+	1    4000 4050
 	1    0    0    -1
 $EndComp
@@
 L power:GND #PWR025
 U 1 1 61230D7B
-P 4600 4200
-F 0 "#PWR025" H 4600 3950 50  0001 C CNN
-F 1 "GND" H 4605 4027 50  0000 C CNN
-F 2 "" H 4600 4200 50  0001 C CNN
-F 3 "" H 4600 4200 50  0001 C CNN
-	1    4600 4200
+P 4000 4250
+F 0 "#PWR025" H 4000 4000 50  0001 C CNN
+F 1 "GND" H 4005 4077 50  0000 C CNN
+F 2 "" H 4000 4250 50  0001 C CNN
+F 3 "" H 4000 4250 50  0001 C CNN
+	1    4000 4250
 	1    0    0    -1
 $EndComp
@@
 	950  5200 950  5150
 Text Label 7300 2400 0    50   ~ 0
-cs1
+CS1
 $EndSCHEMATC
