File: KiCAD files/preTTY/preTTY.sch (KiCad schematic (older format))
At the start: 35 parts, among them J1 Power Bus, J2 Signal Buss, J3 Card addr, J4 ISP, J5 TTL/RS232, J6 TTL PORT0, J7 DB9, U1 ATmega328P-PU, U2 74LS07, U3 74LS00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

Commit message: office
Parts:
- added C15: 10nF, symbol Device:C
- added unit 3 of U6
- added U8: 74LS245, symbol 74xx:74LS245
Connections:
- net +5V: now also C15.1, U8.20 (VCC)
- net CS0: now also U6.9
- net CS1: now also U6.10
- net GND: now also C15.2, U8.10 (GND)
- net d00: now also U8.2 (A0); no longer U1.14 (PB0)
- net d01: now also U8.3 (A1); no longer U1.15 (PB1)
- net d02: now also U8.4 (A2); no longer U1.16 (PB2)
- net d03: now also U8.5 (A3); no longer U1.5 (PD3)
- net d04: now also U8.6 (A4); no longer U1.6 (PD4)
- net d05: now also U8.7 (A5); no longer U1.11 (PD5)
- net d06: now also U8.8 (A6); no longer U1.12 (PD6)
- net d07: now also U8.9 (A7); no longer U1.13 (PD7)
- net rd: now also U8.1 (A->B)
- new net: U6.8, U8.19 (CE)
- new net B00: U1.14 (PB0), U8.18 (B0)
- new net B01: U1.15 (PB1), U8.17 (B1)
- new net B02: U1.16 (PB2), U8.16 (B2)
- new net B03: U1.5 (PD3), U8.15 (B3)
- new net B04: U1.6 (PD4), U8.14 (B4)
- new net B05: U1.11 (PD5), U8.13 (B5)
- new net B06: U1.12 (PD6), U8.12 (B6)
- new net B07: U1.13 (PD7), U8.11 (B7)
- no-connect marks 42 -> 41
Other:
- moved on the sheet: C8, J4, J5
Changed lines of the file:
@@
 L Device:CP C8
 U 1 1 60E8B5C2
-P 3300 7200
-F 0 "C8" H 3400 7250 50  0000 L CNN
-F 1 "1uF" H 3400 7150 50  0000 L CNN
-F 2 "" H 3338 7050 50  0001 C CNN
-F 3 "~" H 3300 7200 50  0001 C CNN
-	1    3300 7200
+P 8850 3650
+F 0 "C8" H 8950 3700 50  0000 L CNN
+F 1 "1uF" H 8950 3600 50  0000 L CNN
+F 2 "" H 8888 3500 50  0001 C CNN
+F 3 "~" H 8850 3650 50  0001 C CNN
+	1    8850 3650
 	1    0    0    -1
 $EndComp
@@
 L power:+5V #PWR017
 U 1 1 60E8DB35
-P 3300 7050
-F 0 "#PWR017" H 3300 6900 50  0001 C CNN
-F 1 "+5V" H 3315 7223 50  0000 C CNN
-F 2 "" H 3300 7050 50  0001 C CNN
-F 3 "" H 3300 7050 50  0001 C CNN
-	1    3300 7050
+P 8850 3500
+F 0 "#PWR017" H 8850 3350 50  0001 C CNN
+F 1 "+5V" H 8865 3673 50  0000 C CNN
+F 2 "" H 8850 3500 50  0001 C CNN
+F 3 "" H 8850 3500 50  0001 C CNN
+	1    8850 3500
 	1    0    0    -1
 $EndComp
@@
 L power:GND #PWR018
 U 1 1 60E8E4E5
-P 3300 7350
-F 0 "#PWR018" H 3300 7100 50  0001 C CNN
-F 1 "GND" H 3305 7177 50  0000 C CNN
-F 2 "" H 3300 7350 50  0001 C CNN
-F 3 "" H 3300 7350 50  0001 C CNN
-	1    3300 7350
+P 8850 3800
+F 0 "#PWR018" H 8850 3550 50  0001 C CNN
+F 1 "GND" H 8855 3627 50  0000 C CNN
+F 2 "" H 8850 3800 50  0001 C CNN
+F 3 "" H 8850 3800 50  0001 C CNN
+	1    8850 3800
 	1    0    0    -1
 $EndComp
@@
 Text Label 9900 5800 2    50   ~ 0
 RX0TTL
-Text Label 5200 4050 2    50   ~ 0
+Text Label 5500 4500 2    50   ~ 0
 RX0TTL
-Text Label 5200 4150 2    50   ~ 0
+Text Label 5500 4600 2    50   ~ 0
 RX0
-Text Label 5200 4250 2    50   ~ 0
+Text Label 5500 4700 2    50   ~ 0
 RX0RS232
 $Comp
@@
 NoConn ~ 10150 1300
 NoConn ~ 10150 1400
-NoConn ~ 7300 2400
 NoConn ~ 6700 4950
 NoConn ~ 6700 5350
@@
 L Connector_Generic:Conn_01x03 J5
 U 1 1 61202836
-P 5400 4150
-F 0 "J5" H 5480 4192 50  0000 L CNN
-F 1 "TTL/RS232" H 5480 4101 50  0000 L CNN
-F 2 "" H 5400 4150 50  0001 C CNN
-F 3 "~" H 5400 4150 50  0001 C CNN
-	1    5400 4150
+P 5700 4600
+F 0 "J5" H 5780 4642 50  0000 L CNN
+F 1 "TTL/RS232" H 5780 4551 50  0000 L CNN
+F 2 "" H 5700 4600 50  0001 C CNN
+F 3 "~" H 5700 4600 50  0001 C CNN
+	1    5700 4600
 	1    0    0    -1
 $EndComp
@@
 	1400 4300 1400 4200
 Text Label 1600 3700 2    50   ~ 0
-d00
+B00
 Text Label 1600 3800 2    50   ~ 0
-d01
+B01
 Text Label 1600 3900 2    50   ~ 0
-d02
+B02
 Text Label 1600 4000 2    50   ~ 0
 MOSI
@@
 CS0
 Text Label 1600 5700 2    50   ~ 0
-d03
+B03
 Text Label 1600 5800 2    50   ~ 0
-d04
+B04
 Text Label 1600 5900 2    50   ~ 0
-d05
+B05
 Text Label 1600 6000 2    50   ~ 0
-d06
+B06
 Text Label 1600 6100 2    50   ~ 0
-d07
+B07
 $Comp
 L Connector_Generic:Conn_02x03_Odd_Even J4
 U 1 1 61227C0B
-P 3700 4150
-F 0 "J4" H 3750 4467 50  0000 C CNN
-F 1 "ISP" H 3750 4376 50  0000 C CNN
-F 2 "" H 3700 4150 50  0001 C CNN
-F 3 "~" H 3700 4150 50  0001 C CNN
-	1    3700 4150
-	1    0    0    -1
-$EndComp
-Text Label 3500 4050 2    50   ~ 0
+P 5650 3950
+F 0 "J4" H 5700 4267 50  0000 C CNN
+F 1 "ISP" H 5700 4176 50  0000 C CNN
+F 2 "" H 5650 3950 50  0001 C CNN
+F 3 "~" H 5650 3950 50  0001 C CNN
+	1    5650 3950
+	1    0    0    -1
+$EndComp
+Text Label 5450 3850 2    50   ~ 0
 MISO
-Text Label 3500 4150 2    50   ~ 0
+Text Label 5450 3950 2    50   ~ 0
 SCK
-Text Label 3500 4250 2    50   ~ 0
+Text Label 5450 4050 2    50   ~ 0
 reset
-Text Label 4000 4150 0    50   ~ 0
+Text Label 5950 3950 0    50   ~ 0
 MOSI
 $Comp
 L power:+5V #PWR024
 U 1 1 6122E66E
-P 4000 4050
-F 0 "#PWR024" H 4000 3900 50  0001 C CNN
-F 1 "+5V" H 4015 4223 50  0000 C CNN
-F 2 "" H 4000 4050 50  0001 C CNN
-F 3 "" H 4000 4050 50  0001 C CNN
-	1    4000 4050
+P 5950 3850
+F 0 "#PWR024" H 5950 3700 50  0001 C CNN
+F 1 "+5V" H 5965 4023 50  0000 C CNN
+F 2 "" H 5950 3850 50  0001 C CNN
+F 3 "" H 5950 3850 50  0001 C CNN
+	1    5950 3850
 	1    0    0    -1
 $EndComp
@@
 L power:GND #PWR025
 U 1 1 61230D7B
-P 4000 4250
-F 0 "#PWR025" H 4000 4000 50  0001 C CNN
-F 1 "GND" H 4005 4077 50  0000 C CNN
-F 2 "" H 4000 4250 50  0001 C CNN
-F 3 "" H 4000 4250 50  0001 C CNN
-	1    4000 4250
+P 5950 4050
+F 0 "#PWR025" H 5950 3800 50  0001 C CNN
+F 1 "GND" H 5955 3877 50  0000 C CNN
+F 2 "" H 5950 4050 50  0001 C CNN
+F 3 "" H 5950 4050 50  0001 C CNN
+	1    5950 4050
 	1    0    0    -1
 $EndComp
@@
 	1    0    0    -1
 $EndComp
+$Comp
+L 74xx:74LS245 U8
+U 1 1 6130BFED
+P 4400 3450
+F 0 "U8" H 4750 4300 50  0000 C CNN
+F 1 "74LS245" H 4750 4200 50  0000 C CNN
+F 2 "" H 4400 3450 50  0001 C CNN
+F 3 "http://www.ti.com/lit/gpn/sn74LS245" H 4400 3450 50  0001 C CNN
+	1    4400 3450
+	1    0    0    -1
+$EndComp
+$Comp
+L Device:C C15
+U 1 1 6131AA6F
+P 3150 7200
+F 0 "C15" H 3265 7246 50  0000 L CNN
+F 1 "10nF" H 3265 7155 50  0000 L CNN
+F 2 "" H 3188 7050 50  0001 C CNN
+F 3 "~" H 3150 7200 50  0001 C CNN
+	1    3150 7200
+	1    0    0    -1
+$EndComp
+$Comp
+L power:GND #PWR053
+U 1 1 6131AA79
+P 3150 7350
+F 0 "#PWR053" H 3150 7100 50  0001 C CNN
+F 1 "GND" H 3155 7177 50  0000 C CNN
+F 2 "" H 3150 7350 50  0001 C CNN
+F 3 "" H 3150 7350 50  0001 C CNN
+	1    3150 7350
+	1    0    0    -1
+$EndComp
+$Comp
+L power:+5V #PWR052
+U 1 1 6131AA83
+P 3150 7050
+F 0 "#PWR052" H 3150 6900 50  0001 C CNN
+F 1 "+5V" H 3165 7223 50  0000 C CNN
+F 2 "" H 3150 7050 50  0001 C CNN
+F 3 "" H 3150 7050 50  0001 C CNN
+	1    3150 7050
+	1    0    0    -1
+$EndComp
+$Comp
+L 74xx:74LS08 U6
+U 3 1 61320FC1
+P 3450 3950
+F 0 "U6" H 3450 4275 50  0000 C CNN
+F 1 "74LS08" H 3450 4184 50  0000 C CNN
+F 2 "" H 3450 3950 50  0001 C CNN
+F 3 "http://www.ti.com/lit/gpn/sn74LS08" H 3450 3950 50  0001 C CNN
+	3    3450 3950
+	1    0    0    -1
+$EndComp
+Text Label 3150 3850 2    50   ~ 0
+CS0
+Text Label 3150 4050 2    50   ~ 0
+CS1
+Text Label 3900 3850 2    50   ~ 0
+rd
+Text Label 3900 2950 2    50   ~ 0
+d00
+Text Label 3900 3050 2    50   ~ 0
+d01
+Text Label 3900 3150 2    50   ~ 0
+d02
+Text Label 3900 3250 2    50   ~ 0
+d03
+Text Label 3900 3350 2    50   ~ 0
+d04
+Text Label 3900 3450 2    50   ~ 0
+d05
+Text Label 3900 3550 2    50   ~ 0
+d06
+Text Label 3900 3650 2    50   ~ 0
+d07
+Text Label 4900 2950 0    50   ~ 0
+B00
+Text Label 4900 3050 0    50   ~ 0
+B01
+Text Label 4900 3150 0    50   ~ 0
+B02
+Text Label 4900 3250 0    50   ~ 0
+B03
+Text Label 4900 3350 0    50   ~ 0
+B04
+Text Label 4900 3450 0    50   ~ 0
+B05
+Text Label 4900 3550 0    50   ~ 0
+B06
+Text Label 4900 3650 0    50   ~ 0
+B07
+Wire Wire Line
+	3900 3950 3750 3950
+$Comp
+L power:GND #PWR055
+U 1 1 6135B82A
+P 4400 4250
+F 0 "#PWR055" H 4400 4000 50  0001 C CNN
+F 1 "GND" H 4405 4077 50  0000 C CNN
+F 2 "" H 4400 4250 50  0001 C CNN
+F 3 "" H 4400 4250 50  0001 C CNN
+	1    4400 4250
+	1    0    0    -1
+$EndComp
+$Comp
+L power:+5V #PWR054
+U 1 1 6135EA7D
+P 4400 2650
+F 0 "#PWR054" H 4400 2500 50  0001 C CNN
+F 1 "+5V" H 4415 2823 50  0000 C CNN
+F 2 "" H 4400 2650 50  0001 C CNN
+F 3 "" H 4400 2650 50  0001 C CNN
+	1    4400 2650
+	1    0    0    -1
+$EndComp

Commit message: HOME
Changed lines of the file:
@@
 EESchema Schematic File Version 4
+LIBS:preTTY-cache
 EELAYER 30 0
 EELAYER END
@@
 	1    0    0    -1
 $EndComp
+Wire Wire Line
+	2800 2200 2450 2200
+Wire Wire Line
+	2450 2200 2450 2050
+Wire Wire Line
+	2800 2300 2350 2300
+Wire Wire Line
+	2350 2300 2350 2050
 $EndSCHEMATC
