File: KiCAD files/MEM/MEM.sch (KiCad schematic (older format))
At the start: 36 parts, among them J1 Power Bus, J2 Signal Bus, J3 card addr, J4 ROM block, J5 RAM bank, Q1 BC547, Q2 BC547, Q3 BC547, Q4 BC547, U1 74LS139, U2 74LS00, U3 74LS85, U4 74LS74, U5 W27C512, U6 628128

Commit message: office
Parts:
- removed R3, R4, R5, R6: 10k, symbol Device:R
- added RN1: 4x10k, Resistor_THT:R_Array_SIP5, symbol Device:R_Network04
Connections:
- net +5V: now also RN1.1 (common)
- net at J3.2 (Pin_2), U3.1 (B3): now also RN1.2 (R1)
- net at J3.6 (Pin_6), U3.11 (B1): now also RN1.4 (R3)
- net at J3.4 (Pin_4), U3.14 (B2): now also RN1.3 (R2)
- net at J3.8 (Pin_8), U3.9 (B0): now also RN1.5 (R4)
Changed lines of the file:
@@
 EESchema Schematic File Version 4
-LIBS:MEM-cache
 EELAYER 30 0
 EELAYER END
@@
 $EndComp
 Wire Wire Line
-	2400 3950 1600 3950
-Wire Wire Line
-	1500 4050 1800 4050
-Wire Wire Line
-	2400 4150 2000 4150
-Wire Wire Line
-	1500 4250 2200 4250
-Wire Wire Line
 	1000 3950 1000 4050
 Wire Wire Line
@@
 Connection ~ 3400 3950
 $Comp
-L Device:R R3
-U 1 1 5E8F1A02
-P 1600 3650
-F 0 "R3" V 1700 3750 50  0000 C CNN
-F 1 "10k" V 1700 3600 50  0000 C CNN
-F 2 "" V 1530 3650 50  0001 C CNN
-F 3 "~" H 1600 3650 50  0001 C CNN
-	1    1600 3650
-	1    0    0    -1
-$EndComp
-$Comp
-L Device:R R4
-U 1 1 5E8F954C
-P 1800 3650
-F 0 "R4" V 1900 3750 50  0000 C CNN
-F 1 "10k" V 1900 3600 50  0000 C CNN
-F 2 "" V 1730 3650 50  0001 C CNN
-F 3 "~" H 1800 3650 50  0001 C CNN
-	1    1800 3650
-	1    0    0    -1
-$EndComp
-$Comp
-L Device:R R5
-U 1 1 5E8FB1E6
-P 2000 3650
-F 0 "R5" V 2100 3750 50  0000 C CNN
-F 1 "10k" V 2100 3600 50  0000 C CNN
-F 2 "" V 1930 3650 50  0001 C CNN
-F 3 "~" H 2000 3650 50  0001 C CNN
-	1    2000 3650
-	1    0    0    -1
-$EndComp
-$Comp
-L Device:R R6
-U 1 1 5E8FCDB9
-P 2200 3650
-F 0 "R6" V 2300 3750 50  0000 C CNN
-F 1 "10k" V 2300 3600 50  0000 C CNN
-F 2 "" V 2130 3650 50  0001 C CNN
-F 3 "~" H 2200 3650 50  0001 C CNN
-	1    2200 3650
-	1    0    0    -1
-$EndComp
-Wire Wire Line
-	1600 3800 1600 3950
-Connection ~ 1600 3950
-Wire Wire Line
-	1600 3950 1500 3950
-Wire Wire Line
-	1800 3800 1800 4050
-Connection ~ 1800 4050
-Wire Wire Line
-	1800 4050 2400 4050
-Wire Wire Line
-	2000 3800 2000 4150
-Connection ~ 2000 4150
-Wire Wire Line
-	2000 4150 1500 4150
-Wire Wire Line
-	2200 3800 2200 4250
-Connection ~ 2200 4250
-Wire Wire Line
-	2200 4250 2400 4250
-Wire Wire Line
-	1600 3500 1600 3400
-Wire Wire Line
-	1600 3400 1800 3400
-Wire Wire Line
-	2200 3400 2200 3500
-Wire Wire Line
-	2000 3500 2000 3400
-Connection ~ 2000 3400
-Wire Wire Line
-	2000 3400 2200 3400
-Wire Wire Line
-	1800 3500 1800 3400
-Connection ~ 1800 3400
-$Comp
 L power:+5V #PWR019
 U 1 1 5E914060
-P 1800 3250
-F 0 "#PWR019" H 1800 3100 50  0001 C CNN
-F 1 "+5V" H 1815 3423 50  0000 C CNN
-F 2 "" H 1800 3250 50  0001 C CNN
-F 3 "" H 1800 3250 50  0001 C CNN
-	1    1800 3250
-	1    0    0    -1
-$EndComp
-Wire Wire Line
-	1800 3250 1800 3400
+P 1750 3300
+F 0 "#PWR019" H 1750 3150 50  0001 C CNN
+F 1 "+5V" H 1765 3473 50  0000 C CNN
+F 2 "" H 1750 3300 50  0001 C CNN
+F 3 "" H 1750 3300 50  0001 C CNN
+	1    1750 3300
+	1    0    0    -1
+$EndComp
 $Comp
 L power:GND #PWR05
@@
 NoConn ~ 3400 4550
 NoConn ~ 3400 4650
-Wire Wire Line
-	1800 3400 2000 3400
 $Comp
 L Connector_Generic:Conn_02x02_Odd_Even J4
@@
 Text Notes 7900 5900 0    50   ~ 0
 (ROM enabled)
+$Comp
+L Device:R_Network04 RN1
+U 1 1 60D326E0
+P 1950 3600
+F 0 "RN1" H 2138 3646 50  0000 L CNN
+F 1 "4x10k" H 2138 3555 50  0000 L CNN
+F 2 "Resistor_THT:R_Array_SIP5" V 2225 3600 50  0001 C CNN
+F 3 "http://www.vishay.com/docs/31509/csc.pdf" H 1950 3600 50  0001 C CNN
+	1    1950 3600
+	1    0    0    -1
+$EndComp
+Wire Wire Line
+	1500 3950 1750 3950
+Wire Wire Line
+	1500 4050 1850 4050
+Wire Wire Line
+	1500 4150 1950 4150
+Wire Wire Line
+	1500 4250 2050 4250
+Wire Wire Line
+	1750 3800 1750 3950
+Connection ~ 1750 3950
+Wire Wire Line
+	1750 3950 2400 3950
+Wire Wire Line
+	1850 3800 1850 4050
+Connection ~ 1850 4050
+Wire Wire Line
+	1850 4050 2400 4050
+Wire Wire Line
+	1950 3800 1950 4150
+Connection ~ 1950 4150
+Wire Wire Line
+	1950 4150 2400 4150
+Wire Wire Line
+	2050 3800 2050 4250
+Connection ~ 2050 4250
+Wire Wire Line
+	2050 4250 2400 4250
+Wire Wire Line
+	1750 3300 1750 3400
 $EndSCHEMATC

Commit message: home
Parts:
- removed C1: 10n, symbol Device:C
- removed Q1, Q2, Q3, Q4: BC547, Package_TO_SOT_THT:TO-92_Inline, symbol Transistor_BJT:BC547
- removed R10, R12, R14, R9: 10k, symbol Device:R
- removed U2: 74LS00, symbol 74xx:74LS00
- added C3, C4, C5, C6, C7, C8: 10nF, symbol Device:C
- added U2: 74LS04, symbol 74xx:74LS04
- added U5: SN74LS07N, symbol 74xx:SN74LS07N
- C2: value 10n -> 10nF
- R1, R2: value 470 -> 220
- R3: renamed from R11; value 470 -> 220
- R4: renamed from R13; value 470 -> 220
- renumbered C3 to C1, D2 to D1, D1 to D2, J3 to J1, J1 to J2, J2 to J3, J5 to J4, J4 to J5, R7 to R5, R8 to R6, U4 to U3, U3 to U4, U5 to U7
Connections:
- net +5V: now also C3.1, C4.1, C5.1, C6.1, C7.1, C8.1, U2.14 (VCC), U5.14 (VCC)
- net GND: now also C3.2, C4.2, C5.2, C6.2, C7.2, C8.2, U2.13, U2.7 (GND), U5.11, U5.13, U5.7 (GND)
- net iorq: now also U2.1
- net at J5.4 (Pin_4), R5.2, U7.1 (A15): now also U2.11
- net at J5.2 (Pin_2), R6.2, U7.27 (A14): now also U2.9
- net at J4.2 (Pin_2), J4.4 (Pin_4), J4.6 (Pin_6)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: now also U2.3
- net at U3.6 (~Q): now also U2.5
- net at R2.1: now also U5.4
- net at U4.3 (Ia=b): now also U2.2
- net at R4.1: now also U5.8
- net at R3.1: now also U5.6
- net at R1.1: now also U5.2
- new net: U2.4, U5.1
- new net: U2.6, U5.3
- new net: U2.8, U5.5
- new net: U2.10, U5.9
- no-connect marks 19 -> 22
Other:
- moved on the sheet: D1, D2, R1, R2, U1C, U3C

Commit message: home
Parts:
- removed R1, R2, R3, R4: 220, symbol Device:R
- added RN2: 4x220, Resistor_THT:R_Array_SIP5, symbol Device:R_Network04
- C1: footprint (none) -> Capacitor_THT:CP_Radial_D5.0mm_P2.50mm
- C2, C3, C4, C5, C6, C7, C8: footprint (none) -> Capacitor_THT:C_Disc_D3.8mm_W2.6mm_P2.50mm
- D1: renamed from D3; footprint (none) -> LED_THT:LED_D3.0mm
- D2: renamed from D4; footprint (none) -> LED_THT:LED_D3.0mm
- D3: renamed from D1; footprint (none) -> LED_THT:LED_D3.0mm
- D4: renamed from D2; footprint (none) -> LED_THT:LED_D3.0mm
- J1: footprint (none) -> Connector_PinHeader_2.54mm:PinHeader_2x04_P2.54mm_Vertical
- J2: footprint (none) -> Connector_PinHeader_2.54mm:PinHeader_2x05_P2.54mm_Vertical
- J3: footprint (none) -> Connector_PinHeader_2.54mm:PinHeader_2x20_P2.54mm_Vertical
- J4: footprint (none) -> Connector_PinSocket_2.54mm:PinSocket_2x03_P2.54mm_Vertical
- J5: footprint (none) -> Connector_PinHeader_2.54mm:PinHeader_2x02_P2.54mm_Vertical
- R1: renamed from R5; footprint (none) -> Resistor_THT:R_Axial_DIN0207_L6.3mm_D2.5mm_P10.16mm_Horizontal
- R2: renamed from R6; footprint (none) -> Resistor_THT:R_Axial_DIN0207_L6.3mm_D2.5mm_P10.16mm_Horizontal
- U1, U4: footprint (none) -> Package_DIP:DIP-16_W7.62mm_Socket_LongPads
- U2, U3, U5: footprint (none) -> Package_DIP:DIP-14_W7.62mm_Socket_LongPads
- U6: footprint (none) -> Package_DIP:DIP-32_W15.24mm_Socket_LongPads
- U7: footprint Package_DIP:DIP-28_W15.24mm -> Socket:DIP_Socket-28_W11.9_W12.7_W15.24_W17.78_W18.5_3M_228-1277-00-0602J
Connections:
- net +5V: now also RN2.1 (common); no longer D1.2 (A), D2.2 (A), D3.2 (A), D4.2 (A)
- net ram_bank: now reaches J4.2 (Pin_2), J4.4 (Pin_4), J4.6 (Pin_6), U2.3, U6.2 (A16)
- net at U5.4: now also D4.1 (K)
- net at D2.1 (K): now also U5.8
- net at D1.1 (K): now also U5.6
- net at D3.1 (K): now also U5.2
- new net: D4.2 (A), RN2.5 (R4)
- new net: D2.2 (A), RN2.3 (R2)
- new net: D1.2 (A), RN2.2 (R1)
- new net: D3.2 (A), RN2.4 (R3)
Other:
- note added: "ram\nbank"
- moved on the sheet: D1, D2, D3, D4, U2B, U2C, U2D, U2E, U2F, U5A, U5B, U5C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

Commit message: home
Parts:
- J4: footprint Connector_PinSocket_2.54mm:PinSocket_2x03_P2.54mm_Vertical -> Connector_PinHeader_2.54mm:PinHeader_2x03_P2.54mm_Vertical
Changed lines of the file:
@@
 F 0 "J4" H 5700 3167 50  0000 C CNN
 F 1 "RAM bank" H 5700 3076 50  0000 C CNN
-F 2 "Connector_PinSocket_2.54mm:PinSocket_2x03_P2.54mm_Vertical" H 5650 2850 50  0001 C CNN
+F 2 "Connector_PinHeader_2.54mm:PinHeader_2x03_P2.54mm_Vertical" H 5650 2850 50  0001 C CNN
 F 3 "~" H 5650 2850 50  0001 C CNN
 	1    5650 2850
