File: KiCAD files/TTY/TTY.sch (KiCad schematic (older format))
At the start: 44 parts, among them J1 Power Bus, J2 Signal Buss, J3 TTL/RS232, J4 Card addr, J5 TTL/RS232, J6 TTY1, J7 TTY0, J8 DB9, U1 74LS07, U2 74LS74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

Commit message: office
Parts:
- U3, U4: symbol preTTY-rescue:ATmega328P-PU-MCU_Microchip_ATmega -> MCU_Microchip_ATmega:ATmega328P-PU
Changed lines of the file:
@@
 EESchema Schematic File Version 4
-LIBS:TTY-cache
 EELAYER 30 0
 EELAYER END
@@
 RX0RS232
 $Comp
-L preTTY-rescue:ATmega328P-PU-MCU_Microchip_ATmega U3
+L MCU_Microchip_ATmega:ATmega328P-PU U3
 U 1 1 60FA7136
 P 2200 4900
@@
 Wire Wire Line
 	2100 3400 2200 3400
-Connection ~ 2200 3400
 $Comp
 L Device:C C10
@@
 $EndComp
 $Comp
-L preTTY-rescue:ATmega328P-PU-MCU_Microchip_ATmega U4
+L MCU_Microchip_ATmega:ATmega328P-PU U4
 U 1 1 6150E52C
 P 4400 4700
@@
 Wire Wire Line
 	4300 3200 4400 3200
-Connection ~ 4400 3200
 Connection ~ 3400 4000
 Wire Wire Line
