File: KiCAD files/TTY/TTY.kicad_pcb (KiCad board)
At the start: 2 copper layers, 99.7 x 69.9 mm, 44 parts, among them J1 Power Bus, J2 Signal Buss, J3 TTL/RS232, J4 Card addr, J5 TTL/RS232, J6 TTY1, J7 TTY0, J8 DB9, U1 74LS07, U2 74LS74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

Commit message: office updates
Other:
- net class Default removed
- net class Power removed
