File: KiCAD files/Backplane v2/Backplane v2.kicad_pcb (KiCad board)
At the start: 2 copper layers, 233.7 x 69.8 mm, 30 parts, among them J1 Conn_02x05_Odd_Even, J10 Conn_02x20_Odd_Even, J2 Conn_02x20_Odd_Even, J3 Conn_02x05_Odd_Even, J4 Conn_02x20_Odd_Even, J5 Conn_02x05_Odd_Even, J6 Conn_02x20_Odd_Even, J7 Conn_02x05_Odd_Even, J8 Conn_02x20_Odd_Even, J9 Conn_02x05_Odd_Even

Commit message: office
Parts:
- moved J10 123.5 mm to (177.8, 72.4)
- moved J5 123.5 mm to (146.1, 57.1)
- moved J6 123.5 mm to (146.1, 72.4)
- moved J9 123.5 mm to (177.8, 57.1)
- moved J1 123.5 mm to (34.3, 57.1)
- moved J1 123.5 mm to (194.3, 57.1)
- moved J1 123.5 mm to (114.3, 57.1)
- moved J10 123.5 mm to (97.8, 72.4)
- moved J10 123.5 mm to (257.8, 72.4)
- moved J2 123.5 mm to (34.3, 72.4)
- moved J2 123.5 mm to (194.3, 72.4)
- moved J2 123.5 mm to (114.3, 72.4)
- moved J3 123.5 mm to (39.4, 57.1)
- moved J3 123.5 mm to (199.4, 57.1)
- moved J3 123.5 mm to (119.4, 57.1)
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Routing:
- added copper zone on B.Cu, net /gnd

Commit message: office
Parts:
- removed the J1 at (34.3, 57.1)
- removed the J1 at (194.3, 57.1)
- removed the J10 at (97.8, 72.4)
- removed the J10 at (257.8, 72.4)
- removed the J2 at (34.3, 72.4)
- removed the J2 at (194.3, 72.4)
- removed the J3 at (39.4, 57.1)
- removed the J3 at (199.4, 57.1)
- removed the J4 at (39.4, 72.4)
- removed the J4 at (199.4, 72.4)
- removed the J5 at (66.0, 57.1)
- removed the J5 at (226.1, 57.1)
- removed the J6 at (66.0, 72.4)
- removed the J6 at (226.1, 72.4)
- removed the J7 at (92.7, 57.1)
- removed the J7 at (252.7, 57.1)
- removed the J8 at (92.7, 72.4)
- removed the J8 at (252.7, 72.4)
- removed the J9 at (97.8, 57.1)
- removed the J9 at (257.8, 57.1)
Routing:
- net /gnd: vias 6 -> 2
Other:
- board size 233.7 x 69.8 mm -> 73.7 x 69.8 mm

Commit message: office
Routing:
- net /gnd: vias 2 -> 4
Other:
- board size 73.7 x 69.8 mm -> 72.4 x 85.1 mm
Changed lines of the file:
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@@
     (thickness 1.6)
     (drawings 4)
-    (tracks 2)
+    (tracks 4)
     (zones 0)
     (modules 10)
@@
     )
   )
-  (gr_line (start 111.125 123.825) (end 184.785 123.825) (layer Edge.Cuts) (width 0.05))
-  (gr_line (start 184.785 53.975) (end 184.785 123.825) (layer Edge.Cuts) (width 0.05))
-  (gr_line (start 111.125 53.975) (end 111.125 123.825) (layer Edge.Cuts) (width 0.05))
-  (gr_line (start 111.125 53.975) (end 184.785 53.975) (layer Edge.Cuts) (width 0.05))
-  (via (at 159.385 56.515) (size 5.08) (drill 3.048) (layers F.Cu B.Cu) (net 1))
-  (via (at 135.89 121.285) (size 5.08) (drill 3.048) (layers F.Cu B.Cu) (net 1))
+  (gr_line (start 111.125 131.445) (end 183.515 131.445) (layer Edge.Cuts) (width 0.05))
+  (gr_line (start 183.515 46.355) (end 183.515 131.445) (layer Edge.Cuts) (width 0.05))
+  (gr_line (start 111.125 46.355) (end 111.125 131.445) (layer Edge.Cuts) (width 0.05))
+  (gr_line (start 111.125 46.355) (end 183.515 46.355) (layer Edge.Cuts) (width 0.05))
+  (via (at 120.65 50.8) (size 5.08) (drill 3.048) (layers F.Cu B.Cu) (net 1))
+  (via (at 120.65 127) (size 5.08) (drill 3.048) (layers F.Cu B.Cu) (net 1))
+  (via (at 173.99 127) (size 5.08) (drill 3.048) (layers F.Cu B.Cu) (net 1))
+  (via (at 173.99 50.8) (size 5.08) (drill 3.048) (layers F.Cu B.Cu) (net 1))
   (zone (net 1) (net_name /gnd) (layer B.Cu) (hatch edge 0.508)
     (connect_pads (clearance 0.508))

Commit message: home
Parts:
- added J11: Conn_02x05_Odd_Even, Connector_PinHeader_2.54mm:PinHeader_2x05_P2.54mm_Vertical, F.Cu at (200.7, 63.5)
- added J12: Conn_02x20_Odd_Even, Connector_PinHeader_2.54mm:PinHeader_2x20_P2.54mm_Vertical, F.Cu at (200.7, 78.7)
- added J13: Conn_02x05_Odd_Even, Connector_PinHeader_2.54mm:PinHeader_2x05_P2.54mm_Vertical, F.Cu at (227.3, 63.5)
- added J14: Conn_02x20_Odd_Even, Connector_PinHeader_2.54mm:PinHeader_2x20_P2.54mm_Vertical, F.Cu at (227.3, 78.7)
- added J15: Conn_02x05_Odd_Even, Connector_PinHeader_2.54mm:PinHeader_2x05_P2.54mm_Vertical, F.Cu at (254.0, 63.5)
- added J16: Conn_02x20_Odd_Even, Connector_PinHeader_2.54mm:PinHeader_2x20_P2.54mm_Vertical, F.Cu at (254.0, 78.7)
- moved J1 47.4 mm to (67.3, 63.5)
- moved J2 47.4 mm to (67.3, 78.7)
- moved J5 26.2 mm to (120.7, 63.5)
- moved J7 26.2 mm to (147.3, 63.5)
- moved J6 26.2 mm to (120.7, 78.7)
- moved J8 26.2 mm to (147.3, 78.7)
- moved J3 26.2 mm to (94.0, 63.5)
- moved J4 26.2 mm to (94.0, 78.7)
- moved J9 7.41 mm to (174.0, 63.5)
- moved J10 7.41 mm to (174.0, 78.7)
Connections:
- J10 pad 1: /a01 -> /a00
- J10 pad 10: /a08 -> /a09
- J10 pad 11: /a11 -> /a10
- J10 pad 12: /a10 -> /a11
- J10 pad 13: /a13 -> /a12
- J10 pad 14: /a12 -> /a13
- J10 pad 15: /a15 -> /a14
- J10 pad 16: /a14 -> /a15
- J10 pad 17: /d01 -> /d00
- J10 pad 18: /d00 -> /d01
- J10 pad 19: /d03 -> /d02
- J10 pad 2: /a00 -> /a01
- J10 pad 20: /d02 -> /d03
- J10 pad 21: /d05 -> /d04
- J10 pad 22: /d04 -> /d05
- J10 pad 23: /d07 -> /d06
- J10 pad 24: /d06 -> /d07
- J10 pad 25: /wr -> /mreq
- J10 pad 26: /mreq -> /wr
- J10 pad 27: /rd -> /iorq
- J10 pad 28: /iorq -> /rd
- J10 pad 29: /busack -> /busrq
- J10 pad 3: /a03 -> /a02
- J10 pad 30: /busrq -> /busack
- J10 pad 31: /halt -> /wait
- J10 pad 32: /wait -> /halt
- J10 pad 33: /int -> /nmi
- J10 pad 34: /nmi -> /int
- J10 pad 35: /s1 -> /s0
- J10 pad 36: /s0 -> /s1
- J10 pad 37: /m1 -> /s2
- J10 pad 38: /s2 -> /m1
- J10 pad 39: /clk -> /reset
- J10 pad 4: /a02 -> /a03
- J10 pad 40: /reset -> /clk
- J10 pad 5: /a05 -> /a04
- J10 pad 6: /a04 -> /a05
- J10 pad 7: /a07 -> /a06
- J10 pad 8: /a06 -> /a07
- J10 pad 9: /a09 -> /a08
Routing:
- net /gnd: vias 4 -> 0
Other:
- board outline removed

Commit message: home
Parts:
- removed J11, J13, J15: Conn_02x05_Odd_Even, Connector_PinHeader_2.54mm:PinHeader_2x05_P2.54mm_Vertical
- removed J12, J14, J16: Conn_02x20_Odd_Even, Connector_PinHeader_2.54mm:PinHeader_2x20_P2.54mm_Vertical
- moved J10 20.3 mm to (153.7, 78.7)
- moved J9 20.3 mm to (153.7, 63.5)
- moved J1 20.3 mm to (87.6, 63.5)
- moved J2 20.3 mm to (87.6, 78.7)
Connections:
- J10 pad 1: /a00 -> /a01
- J10 pad 10: /a09 -> /a08
- J10 pad 11: /a10 -> /a11
- J10 pad 12: /a11 -> /a10
- J10 pad 13: /a12 -> /a13
- J10 pad 14: /a13 -> /a12
- J10 pad 15: /a14 -> /a15
- J10 pad 16: /a15 -> /a14
- J10 pad 17: /d00 -> /d01
- J10 pad 18: /d01 -> /d00
- J10 pad 19: /d02 -> /d03
- J10 pad 2: /a01 -> /a00
- J10 pad 20: /d03 -> /d02
- J10 pad 21: /d04 -> /d05
- J10 pad 22: /d05 -> /d04
- J10 pad 23: /d06 -> /d07
- J10 pad 24: /d07 -> /d06
- J10 pad 25: /mreq -> /wr
- J10 pad 26: /wr -> /mreq
- J10 pad 27: /iorq -> /rd
- J10 pad 28: /rd -> /iorq
- J10 pad 29: /busrq -> /busack
- J10 pad 3: /a02 -> /a03
- J10 pad 30: /busack -> /busrq
- J10 pad 31: /wait -> /halt
- J10 pad 32: /halt -> /wait
- J10 pad 33: /nmi -> /int
- J10 pad 34: /int -> /nmi
- J10 pad 35: /s0 -> /s1
- J10 pad 36: /s1 -> /s0
- J10 pad 37: /s2 -> /m1
- J10 pad 38: /m1 -> /s2
- J10 pad 39: /reset -> /clk
- J10 pad 4: /a03 -> /a02
- J10 pad 40: /clk -> /reset
- J10 pad 5: /a04 -> /a05
- J10 pad 6: /a05 -> /a04
- J10 pad 7: /a06 -> /a07
- J10 pad 8: /a07 -> /a06
- J10 pad 9: /a08 -> /a09
Routing:
- net /gnd: track 0.00 -> 149.4 mm
- net /a00: track 0.00 -> 73.1 mm
- net /a04: track 0.00 -> 72.6 mm
- net /d04: track 0.00 -> 72.6 mm
- net /a12: track 0.00 -> 72.6 mm
- net /busrq: track 0.00 -> 72.6 mm
- net /s2: track 0.00 -> 72.5 mm
- net /nmi: track 0.00 -> 72.5 mm
- net /d02: track 0.00 -> 72.5 mm
- net /a14: track 0.00 -> 72.5 mm
- net /reset: track 0.00 -> 72.5 mm
- net /a10: track 0.00 -> 72.5 mm
- net /a08: track 0.00 -> 72.5 mm
- net /wait: track 0.00 -> 72.5 mm
- net /s0: track 0.00 -> 72.5 mm
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Other:
- board outline added: 77.5 x 99.1 mm
- net class Power added: clearance 0.4064, trace_width 0.508, via_dia 0.8, via_drill 0.4
- board text added: "Back Side"
- board text added: "Bottom"
- board text added: "Component Side"
- board text added: "December/2021 by Kaltchuk"
- board text added: "Slot 1"
- board text added: "Slot 3"
- board text added: "Solt 2"
- board text added: "Z80 Modular Computer Backplane v2"

Commit message: office
Parts:
- added J1: Conn_02x05_Odd_Even, Connector_PinHeader_2.54mm:PinHeader_2x05_P2.54mm_Vertical, F.Cu at (170.2, 63.5)
- added J10: Conn_02x20_Odd_Even, Connector_PinHeader_2.54mm:PinHeader_2x20_P2.54mm_Vertical, F.Cu at (236.2, 78.7)
- added J2: Conn_02x20_Odd_Even, Connector_PinHeader_2.54mm:PinHeader_2x20_P2.54mm_Vertical, F.Cu at (170.2, 78.7)
- added J3: Conn_02x05_Odd_Even, Connector_PinHeader_2.54mm:PinHeader_2x05_P2.54mm_Vertical, F.Cu at (176.5, 63.5)
- added J4: Conn_02x20_Odd_Even, Connector_PinHeader_2.54mm:PinHeader_2x20_P2.54mm_Vertical, F.Cu at (176.5, 78.7)
- added J5: Conn_02x05_Odd_Even, Connector_PinHeader_2.54mm:PinHeader_2x05_P2.54mm_Vertical, F.Cu at (203.2, 63.5)
- added J6: Conn_02x20_Odd_Even, Connector_PinHeader_2.54mm:PinHeader_2x20_P2.54mm_Vertical, F.Cu at (203.2, 78.7)
- added J7: Conn_02x05_Odd_Even, Connector_PinHeader_2.54mm:PinHeader_2x05_P2.54mm_Vertical, F.Cu at (229.9, 63.5)
- added J8: Conn_02x20_Odd_Even, Connector_PinHeader_2.54mm:PinHeader_2x20_P2.54mm_Vertical, F.Cu at (229.9, 78.7)
- added J9: Conn_02x05_Odd_Even, Connector_PinHeader_2.54mm:PinHeader_2x05_P2.54mm_Vertical, F.Cu at (236.2, 63.5)
Routing:
- net /gnd: track 149.4 -> 298.7 mm
- net /a00: track 73.1 -> 146.2 mm
- net /a04: track 72.6 -> 145.3 mm
- net /d04: track 72.6 -> 145.3 mm
- net /a12: track 72.6 -> 145.3 mm
- net /busrq: track 72.6 -> 145.1 mm
- net /reset: track 72.5 -> 144.9 mm
- net /a10: track 72.5 -> 144.9 mm
- net /s2: track 72.5 -> 144.9 mm
- net /nmi: track 72.5 -> 144.9 mm
- net /d02: track 72.5 -> 144.9 mm
- net /a14: track 72.5 -> 144.9 mm
- net /wait: track 72.5 -> 144.9 mm
- net /s0: track 72.5 -> 144.9 mm
- net /mreq: track 72.5 -> 144.9 mm
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Other:
- board size 77.5 x 99.1 mm -> 160 x 99.1 mm

Commit message: home
Parts:
- removed the J1 at (170.2, 63.5)
- removed the J10 at (236.2, 78.7)
- removed the J2 at (170.2, 78.7)
- removed the J3 at (176.5, 63.5)
- removed the J4 at (176.5, 78.7)
- removed the J5 at (203.2, 63.5)
- removed the J6 at (203.2, 78.7)
- removed the J7 at (229.9, 63.5)
- removed the J8 at (229.9, 78.7)
- removed the J9 at (236.2, 63.5)
- removed the J9 at (153.7, 63.5)
- added J9: Conn_02x05_Odd_Even, Connector_PinHeader_2.54mm:PinHeader_2x05_P2.54mm_Vertical, F.Cu at (152.4, 63.5)
- moved J1 1.27 mm to (88.9, 63.5)
- moved J2 1.27 mm to (88.9, 78.7)
- moved J10 1.27 mm to (152.4, 78.7)
Routing:
- net /gnd: track 298.7 -> 144.3 mm
- net /a00: track 146.2 -> 70.8 mm
- net /a04: track 145.3 -> 69.9 mm
- net /d04: track 145.3 -> 69.9 mm
- net /a12: track 145.3 -> 69.9 mm
- net /busrq: track 145.1 -> 70.0 mm
- net /reset: track 144.9 -> 69.9 mm
- net /a10: track 144.9 -> 69.9 mm
- net /s2: track 144.9 -> 69.9 mm
- net /nmi: track 144.9 -> 69.9 mm
- net /d02: track 144.9 -> 69.9 mm
- net /a14: track 144.9 -> 69.9 mm
- net /wait: track 144.9 -> 69.9 mm
- net /s0: track 144.9 -> 69.9 mm
- net /mreq: track 144.9 -> 69.9 mm
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Other:
- board size 160 x 99.1 mm -> 77.5 x 99.1 mm

Commit message: pcb updates
Other:
- net class Default removed
- net class Power removed
