File: KiCAD files/Front Panel Template/Front Panel Template.kicad_pcb (KiCad board)
At the start: 2 copper layers, 120 x 80 mm, 0 parts

Commit message: home
Other:
- board size 120 x 80 mm -> 151.8 x 80.6 mm
- board text added: "TTY"
Changed lines of the file:
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@@
-(kicad_pcb (version 20171130) (host pcbnew "(5.1.6)-1")
+(kicad_pcb (version 20171130) (host pcbnew "(5.1.4)-1")
   (general
     (thickness 1.6)
-    (drawings 57)
+    (drawings 71)
     (tracks 0)
     (zones 0)
@@
     (uvia_drill 0.1)
   )
-  (gr_text "RAM\nbank" (at 105.41 66.675) (layer F.SilkS)
-    (effects (font (size 2.0828 2.0828) (thickness 0.3302)) (justify left))
+  (gr_text ADDR (at 163.195 103.505) (layer F.SilkS)
+    (effects (font (size 2.0828 2.0828) (thickness 0.3302)))
   )
-  (gr_text CARD (at 42.545 31.75) (layer F.SilkS)
+  (gr_text TTY (at 169.545 31.115) (layer F.SilkS)
     (effects (font (size 5.334 5.334) (thickness 0.7874)))
   )
-  (gr_text "ROM\nblock" (at 105.41 47.625) (layer F.SilkS)
-    (effects (font (size 2.0828 2.0828) (thickness 0.3302)) (justify left))
-  )
-  (gr_text ADDR (at 67.945 104.14) (layer F.SilkS)
-    (effects (font (size 2.794 2.794) (thickness 0.4318)))
-  )
-  (gr_text MEM (at 106.045 31.75) (layer F.SilkS)
-    (effects (font (size 5.334 5.334) (thickness 0.7874)))
-  )
-  (gr_text FLASH (at 73.66 31.75) (layer F.SilkS)
-    (effects (font (size 5.334 5.334) (thickness 0.7874)))
-  )
-  (gr_text ADDR (at 99.695 104.14) (layer F.SilkS)
-    (effects (font (size 2.794 2.794) (thickness 0.4318)))
-  )
-  (gr_text ADDR (at 36.195 104.14) (layer F.SilkS)
-    (effects (font (size 2.794 2.794) (thickness 0.4318)))
-  )
-  (gr_text "ROM\nactive" (at 105.41 57.15) (layer F.SilkS)
-    (effects (font (size 2.0828 2.0828) (thickness 0.3302)) (justify left))
-  )
+  (gr_line (start 171.45 40.005) (end 176.53 40.005) (layer F.CrtYd) (width 0.05))
+  (gr_line (start 156.845 106.68) (end 181.61 106.68) (layer Edge.Cuts) (width 0.05))
+  (gr_line (start 176.53 26.67) (end 176.53 106.68) (layer F.CrtYd) (width 0.0254))
+  (gr_line (start 171.45 99.695) (end 176.53 99.695) (layer F.CrtYd) (width 0.05))
+  (gr_circle (center 171.45 36.83) (end 168.275 36.83) (layer F.CrtYd) (width 0.05))
+  (gr_circle (center 171.45 36.83) (end 172.974 36.83) (layer Edge.Cuts) (width 0.05))
+  (gr_circle (center 171.45 96.52) (end 172.974 96.52) (layer Edge.Cuts) (width 0.15))
+  (gr_line (start 156.845 26.67) (end 181.61 26.67) (layer Edge.Cuts) (width 0.05))
+  (gr_line (start 156.845 26.67) (end 156.845 106.68) (layer Edge.Cuts) (width 0.05))
+  (gr_circle (center 171.45 96.52) (end 168.275 96.52) (layer F.CrtYd) (width 0.05))
+  (gr_line (start 181.61 106.68) (end 181.61 26.67) (layer Edge.Cuts) (width 0.05))
+  (gr_line (start 171.45 33.655) (end 176.53 33.655) (layer F.CrtYd) (width 0.05))
+  (gr_line (start 171.45 93.345) (end 176.53 93.345) (layer F.CrtYd) (width 0.05))
+  (gr_line (start 72.39 94.615) (end 72.39 40.64) (layer Edge.Cuts) (width 0.05))
+  (gr_line (start 61.595 27.305) (end 86.36 27.305) (layer Edge.Cuts) (width 0.05))
+  (gr_line (start 44.45 93.98) (end 49.53 93.98) (layer F.CrtYd) (width 0.05))
   (gr_circle (center 100.965 66.04) (end 102.489 66.04) (layer Edge.Cuts) (width 0.05))
   (gr_circle (center 100.965 56.515) (end 102.489 56.515) (layer Edge.Cuts) (width 0.05))
   (gr_circle (center 100.965 46.99) (end 102.489 46.99) (layer Edge.Cuts) (width 0.05))
-  (gr_line (start 73.66 94.615) (end 73.66 40.64) (layer Edge.Cuts) (width 0.05))
-  (gr_line (start 61.595 27.305) (end 86.36 27.305) (layer Edge.Cuts) (width 0.05))
-  (gr_line (start 44.45 93.98) (end 49.53 93.98) (layer F.CrtYd) (width 0.05))
   (gr_line (start 61.595 27.305) (end 61.595 107.315) (layer Edge.Cuts) (width 0.05))
   (gr_line (start 44.45 34.29) (end 49.53 34.29) (layer F.CrtYd) (width 0.05))
-  (gr_line (start 73.66 40.64) (end 81.28 40.64) (layer Edge.Cuts) (width 0.05))
+  (gr_line (start 72.39 40.64) (end 81.28 40.64) (layer Edge.Cuts) (width 0.05))
   (gr_line (start 93.345 107.315) (end 118.11 107.315) (layer Edge.Cuts) (width 0.05))
   (gr_line (start 54.61 107.315) (end 54.61 27.305) (layer Edge.Cuts) (width 0.05))
   (gr_circle (center 96.52 46.99) (end 98.044 46.99) (layer Edge.Cuts) (width 0.05))
   (gr_line (start 81.28 40.64) (end 81.28 94.615) (layer Edge.Cuts) (width 0.05))
+  (gr_circle (center 44.45 97.155) (end 41.275 97.155) (layer F.CrtYd) (width 0.05))
   (gr_line (start 29.845 27.305) (end 29.845 107.315) (layer Edge.Cuts) (width 0.05))
   (gr_line (start 29.845 27.305) (end 54.61 27.305) (layer Edge.Cuts) (width 0.05))
-  (gr_circle (center 44.45 97.155) (end 41.275 97.155) (layer F.CrtYd) (width 0.05))
   (gr_line (start 61.595 107.315) (end 86.36 107.315) (layer Edge.Cuts) (width 0.05))
   (gr_line (start 93.345 27.305) (end 93.345 107.315) (layer Edge.Cuts) (width 0.05))
@@
   (gr_circle (center 76.2 37.465) (end 77.724 37.465) (layer Edge.Cuts) (width 0.05))
   (gr_circle (center 76.2 97.155) (end 77.724 97.155) (layer Edge.Cuts) (width 0.15))
-  (gr_line (start 76.2 40.64) (end 81.28 40.64) (layer F.CrtYd) (width 0.05))
-  (gr_line (start 81.28 94.615) (end 73.66 94.615) (layer Edge.Cuts) (width 0.05))
-  (gr_text "Reset\n" (at 136.525 56.515) (layer F.SilkS)
+  (gr_line (start 81.28 94.615) (end 72.39 94.615) (layer Edge.Cuts) (width 0.05))
+  (gr_text "RAM\nbank" (at 105.41 66.675) (layer F.SilkS)
     (effects (font (size 2.0828 2.0828) (thickness 0.3302)) (justify left))
   )
-  (gr_circle (center 132.08 51.054) (end 135.636 51.054) (layer Edge.Cuts) (width 0.05))
-  (gr_circle (center 132.08 65.405) (end 133.604 65.405) (layer Edge.Cuts) (width 0.05))
-  (gr_circle (center 132.08 74.93) (end 133.604 74.93) (layer Edge.Cuts) (width 0.05))
-  (gr_text "Power\n" (at 136.525 65.405) (layer F.SilkS)
+  (gr_text CARD (at 42.545 31.75) (layer F.SilkS)
+    (effects (font (size 5.334 5.334) (thickness 0.7874)))
+  )
+  (gr_text "ROM\nblock" (at 105.41 47.625) (layer F.SilkS)
     (effects (font (size 2.0828 2.0828) (thickness 0.3302)) (justify left))
   )
-  (gr_text Halted (at 136.525 74.93) (layer F.SilkS)
+  (gr_text ADDR (at 67.945 104.14) (layer F.SilkS)
+    (effects (font (size 2.0828 2.0828) (thickness 0.3302)))
+  )
+  (gr_text MEM (at 106.045 31.75) (layer F.SilkS)
+    (effects (font (size 5.334 5.334) (thickness 0.7874)))
+  )
+  (gr_text FLASH (at 73.66 31.75) (layer F.SilkS)
+    (effects (font (size 5.334 5.334) (thickness 0.7874)))
+  )
+  (gr_text ADDR (at 99.695 104.14) (layer F.SilkS)
+    (effects (font (size 2.0828 2.0828) (thickness 0.3302)))
+  )
+  (gr_text ADDR (at 36.195 104.14) (layer F.SilkS)
+    (effects (font (size 2.0828 2.0828) (thickness 0.3302)))
+  )
+  (gr_text "ROM\nactive" (at 105.41 57.15) (layer F.SilkS)
+    (effects (font (size 2.0828 2.0828) (thickness 0.3302)) (justify left))
+  )
+  (gr_text "Reset\n" (at 136.525 90.17) (layer F.SilkS)
+    (effects (font (size 2.0828 2.0828) (thickness 0.3302)) (justify left))
+  )
+  (gr_circle (center 132.08 84.709) (end 135.636 84.709) (layer Edge.Cuts) (width 0.05))
+  (gr_circle (center 132.08 56.515) (end 133.604 56.515) (layer Edge.Cuts) (width 0.05))
+  (gr_circle (center 132.08 66.04) (end 133.604 66.04) (layer Edge.Cuts) (width 0.05))
+  (gr_text "Power\n" (at 136.525 56.515) (layer F.SilkS)
+    (effects (font (size 2.0828 2.0828) (thickness 0.3302)) (justify left))
+  )
+  (gr_text Halted (at 136.525 66.04) (layer F.SilkS)
     (effects (font (size 2.0828 2.0828) (thickness 0.3302)) (justify left))
   )
@@
   (gr_line (start 149.86 107.315) (end 149.86 27.305) (layer Edge.Cuts) (width 0.05))
   (gr_text ADDR (at 131.445 104.14) (layer F.SilkS)
-    (effects (font (size 2.794 2.794) (thickness 0.4318)))
+    (effects (font (size 2.0828 2.0828) (thickness 0.3302)))
   )
   (gr_text CPU (at 137.795 31.75) (layer F.SilkS)

Commit message: home
Other:
- board size 151.8 x 80.6 mm -> 151.8 x 80 mm
Changed lines of the file:
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@@
     (uvia_drill 0.1)
   )
-  (gr_text ADDR (at 163.195 103.505) (layer F.SilkS)
+  (gr_text ADDR (at 163.195 104.14) (layer F.SilkS)
     (effects (font (size 2.0828 2.0828) (thickness 0.3302)))
   )
-  (gr_text TTY (at 169.545 31.115) (layer F.SilkS)
+  (gr_text TTY (at 169.545 31.75) (layer F.SilkS)
     (effects (font (size 5.334 5.334) (thickness 0.7874)))
   )
-  (gr_line (start 171.45 40.005) (end 176.53 40.005) (layer F.CrtYd) (width 0.05))
-  (gr_line (start 156.845 106.68) (end 181.61 106.68) (layer Edge.Cuts) (width 0.05))
-  (gr_line (start 176.53 26.67) (end 176.53 106.68) (layer F.CrtYd) (width 0.0254))
-  (gr_line (start 171.45 99.695) (end 176.53 99.695) (layer F.CrtYd) (width 0.05))
-  (gr_circle (center 171.45 36.83) (end 168.275 36.83) (layer F.CrtYd) (width 0.05))
-  (gr_circle (center 171.45 36.83) (end 172.974 36.83) (layer Edge.Cuts) (width 0.05))
-  (gr_circle (center 171.45 96.52) (end 172.974 96.52) (layer Edge.Cuts) (width 0.15))
-  (gr_line (start 156.845 26.67) (end 181.61 26.67) (layer Edge.Cuts) (width 0.05))
-  (gr_line (start 156.845 26.67) (end 156.845 106.68) (layer Edge.Cuts) (width 0.05))
-  (gr_circle (center 171.45 96.52) (end 168.275 96.52) (layer F.CrtYd) (width 0.05))
-  (gr_line (start 181.61 106.68) (end 181.61 26.67) (layer Edge.Cuts) (width 0.05))
-  (gr_line (start 171.45 33.655) (end 176.53 33.655) (layer F.CrtYd) (width 0.05))
-  (gr_line (start 171.45 93.345) (end 176.53 93.345) (layer F.CrtYd) (width 0.05))
-  (gr_line (start 72.39 94.615) (end 72.39 40.64) (layer Edge.Cuts) (width 0.05))
+  (gr_line (start 171.45 40.64) (end 176.53 40.64) (layer F.CrtYd) (width 0.05))
+  (gr_line (start 156.845 107.315) (end 181.61 107.315) (layer Edge.Cuts) (width 0.05))
+  (gr_line (start 176.53 27.305) (end 176.53 107.315) (layer F.CrtYd) (width 0.0254))
+  (gr_line (start 171.45 100.33) (end 176.53 100.33) (layer F.CrtYd) (width 0.05))
+  (gr_circle (center 171.45 37.465) (end 168.275 37.465) (layer F.CrtYd) (width 0.05))
+  (gr_circle (center 171.45 37.465) (end 172.974 37.465) (layer Edge.Cuts) (width 0.05))
+  (gr_circle (center 171.45 97.155) (end 172.974 97.155) (layer Edge.Cuts) (width 0.15))
+  (gr_line (start 156.845 27.305) (end 181.61 27.305) (layer Edge.Cuts) (width 0.05))
+  (gr_line (start 156.845 27.305) (end 156.845 107.315) (layer Edge.Cuts) (width 0.05))
+  (gr_circle (center 171.45 97.155) (end 168.275 97.155) (layer F.CrtYd) (width 0.05))
+  (gr_line (start 181.61 107.315) (end 181.61 27.305) (layer Edge.Cuts) (width 0.05))
+  (gr_line (start 171.45 34.29) (end 176.53 34.29) (layer F.CrtYd) (width 0.05))
+  (gr_line (start 171.45 93.98) (end 176.53 93.98) (layer F.CrtYd) (width 0.05))
+  (gr_line (start 72.39 93.98) (end 72.39 40.64) (layer Edge.Cuts) (width 0.05))
   (gr_line (start 61.595 27.305) (end 86.36 27.305) (layer Edge.Cuts) (width 0.05))
   (gr_line (start 44.45 93.98) (end 49.53 93.98) (layer F.CrtYd) (width 0.05))
@@
   (gr_line (start 54.61 107.315) (end 54.61 27.305) (layer Edge.Cuts) (width 0.05))
   (gr_circle (center 96.52 46.99) (end 98.044 46.99) (layer Edge.Cuts) (width 0.05))
-  (gr_line (start 81.28 40.64) (end 81.28 94.615) (layer Edge.Cuts) (width 0.05))
+  (gr_line (start 81.28 40.64) (end 81.28 93.98) (layer Edge.Cuts) (width 0.05))
   (gr_circle (center 44.45 97.155) (end 41.275 97.155) (layer F.CrtYd) (width 0.05))
   (gr_line (start 29.845 27.305) (end 29.845 107.315) (layer Edge.Cuts) (width 0.05))
@@
   (gr_circle (center 76.2 37.465) (end 77.724 37.465) (layer Edge.Cuts) (width 0.05))
   (gr_circle (center 76.2 97.155) (end 77.724 97.155) (layer Edge.Cuts) (width 0.15))
-  (gr_line (start 81.28 94.615) (end 72.39 94.615) (layer Edge.Cuts) (width 0.05))
+  (gr_line (start 81.28 93.98) (end 72.39 93.98) (layer Edge.Cuts) (width 0.05))
   (gr_text "RAM\nbank" (at 105.41 66.675) (layer F.SilkS)
     (effects (font (size 2.0828 2.0828) (thickness 0.3302)) (justify left))

Commit message: office
Other:
- outline, holes or cut-outs redrawn
- board text added: "CPU halted"
- board text added: "RX"
- board text added: "TTY 0"
- board text added: "TTY 1"
- board text added: "TX"
- board text removed: "Halted"
Changed lines of the file:
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@@
-(kicad_pcb (version 20171130) (host pcbnew "(5.1.4)-1")
+(kicad_pcb (version 20171130) (host pcbnew "(5.1.6)-1")
   (general
     (thickness 1.6)
-    (drawings 71)
+    (drawings 87)
     (tracks 0)
     (zones 0)
@@
     (uvia_drill 0.1)
   )
+  (gr_poly (pts (xy 51.435 106.045) (xy 43.18 106.045) (xy 43.18 101.6) (xy 51.435 101.6)) (layer F.SilkS) (width 0.1))
+  (gr_poly (pts (xy 83.185 106.045) (xy 74.93 106.045) (xy 74.93 101.6) (xy 83.185 101.6)) (layer F.SilkS) (width 0.1))
+  (gr_poly (pts (xy 114.935 106.045) (xy 106.68 106.045) (xy 106.68 101.6) (xy 114.935 101.6)) (layer F.SilkS) (width 0.1))
+  (gr_poly (pts (xy 146.685 106.045) (xy 138.43 106.045) (xy 138.43 101.6) (xy 146.685 101.6)) (layer F.SilkS) (width 0.1))
+  (gr_poly (pts (xy 178.435 106.045) (xy 170.18 106.045) (xy 170.18 101.6) (xy 178.435 101.6)) (layer F.SilkS) (width 0.1))
+  (gr_text "TTY 1" (at 179.07 92.075 90) (layer F.SilkS)
+    (effects (font (size 2.0828 2.0828) (thickness 0.3302)) (justify left))
+  )
+  (gr_text "TTY 0" (at 179.07 62.865 90) (layer F.SilkS)
+    (effects (font (size 2.0828 2.0828) (thickness 0.3302)) (justify left))
+  )
+  (gr_line (start 176.53 82.55) (end 181.61 82.55) (layer F.SilkS) (width 0.3302))
+  (gr_text TX (at 161.29 85.725) (layer F.SilkS)
+    (effects (font (size 2.0828 2.0828) (thickness 0.3302)) (justify left))
+  )
+  (gr_text RX (at 161.29 90.17) (layer F.SilkS)
+    (effects (font (size 2.0828 2.0828) (thickness 0.3302)) (justify left))
+  )
+  (gr_text TX (at 161.29 75.565) (layer F.SilkS)
+    (effects (font (size 2.0828 2.0828) (thickness 0.3302)) (justify left))
+  )
+  (gr_text RX (at 161.29 80.01) (layer F.SilkS)
+    (effects (font (size 2.0828 2.0828) (thickness 0.3302)) (justify left))
+  )
+  (gr_circle (center 159.385 85.725) (end 159.385 84.201) (layer Edge.Cuts) (width 0.05))
+  (gr_circle (center 159.385 90.17) (end 159.385 88.646) (layer Edge.Cuts) (width 0.05))
+  (gr_circle (center 159.385 80.01) (end 159.385 78.486) (layer Edge.Cuts) (width 0.05))
+  (gr_circle (center 159.385 75.565) (end 159.385 74.041) (layer Edge.Cuts) (width 0.05))
+  (gr_line (start 156.845 82.55) (end 170.18 82.55) (layer F.SilkS) (width 0.3302))
+  (gr_line (start 176.53 93.345) (end 176.53 41.275) (layer Edge.Cuts) (width 0.05))
+  (gr_line (start 170.18 93.345) (end 176.53 93.345) (layer Edge.Cuts) (width 0.05))
+  (gr_line (start 170.18 73.025) (end 170.18 93.345) (layer Edge.Cuts) (width 0.05))
+  (gr_line (start 163.83 73.025) (end 170.18 73.025) (layer Edge.Cuts) (width 0.05))
+  (gr_line (start 163.83 41.275) (end 163.83 73.025) (layer Edge.Cuts) (width 0.05))
+  (gr_line (start 176.53 41.275) (end 163.83 41.275) (layer Edge.Cuts) (width 0.05))
   (gr_text ADDR (at 163.195 104.14) (layer F.SilkS)
     (effects (font (size 2.0828 2.0828) (thickness 0.3302)))
@@
     (effects (font (size 5.334 5.334) (thickness 0.7874)))
   )
-  (gr_line (start 171.45 40.64) (end 176.53 40.64) (layer F.CrtYd) (width 0.05))
   (gr_line (start 156.845 107.315) (end 181.61 107.315) (layer Edge.Cuts) (width 0.05))
-  (gr_line (start 176.53 27.305) (end 176.53 107.315) (layer F.CrtYd) (width 0.0254))
-  (gr_line (start 171.45 100.33) (end 176.53 100.33) (layer F.CrtYd) (width 0.05))
-  (gr_circle (center 171.45 37.465) (end 168.275 37.465) (layer F.CrtYd) (width 0.05))
   (gr_circle (center 171.45 37.465) (end 172.974 37.465) (layer Edge.Cuts) (width 0.05))
   (gr_circle (center 171.45 97.155) (end 172.974 97.155) (layer Edge.Cuts) (width 0.15))
   (gr_line (start 156.845 27.305) (end 181.61 27.305) (layer Edge.Cuts) (width 0.05))
   (gr_line (start 156.845 27.305) (end 156.845 107.315) (layer Edge.Cuts) (width 0.05))
-  (gr_circle (center 171.45 97.155) (end 168.275 97.155) (layer F.CrtYd) (width 0.05))
   (gr_line (start 181.61 107.315) (end 181.61 27.305) (layer Edge.Cuts) (width 0.05))
-  (gr_line (start 171.45 34.29) (end 176.53 34.29) (layer F.CrtYd) (width 0.05))
-  (gr_line (start 171.45 93.98) (end 176.53 93.98) (layer F.CrtYd) (width 0.05))
   (gr_line (start 72.39 93.98) (end 72.39 40.64) (layer Edge.Cuts) (width 0.05))
   (gr_line (start 61.595 27.305) (end 86.36 27.305) (layer Edge.Cuts) (width 0.05))
@@
     (effects (font (size 2.0828 2.0828) (thickness 0.3302)) (justify left))
   )
-  (gr_text Halted (at 136.525 66.04) (layer F.SilkS)
-    (effects (font (size 2.0828 2.0828) (thickness 0.3302)) (justify left))
-  )
+  (gr_text "CPU\nhalted" (at 136.525 66.04) (layer F.SilkS)
+    (effects (font (size 2.0828 2.0828) (thickness 0.3302)) (justify left))
+  )

Commit message: office
Other:
- board size 151.8 x 80 mm -> 99.1 x 80 mm
- board text removed: "CARD"
