File: KiCAD files/Front Panel Template/Front Panel Template.kicad_pcb (KiCad board)
At the start: 2 copper layers, 99.1 x 80 mm, 0 parts

Commit message: office
Routing:
- net (no net): vias 0 -> 19
Other:
- outline, holes or cut-outs redrawn
- board text added: "Design by Kaltchuk 2021"
Changed lines of the file:
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@@
   (general
     (thickness 1.6)
-    (drawings 72)
-    (tracks 0)
+    (drawings 57)
+    (tracks 19)
     (zones 0)
     (modules 0)
@@
     (visible_elements 7FFFFFFF)
     (pcbplotparams
-      (layerselection 0x010fc_ffffffff)
+      (layerselection 0x030ff_ffffffff)
       (usegerberextensions false)
       (usegerberattributes true)
@@
       (outputformat 1)
       (mirror false)
-      (drillshape 1)
+      (drillshape 0)
       (scaleselection 1)
       (outputdirectory ""))
@@
     (uvia_dia 0.3)
     (uvia_drill 0.1)
+  )
+  (gr_text "Design by\nKaltchuk\n2021" (at 162.56 37.465) (layer F.SilkS)
+    (effects (font (size 1 1) (thickness 0.15)))
+  )
+  (gr_text "Design by\nKaltchuk\n2021" (at 137.795 37.465) (layer F.SilkS)
+    (effects (font (size 1 1) (thickness 0.15)))
+  )
+  (gr_text "Design by\nKaltchuk\n2021" (at 113.03 37.465) (layer F.SilkS)
+    (effects (font (size 1 1) (thickness 0.15)))
+  )
+  (gr_text "Design by\nKaltchuk\n2021" (at 88.138 37.465) (layer F.SilkS)
+    (effects (font (size 1 1) (thickness 0.15)))
   )
   (gr_line (start 179.07 77.47) (end 179.07 71.755) (layer F.SilkS) (width 0.12))
@@
   )
   (gr_line (start 176.53 82.55) (end 181.61 82.55) (layer F.SilkS) (width 0.3302))
-  (gr_text TX (at 161.29 85.725) (layer F.SilkS)
-    (effects (font (size 2.0828 2.0828) (thickness 0.3302)) (justify left))
-  )
-  (gr_text RX (at 161.29 90.17) (layer F.SilkS)
-    (effects (font (size 2.0828 2.0828) (thickness 0.3302)) (justify left))
-  )
-  (gr_text TX (at 161.29 75.565) (layer F.SilkS)
-    (effects (font (size 2.0828 2.0828) (thickness 0.3302)) (justify left))
-  )
-  (gr_text RX (at 161.29 80.01) (layer F.SilkS)
-    (effects (font (size 2.0828 2.0828) (thickness 0.3302)) (justify left))
-  )
-  (gr_circle (center 159.385 85.725) (end 159.385 84.201) (layer Edge.Cuts) (width 0.05))
-  (gr_circle (center 159.385 90.17) (end 159.385 88.646) (layer Edge.Cuts) (width 0.05))
-  (gr_circle (center 159.385 80.01) (end 159.385 78.486) (layer Edge.Cuts) (width 0.05))
-  (gr_circle (center 159.385 75.565) (end 159.385 74.041) (layer Edge.Cuts) (width 0.05))
+  (gr_text TX (at 163.195 85.725) (layer F.SilkS)
+    (effects (font (size 2.0828 2.0828) (thickness 0.3302)) (justify left))
+  )
+  (gr_text RX (at 163.195 90.17) (layer F.SilkS)
+    (effects (font (size 2.0828 2.0828) (thickness 0.3302)) (justify left))
+  )
+  (gr_text TX (at 163.195 75.565) (layer F.SilkS)
+    (effects (font (size 2.0828 2.0828) (thickness 0.3302)) (justify left))
+  )
+  (gr_text RX (at 163.195 80.01) (layer F.SilkS)
+    (effects (font (size 2.0828 2.0828) (thickness 0.3302)) (justify left))
+  )
   (gr_line (start 156.845 82.55) (end 170.18 82.55) (layer F.SilkS) (width 0.3302))
   (gr_line (start 176.53 93.345) (end 176.53 41.275) (layer Edge.Cuts) (width 0.05))
@@
   )
   (gr_line (start 156.845 107.315) (end 181.61 107.315) (layer Edge.Cuts) (width 0.05))
-  (gr_circle (center 171.45 37.465) (end 172.974 37.465) (layer Edge.Cuts) (width 0.05))
-  (gr_circle (center 171.45 97.155) (end 172.974 97.155) (layer Edge.Cuts) (width 0.15))
   (gr_line (start 156.845 27.305) (end 181.61 27.305) (layer Edge.Cuts) (width 0.05))
   (gr_line (start 181.61 107.315) (end 181.61 27.305) (layer Edge.Cuts) (width 0.05))
   (gr_line (start 93.345 93.98) (end 93.345 40.64) (layer Edge.Cuts) (width 0.05))
   (gr_line (start 82.55 27.305) (end 107.315 27.305) (layer Edge.Cuts) (width 0.05))
-  (gr_circle (center 114.935 66.04) (end 116.459 66.04) (layer Edge.Cuts) (width 0.05))
-  (gr_circle (center 114.935 56.515) (end 116.459 56.515) (layer Edge.Cuts) (width 0.05))
-  (gr_circle (center 114.935 46.99) (end 116.459 46.99) (layer Edge.Cuts) (width 0.05))
   (gr_line (start 82.55 27.305) (end 82.55 107.315) (layer Edge.Cuts) (width 0.05))
   (gr_line (start 93.345 40.64) (end 102.235 40.64) (layer Edge.Cuts) (width 0.05))
   (gr_line (start 107.315 107.315) (end 132.08 107.315) (layer Edge.Cuts) (width 0.05))
-  (gr_circle (center 110.49 46.99) (end 112.014 46.99) (layer Edge.Cuts) (width 0.05))
   (gr_line (start 102.235 40.64) (end 102.235 93.98) (layer Edge.Cuts) (width 0.05))
   (gr_line (start 82.55 107.315) (end 107.315 107.315) (layer Edge.Cuts) (width 0.05))
-  (gr_circle (center 121.92 37.465) (end 123.444 37.465) (layer Edge.Cuts) (width 0.05))
-  (gr_circle (center 121.92 97.155) (end 123.444 97.155) (layer Edge.Cuts) (width 0.15))
   (gr_line (start 107.315 27.305) (end 132.08 27.305) (layer Edge.Cuts) (width 0.05))
   (gr_line (start 107.315 107.315) (end 107.315 27.305) (layer F.SilkS) (width 0.254))
-  (gr_circle (center 97.155 37.465) (end 98.679 37.465) (layer Edge.Cuts) (width 0.05))
-  (gr_circle (center 97.155 97.155) (end 98.679 97.155) (layer Edge.Cuts) (width 0.15))
   (gr_line (start 102.235 93.98) (end 93.345 93.98) (layer Edge.Cuts) (width 0.05))
   (gr_text "RAM\nbank" (at 119.38 66.675) (layer F.SilkS)
@@
     (effects (font (size 2.0828 2.0828) (thickness 0.3302)) (justify left))
   )
-  (gr_circle (center 139.065 84.709) (end 142.621 84.709) (layer Edge.Cuts) (width 0.05))
-  (gr_circle (center 139.065 56.515) (end 140.589 56.515) (layer Edge.Cuts) (width 0.05))
-  (gr_circle (center 139.065 66.04) (end 140.589 66.04) (layer Edge.Cuts) (width 0.05))
   (gr_text "Power\n" (at 143.51 56.515) (layer F.SilkS)
     (effects (font (size 2.0828 2.0828) (thickness 0.3302)) (justify left))
@@
   )
   (gr_line (start 132.08 107.315) (end 156.845 107.315) (layer Edge.Cuts) (width 0.05))
-  (gr_circle (center 146.685 37.465) (end 148.209 37.465) (layer Edge.Cuts) (width 0.05))
-  (gr_circle (center 146.685 97.155) (end 148.209 97.155) (layer Edge.Cuts) (width 0.15))
   (gr_line (start 132.08 27.305) (end 156.845 27.305) (layer Edge.Cuts) (width 0.05))
   (gr_line (start 132.08 27.305) (end 132.08 107.315) (layer F.SilkS) (width 0.254))
@@
     (effects (font (size 5.334 5.334) (thickness 0.7874)))
   )
+  (via (at 171.45 37.465) (size 5.08) (drill 3.048) (layers F.Cu B.Cu) (net 0))
+  (via (at 146.685 37.465) (size 5.08) (drill 3.048) (layers F.Cu B.Cu) (net 0))
+  (via (at 121.92 37.465) (size 5.08) (drill 3.048) (layers F.Cu B.Cu) (net 0))
+  (via (at 97.155 37.465) (size 5.08) (drill 3.048) (layers F.Cu B.Cu) (net 0))
+  (via (at 97.155 97.155) (size 5.08) (drill 3.048) (layers F.Cu B.Cu) (net 0))
+  (via (at 121.92 97.155) (size 5.08) (drill 3.048) (layers F.Cu B.Cu) (net 0))
+  (via (at 146.685 97.155) (size 5.08) (drill 3.048) (layers F.Cu B.Cu) (net 0))
+  (via (at 171.45 97.155) (size 5.08) (drill 3.048) (layers F.Cu B.Cu) (net 0))
+  (via (at 110.49 46.99) (size 4.064) (drill 3.048) (layers F.Cu B.Cu) (net 0))
+  (via (at 114.935 46.99) (size 4.064) (drill 3.048) (layers F.Cu B.Cu) (net 0))
+  (via (at 114.935 56.515) (size 4.064) (drill 3.048) (layers F.Cu B.Cu) (net 0))
+  (via (at 114.935 66.04) (size 4.064) (drill 3.048) (layers F.Cu B.Cu) (net 0))
+  (via (at 139.065 56.515) (size 4.064) (drill 3.048) (layers F.Cu B.Cu) (net 0))
+  (via (at 139.065 66.04) (size 4.064) (drill 3.048) (layers F.Cu B.Cu) (net 0))
+  (via (at 161.29 75.565) (size 4.064) (drill 3.048) (layers F.Cu B.Cu) (net 0))
+  (via (at 161.29 80.01) (size 4.064) (drill 3.048) (layers F.Cu B.Cu) (net 0))
+  (via (at 161.29 85.725) (size 4.064) (drill 3.048) (layers F.Cu B.Cu) (net 0))
+  (via (at 161.29 90.17) (size 4.064) (drill 3.048) (layers F.Cu B.Cu) (net 0))
+  (via (at 139.065 84.709) (size 9.144) (drill 7.112) (layers F.Cu B.Cu) (net 0))
 )

Commit message: home
Other:
- outline, holes or cut-outs redrawn
- board text added: "V-groove"
Changed lines of the file:
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@@
-(kicad_pcb (version 20171130) (host pcbnew "(5.1.6)-1")
+(kicad_pcb (version 20171130) (host pcbnew "(5.1.4)-1")
   (general
     (thickness 1.6)
-    (drawings 57)
+    (drawings 70)
     (tracks 19)
     (zones 0)
@@
     (uvia_drill 0.1)
   )
+  (gr_text V-groove (at 156.21 20.32) (layer Margin)
+    (effects (font (size 2.032 2.032) (thickness 0.3048)))
+  )
+  (gr_text V-groove (at 131.445 20.32) (layer Margin)
+    (effects (font (size 2.032 2.032) (thickness 0.3048)))
+  )
+  (gr_text V-groove (at 107.315 20.32) (layer Margin)
+    (effects (font (size 2.032 2.032) (thickness 0.3048)))
+  )
+  (gr_line (start 170.18 74.295) (end 170.18 92.075) (layer Edge.Cuts) (width 0.05))
+  (gr_line (start 165.1 73.025) (end 168.91 73.025) (layer Edge.Cuts) (width 0.05))
+  (gr_line (start 163.83 42.545) (end 163.83 71.755) (layer Edge.Cuts) (width 0.05))
+  (gr_line (start 175.26 41.275) (end 165.1 41.275) (layer Edge.Cuts) (width 0.05))
+  (gr_line (start 176.53 92.075) (end 176.53 42.545) (layer Edge.Cuts) (width 0.05))
+  (gr_line (start 171.45 93.345) (end 175.26 93.345) (layer Edge.Cuts) (width 0.05))
+  (gr_arc (start 175.26 92.075) (end 175.26 93.345) (angle -90) (layer Edge.Cuts) (width 0.05))
+  (gr_arc (start 171.45 92.075) (end 170.18 92.075) (angle -90) (layer Edge.Cuts) (width 0.05))
+  (gr_arc (start 168.91 74.295) (end 170.18 74.295) (angle -90) (layer Edge.Cuts) (width 0.05))
+  (gr_arc (start 165.1 71.755) (end 163.83 71.755) (angle -90) (layer Edge.Cuts) (width 0.05))
+  (gr_arc (start 165.1 42.545) (end 165.1 41.275) (angle -90) (layer Edge.Cuts) (width 0.05))
+  (gr_arc (start 175.26 42.545) (end 176.53 42.545) (angle -90) (layer Edge.Cuts) (width 0.05))
+  (gr_line (start 93.345 92.71) (end 93.345 41.91) (layer Edge.Cuts) (width 0.05))
+  (gr_line (start 100.965 93.98) (end 94.615 93.98) (layer Edge.Cuts) (width 0.05))
+  (gr_line (start 102.235 41.91) (end 102.235 92.71) (layer Edge.Cuts) (width 0.05))
+  (gr_line (start 100.965 40.64) (end 94.615 40.64) (layer Edge.Cuts) (width 0.05))
+  (gr_arc (start 94.615 92.71) (end 93.345 92.71) (angle -90) (layer Edge.Cuts) (width 0.05))
+  (gr_arc (start 100.965 92.71) (end 100.965 93.98) (angle -90) (layer Edge.Cuts) (width 0.05))
+  (gr_arc (start 100.965 41.91) (end 102.235 41.91) (angle -90) (layer Edge.Cuts) (width 0.05))
+  (gr_arc (start 94.615 41.91) (end 94.615 40.64) (angle -90) (layer Edge.Cuts) (width 0.05))
   (gr_text "Design by\nKaltchuk\n2021" (at 162.56 37.465) (layer F.SilkS)
     (effects (font (size 1 1) (thickness 0.15)))
@@
   )
   (gr_line (start 156.845 82.55) (end 170.18 82.55) (layer F.SilkS) (width 0.3302))
-  (gr_line (start 176.53 93.345) (end 176.53 41.275) (layer Edge.Cuts) (width 0.05))
-  (gr_line (start 170.18 93.345) (end 176.53 93.345) (layer Edge.Cuts) (width 0.05))
-  (gr_line (start 170.18 73.025) (end 170.18 93.345) (layer Edge.Cuts) (width 0.05))
-  (gr_line (start 163.83 73.025) (end 170.18 73.025) (layer Edge.Cuts) (width 0.05))
-  (gr_line (start 163.83 41.275) (end 163.83 73.025) (layer Edge.Cuts) (width 0.05))
-  (gr_line (start 176.53 41.275) (end 163.83 41.275) (layer Edge.Cuts) (width 0.05))
   (gr_text ADDR (at 163.195 104.14) (layer F.SilkS)
     (effects (font (size 2.0828 2.0828) (thickness 0.3302)))
@@
   (gr_line (start 156.845 27.305) (end 181.61 27.305) (layer Edge.Cuts) (width 0.05))
   (gr_line (start 181.61 107.315) (end 181.61 27.305) (layer Edge.Cuts) (width 0.05))
-  (gr_line (start 93.345 93.98) (end 93.345 40.64) (layer Edge.Cuts) (width 0.05))
   (gr_line (start 82.55 27.305) (end 107.315 27.305) (layer Edge.Cuts) (width 0.05))
   (gr_line (start 82.55 27.305) (end 82.55 107.315) (layer Edge.Cuts) (width 0.05))
-  (gr_line (start 93.345 40.64) (end 102.235 40.64) (layer Edge.Cuts) (width 0.05))
   (gr_line (start 107.315 107.315) (end 132.08 107.315) (layer Edge.Cuts) (width 0.05))
-  (gr_line (start 102.235 40.64) (end 102.235 93.98) (layer Edge.Cuts) (width 0.05))
   (gr_line (start 82.55 107.315) (end 107.315 107.315) (layer Edge.Cuts) (width 0.05))
   (gr_line (start 107.315 27.305) (end 132.08 27.305) (layer Edge.Cuts) (width 0.05))
-  (gr_line (start 107.315 107.315) (end 107.315 27.305) (layer F.SilkS) (width 0.254))
-  (gr_line (start 102.235 93.98) (end 93.345 93.98) (layer Edge.Cuts) (width 0.05))
+  (gr_line (start 107.315 107.315) (end 107.315 22.86) (layer Margin) (width 0.254))
   (gr_text "RAM\nbank" (at 119.38 66.675) (layer F.SilkS)
     (effects (font (size 2.0828 2.0828) (thickness 0.3302)) (justify left))
@@
   (gr_line (start 132.08 107.315) (end 156.845 107.315) (layer Edge.Cuts) (width 0.05))
   (gr_line (start 132.08 27.305) (end 156.845 27.305) (layer Edge.Cuts) (width 0.05))
-  (gr_line (start 132.08 27.305) (end 132.08 107.315) (layer F.SilkS) (width 0.254))
-  (gr_line (start 156.845 107.315) (end 156.845 27.305) (layer F.SilkS) (width 0.254))
+  (gr_line (start 132.08 22.86) (end 132.08 107.315) (layer Margin) (width 0.254))
+  (gr_line (start 156.845 107.315) (end 156.845 22.86) (layer Margin) (width 0.254))
   (gr_text ADDR (at 138.43 104.14) (layer F.SilkS)
     (effects (font (size 2.0828 2.0828) (thickness 0.3302)))

Commit message: home
Other:
- board text removed: "V-groove"
Changed lines of the file:
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@@
   (general
     (thickness 1.6)
-    (drawings 70)
+    (drawings 67)
     (tracks 19)
     (zones 0)
@@
     (visible_elements 7FFFFFFF)
     (pcbplotparams
-      (layerselection 0x030ff_ffffffff)
+      (layerselection 0x030e0_ffffffff)
       (usegerberextensions false)
       (usegerberattributes true)
@@
     (uvia_drill 0.1)
   )
-  (gr_text V-groove (at 156.21 20.32) (layer Margin)
-    (effects (font (size 2.032 2.032) (thickness 0.3048)))
-  )
-  (gr_text V-groove (at 131.445 20.32) (layer Margin)
-    (effects (font (size 2.032 2.032) (thickness 0.3048)))
-  )
-  (gr_text V-groove (at 107.315 20.32) (layer Margin)
-    (effects (font (size 2.032 2.032) (thickness 0.3048)))
-  )
   (gr_line (start 170.18 74.295) (end 170.18 92.075) (layer Edge.Cuts) (width 0.05))
   (gr_line (start 165.1 73.025) (end 168.91 73.025) (layer Edge.Cuts) (width 0.05))
@@
   (gr_line (start 82.55 107.315) (end 107.315 107.315) (layer Edge.Cuts) (width 0.05))
   (gr_line (start 107.315 27.305) (end 132.08 27.305) (layer Edge.Cuts) (width 0.05))
-  (gr_line (start 107.315 107.315) (end 107.315 22.86) (layer Margin) (width 0.254))
+  (gr_line (start 107.315 107.315) (end 107.188 27.432) (layer Margin) (width 0.254))
   (gr_text "RAM\nbank" (at 119.38 66.675) (layer F.SilkS)
     (effects (font (size 2.0828 2.0828) (thickness 0.3302)) (justify left))
@@
   (gr_line (start 132.08 107.315) (end 156.845 107.315) (layer Edge.Cuts) (width 0.05))
   (gr_line (start 132.08 27.305) (end 156.845 27.305) (layer Edge.Cuts) (width 0.05))
-  (gr_line (start 132.08 22.86) (end 132.08 107.315) (layer Margin) (width 0.254))
-  (gr_line (start 156.845 107.315) (end 156.845 22.86) (layer Margin) (width 0.254))
+  (gr_line (start 132.08 27.432) (end 132.08 107.315) (layer Margin) (width 0.254))
+  (gr_line (start 156.845 107.315) (end 156.972 27.432) (layer Margin) (width 0.254))
   (gr_text ADDR (at 138.43 104.14) (layer F.SilkS)
     (effects (font (size 2.0828 2.0828) (thickness 0.3302)))
