File: KiCAD files/Front Panel/Front Panel.sch (KiCad schematic (older format))
At the start: 0 parts

Commit message: home
Parts:
- added R1, R2, R3, R4: 1k, Resistor_SMD:R_0603_1608Metric_Pad1.05x0.95mm_HandSolder, symbol Device:R_US
Connections:
- net GND: now also R1.2, R2.2, R3.2, R4.2
- new net +5V: R1.1, R2.1, R3.1, R4.1
- no-connect marks 1 -> 0
Changed lines of the file:
@@
 L power:GND #PWR01
 U 1 1 61EC441F
-P 2800 2200
-F 0 "#PWR01" H 2800 1950 50  0001 C CNN
-F 1 "GND" H 2805 2027 50  0000 C CNN
-F 2 "" H 2800 2200 50  0001 C CNN
-F 3 "" H 2800 2200 50  0001 C CNN
-	1    2800 2200
+P 2050 2400
+F 0 "#PWR01" H 2050 2150 50  0001 C CNN
+F 1 "GND" H 2055 2227 50  0000 C CNN
+F 2 "" H 2050 2400 50  0001 C CNN
+F 3 "" H 2050 2400 50  0001 C CNN
+	1    2050 2400
 	1    0    0    -1
 $EndComp
-NoConn ~ 2800 2200
+$Comp
+L power:+5V #PWR02
+U 1 1 61EDA0DA
+P 2050 1750
+F 0 "#PWR02" H 2050 1600 50  0001 C CNN
+F 1 "+5V" H 2065 1923 50  0000 C CNN
+F 2 "" H 2050 1750 50  0001 C CNN
+F 3 "" H 2050 1750 50  0001 C CNN
+	1    2050 1750
+	1    0    0    -1
+$EndComp
+$Comp
+L Device:R_US R3
+U 1 1 61EDA887
+P 1750 2050
+F 0 "R3" H 1818 2096 50  0000 L CNN
+F 1 "1k" H 1818 2005 50  0000 L CNN
+F 2 "Resistor_SMD:R_0603_1608Metric_Pad1.05x0.95mm_HandSolder" V 1790 2040 50  0001 C CNN
+F 3 "~" H 1750 2050 50  0001 C CNN
+	1    1750 2050
+	1    0    0    -1
+$EndComp
+$Comp
+L Device:R_US R2
+U 1 1 61EDAB12
+P 1450 2050
+F 0 "R2" H 1518 2096 50  0000 L CNN
+F 1 "1k" H 1518 2005 50  0000 L CNN
+F 2 "Resistor_SMD:R_0603_1608Metric_Pad1.05x0.95mm_HandSolder" V 1490 2040 50  0001 C CNN
+F 3 "~" H 1450 2050 50  0001 C CNN
+	1    1450 2050
+	1    0    0    -1
+$EndComp
+$Comp
+L Device:R_US R1
+U 1 1 61EDB279
+P 1150 2050
+F 0 "R1" H 1218 2096 50  0000 L CNN
+F 1 "1k" H 1218 2005 50  0000 L CNN
+F 2 "Resistor_SMD:R_0603_1608Metric_Pad1.05x0.95mm_HandSolder" V 1190 2040 50  0001 C CNN
+F 3 "~" H 1150 2050 50  0001 C CNN
+	1    1150 2050
+	1    0    0    -1
+$EndComp
+$Comp
+L Device:R_US R4
+U 1 1 61EDB9F7
+P 2050 2050
+F 0 "R4" H 2118 2096 50  0000 L CNN
+F 1 "1k" H 2118 2005 50  0000 L CNN
+F 2 "Resistor_SMD:R_0603_1608Metric_Pad1.05x0.95mm_HandSolder" V 2090 2040 50  0001 C CNN
+F 3 "~" H 2050 2050 50  0001 C CNN
+	1    2050 2050
+	1    0    0    -1
+$EndComp
+Wire Wire Line
+	1150 1900 1450 1900
+Wire Wire Line
+	1450 1900 1750 1900
+Connection ~ 1450 1900
+Wire Wire Line
+	1750 1900 2050 1900
+Connection ~ 1750 1900
+Wire Wire Line
+	1150 2200 1450 2200
+Wire Wire Line
+	1450 2200 1750 2200
+Connection ~ 1450 2200
+Wire Wire Line
+	1750 2200 2050 2200
+Connection ~ 1750 2200
+Wire Wire Line
+	2050 2400 2050 2200
+Connection ~ 2050 2200
+Wire Wire Line
+	2050 1750 2050 1900
+Connection ~ 2050 1900
 $EndSCHEMATC

Commit message: home
Parts:
- removed R1, R2, R3, R4: 1k, Resistor_SMD:R_0603_1608Metric_Pad1.05x0.95mm_HandSolder, symbol Device:R_US
- added J1, J2, J3, J4, J5, J6, J7, J8: fixing bolt, Connector_PinHeader_2.54mm:PinHeader_1x01_P2.54mm_Vertical, symbol Connector:Conn_01x01_Male
- added J10, J11, J12, J13, J14, J15, J16, J17, J18, J19: led, Connector_PinHeader_2.54mm:PinHeader_1x01_P2.54mm_Vertical, symbol Connector:Conn_01x01_Male
- added J9: reset button, Connector_PinHeader_2.54mm:PinHeader_1x01_P2.54mm_Vertical, symbol Connector:Conn_01x01_Male
Connections:
- net GND: now also J1.1 (Pin_1), J10.1 (Pin_1), J11.1 (Pin_1), J12.1 (Pin_1), J13.1 (Pin_1), J14.1 (Pin_1), J15.1 (Pin_1), J16.1 (Pin_1), J17.1 (Pin_1), J18.1 (Pin_1), J19.1 (Pin_1), J2.1 (Pin_1), J3.1 (Pin_1), J4.1 (Pin_1), J5.1 (Pin_1), J6.1 (Pin_1), J7.1 (Pin_1), J8.1 (Pin_1), J9.1 (Pin_1)
