File: KiCAD files/Front Panel/Front Panel.kicad_pcb (KiCad board)
At the start: 2 copper layers, 99.1 x 80 mm, 0 parts

Commit message: home
Parts:
- added R1: 1k, Resistor_SMD:R_0603_1608Metric_Pad1.05x0.95mm_HandSolder, B.Cu at (87.9, 75.6)
- added R2: 1k, Resistor_SMD:R_0603_1608Metric_Pad1.05x0.95mm_HandSolder, B.Cu at (119.6, 75.6)
- added R3: 1k, Resistor_SMD:R_0603_1608Metric_Pad1.05x0.95mm_HandSolder, B.Cu at (148.3, 75.4)
- added R4: 1k, Resistor_SMD:R_0603_1608Metric_Pad1.05x0.95mm_HandSolder, B.Cu at (160.4, 61.7)
Routing:
- net GND: track 0.00 -> 143.5 mm
- net +5V: track 0.00 -> 109.4 mm
- added copper zone on B.Cu, net GND
- removed copper zone on B.Cu, net (none)

Commit message: home
Parts:
- removed R1, R2, R3, R4: 1k, Resistor_SMD:R_0603_1608Metric_Pad1.05x0.95mm_HandSolder
- added J1: fixing bolt, Connector_PinHeader_2.54mm:PinHeader_1x01_P2.54mm_Vertical, F.Cu at (97.2, 37.5)
- added J10: led, Connector_PinHeader_2.54mm:PinHeader_1x01_P2.54mm_Vertical, F.Cu at (110.5, 47.0)
- added J11: led, Connector_PinHeader_2.54mm:PinHeader_1x01_P2.54mm_Vertical, F.Cu at (114.9, 47.0)
- added J12: led, Connector_PinHeader_2.54mm:PinHeader_1x01_P2.54mm_Vertical, F.Cu at (114.9, 56.5)
- added J13: led, Connector_PinHeader_2.54mm:PinHeader_1x01_P2.54mm_Vertical, F.Cu at (114.9, 66.0)
- added J14: led, Connector_PinHeader_2.54mm:PinHeader_1x01_P2.54mm_Vertical, F.Cu at (139.1, 56.5)
- added J15: led, Connector_PinHeader_2.54mm:PinHeader_1x01_P2.54mm_Vertical, F.Cu at (139.1, 66.0)
- added J16: led, Connector_PinHeader_2.54mm:PinHeader_1x01_P2.54mm_Vertical, F.Cu at (161.3, 75.6)
- added J17: led, Connector_PinHeader_2.54mm:PinHeader_1x01_P2.54mm_Vertical, F.Cu at (161.3, 80.0)
- added J18: led, Connector_PinHeader_2.54mm:PinHeader_1x01_P2.54mm_Vertical, F.Cu at (161.3, 85.7)
- added J19: led, Connector_PinHeader_2.54mm:PinHeader_1x01_P2.54mm_Vertical, F.Cu at (161.3, 90.2)
- added J2: fixing bolt, Connector_PinHeader_2.54mm:PinHeader_1x01_P2.54mm_Vertical, F.Cu at (97.2, 97.2)
- added J3: fixing bolt, Connector_PinHeader_2.54mm:PinHeader_1x01_P2.54mm_Vertical, F.Cu at (121.9, 37.5)
- added J4: fixing bolt, Connector_PinHeader_2.54mm:PinHeader_1x01_P2.54mm_Vertical, F.Cu at (121.9, 97.2)
- added J5: fixing bolt, Connector_PinHeader_2.54mm:PinHeader_1x01_P2.54mm_Vertical, F.Cu at (146.7, 37.5)
- added J6: fixing bolt, Connector_PinHeader_2.54mm:PinHeader_1x01_P2.54mm_Vertical, F.Cu at (146.7, 97.2)
- added J7: fixing bolt, Connector_PinHeader_2.54mm:PinHeader_1x01_P2.54mm_Vertical, F.Cu at (171.4, 37.5)
- added J8: fixing bolt, Connector_PinHeader_2.54mm:PinHeader_1x01_P2.54mm_Vertical, F.Cu at (171.4, 97.2)
- added J9: reset button, Connector_PinHeader_2.54mm:PinHeader_1x01_P2.54mm_Vertical, F.Cu at (139.2, 84.8)
Routing:
- net GND: track 143.5 -> 0.00 mm
- net +5V: track 109.4 -> 0.00 mm
- net (no net): vias 19 -> 0

Commit message: office
Other:
- net class Default removed
