File: KiCAD files/PSU/PSU.sch (KiCad schematic (older format))
At the start: 7 parts, among them J1 Ext power on, J2 Power switch, J3 Mains, J4 Power bus, K1 SRD-05VDC-SL-C

Commit message: HOME
Connections:
- net LINE: now also K1.5, K1.6; no longer K1.1
- net at F1.1, J2.1 (Pin_1): now also K1.1; no longer K1.5, K1.6
Other:
- moved on the sheet: J2
Changed lines of the file:
@@
 L Connector_Generic:Conn_01x02 J2
 U 1 1 6145B14B
-P 3950 3300
-F 0 "J2" H 3868 3425 50  0000 C CNN
-F 1 "Power switch" H 3868 3426 50  0001 C CNN
-F 2 "Connector_PinHeader_2.54mm:PinHeader_1x02_P2.54mm_Vertical" H 3950 3300 50  0001 C CNN
-F 3 "~" H 3950 3300 50  0001 C CNN
-	1    3950 3300
+P 3950 3200
+F 0 "J2" H 3868 3325 50  0000 C CNN
+F 1 "Power switch" H 3868 3326 50  0001 C CNN
+F 2 "Connector_PinHeader_2.54mm:PinHeader_1x02_P2.54mm_Vertical" H 3950 3200 50  0001 C CNN
+F 3 "~" H 3950 3200 50  0001 C CNN
+	1    3950 3200
 	-1   0    0    -1
 $EndComp
 Text Notes 3800 2900 2    50   ~ 0
 External\nPower on
-Text Notes 3800 3400 2    50   ~ 0
+Text Notes 3800 3300 2    50   ~ 0
 Power on\nSwitch
 Text Notes 3850 4500 2    50   ~ 0
@@
 NoConn ~ 7350 4200
 Wire Wire Line
-	4150 3400 4300 3400
-Wire Wire Line
-	4300 3400 4300 3600
-Wire Wire Line
 	4300 4300 4150 4300
 $Comp
@@
 NoConn ~ 5100 3200
 Wire Wire Line
-	4150 3300 4400 3300
-Wire Wire Line
-	4400 3300 4400 3950
+	4150 3200 4400 3200
 Wire Wire Line
 	4400 3950 4650 3950
-Wire Wire Line
-	4500 3300 4400 3300
-Connection ~ 4400 3300
-Connection ~ 4300 3600
-Wire Wire Line
-	4300 3600 4300 4300
 Wire Wire Line
 	4150 2900 4500 2900
@@
 Wire Wire Line
 	5100 3400 5250 3400
-Wire Wire Line
-	4300 3600 5250 3600
 Wire Wire Line
 	7200 4100 7200 3550
@@
 	1    0    0    -1
 $EndComp
+Wire Wire Line
+	4400 3200 4400 3600
+Wire Wire Line
+	4150 3300 4300 3300
+Connection ~ 4300 3300
+Wire Wire Line
+	4300 3300 4500 3300
+Wire Wire Line
+	4300 3300 4300 4300
+Wire Wire Line
+	5250 3600 4400 3600
+Connection ~ 4400 3600
+Wire Wire Line
+	4400 3600 4400 3950
 $EndSCHEMATC

Commit message: home
Parts:
- removed F1: 100mA, MyStuff:FuseHolder_Cylinder-27x8.5mm_Horizontal, symbol Device:Fuse
- removed J3: Mains, Connector_Phoenix_MC_HighVoltage:PhoenixContact_MC_1,5_3-G-5.08_1x03_P5.08mm_Horizontal, symbol Connector_Generic:Conn_01x03
- added J3: Mains, symbol Connector_Generic:Conn_01x02
- added J5: Mech support, Connector_PinHeader_2.54mm:PinHeader_2x05_P2.54mm_Vertical, symbol Connector_Generic:Conn_02x05_Odd_Even
Connections:
- net LINE: now also J3.1 (Pin_1)
- net NEUT: now also J3.2 (Pin_2)
- net at J2.1 (Pin_1), K1.1: now also PS1.2 (AC/L)
- no-connect marks 6 -> 15
Other:
- note added: "220Vac\n\nLine\nNeutral"
- note removed: "220Vac\n\nLine\nNeutral\nNC"
Changed lines of the file:
@@
-$EndComp
-$Comp
-L Device:Fuse F1
-U 1 1 6144E395
-P 4800 3950
-F 0 "F1" V 4900 3900 50  0000 L CNN
-F 1 "100mA" V 4700 3850 50  0000 L CNN
-F 2 "MyStuff:FuseHolder_Cylinder-27x8.5mm_Horizontal" V 4730 3950 50  0001 C CNN
-F 3 "~" H 4800 3950 50  0001 C CNN
-	1    4800 3950
-	0    -1   -1   0
 $EndComp
 $Comp
@@
 	1    7550 4200
 	1    0    0    -1
-$EndComp
-$Comp
-L Connector_Generic:Conn_01x03 J3
-U 1 1 6145B022
-P 3950 4400
-F 0 "J3" H 3868 4625 50  0000 C CNN
-F 1 "Mains" H 3868 4626 50  0001 C CNN
-F 2 "Connector_Phoenix_MC_HighVoltage:PhoenixContact_MC_1,5_3-G-5.08_1x03_P5.08mm_Horizontal" H 3950 4400 50  0001 C CNN
-F 3 "~" H 3950 4400 50  0001 C CNN
-	1    3950 4400
-	-1   0    0    1
 $EndComp
 $Comp
@@
 Text Notes 3800 3300 2    50   ~ 0
 Power on\nSwitch
-Text Notes 3850 4500 2    50   ~ 0
-220Vac\n\nLine\nNeutral\nNC
-NoConn ~ 4150 4500
-Wire Wire Line
-	4950 3950 5200 3950
+Text Notes 3850 4400 2    50   ~ 0
+220Vac\n\nLine\nNeutral
 Wire Wire Line
 	5200 3950 5200 4200
-Wire Wire Line
-	5200 4200 5650 4200
 Wire Wire Line
 	6450 4400 7200 4400
@@
 	4150 3200 4400 3200
 Wire Wire Line
-	4400 3950 4650 3950
-Wire Wire Line
 	4150 2900 4500 2900
 Wire Wire Line
@@
 	7200 4600 8050 4600
 $Comp
-L power:NEUT #PWR02
+L power:NEUT #PWR0101
 U 1 1 61474800
 P 5000 4300
-F 0 "#PWR02" H 5000 4150 50  0001 C CNN
+F 0 "#PWR0101" H 5000 4150 50  0001 C CNN
 F 1 "NEUT" H 5017 4473 50  0000 C CNN
 F 2 "" H 5000 4300 50  0001 C CNN
@@
 $EndComp
 $Comp
-L power:LINE #PWR01
+L power:LINE #PWR0102
 U 1 1 61475171
 P 4500 4300
-F 0 "#PWR01" H 4500 4150 50  0001 C CNN
+F 0 "#PWR0102" H 4500 4150 50  0001 C CNN
 F 1 "LINE" H 4517 4473 50  0000 C CNN
 F 2 "" H 4500 4300 50  0001 C CNN
@@
 	5000 4300 5000 4400
 $Comp
-L power:PWR_FLAG #FLG01
+L power:PWR_FLAG #FLG0101
 U 1 1 61479542
 P 4500 4600
-F 0 "#FLG01" H 4500 4675 50  0001 C CNN
+F 0 "#FLG0101" H 4500 4675 50  0001 C CNN
 F 1 "PWR_FLAG" H 4500 4773 50  0000 C CNN
 F 2 "" H 4500 4600 50  0001 C CNN
@@
 $EndComp
 $Comp
-L power:PWR_FLAG #FLG02
+L power:PWR_FLAG #FLG0102
 U 1 1 61479DC0
 P 5000 4600
-F 0 "#FLG02" H 5000 4675 50  0001 C CNN
+F 0 "#FLG0102" H 5000 4675 50  0001 C CNN
 F 1 "PWR_FLAG" H 5000 4773 50  0000 C CNN
 F 2 "" H 5000 4600 50  0001 C CNN
@@
 Wire Wire Line
 	4400 3600 4400 3950
+Wire Wire Line
+	4400 3950 5200 3950
+NoConn ~ 7350 4950
+NoConn ~ 7350 5050
+NoConn ~ 7350 5150
+NoConn ~ 7350 5250
+NoConn ~ 7350 5350
+NoConn ~ 7850 5350
+NoConn ~ 7850 5250
+NoConn ~ 7850 5150
+NoConn ~ 7850 5050
+NoConn ~ 7850 4950
+$Comp
+L Connector_Generic:Conn_02x05_Odd_Even J5
+U 1 1 61F18D3E
+P 7550 5150
+F 0 "J5" H 7600 5567 50  0000 C CNN
+F 1 "Mech support" H 7600 5476 50  0000 C CNN
+F 2 "Connector_PinHeader_2.54mm:PinHeader_2x05_P2.54mm_Vertical" H 7550 5150 50  0001 C CNN
+F 3 "~" H 7550 5150 50  0001 C CNN
+	1    7550 5150
+	1    0    0    -1
+$EndComp
+Wire Wire Line
+	5650 4200 5200 4200
+$Comp
+L Connector_Generic:Conn_01x02 J3
+U 1 1 61F19FC2
+P 3950 4300
+F 0 "J3" H 3868 4517 50  0000 C CNN
+F 1 "Mains" H 3868 4426 50  0000 C CNN
+F 2 "" H 3950 4300 50  0001 C CNN
+F 3 "~" H 3950 4300 50  0001 C CNN
+	1    3950 4300
+	-1   0    0    -1
+$EndComp
 $EndSCHEMATC

Commit message: home
Parts:
- J3: footprint (none) -> MyStuff:IEC60320_2pin
Changed lines of the file:
@@
 F 0 "J3" H 3868 4517 50  0000 C CNN
 F 1 "Mains" H 3868 4426 50  0000 C CNN
-F 2 "" H 3950 4300 50  0001 C CNN
+F 2 "MyStuff:IEC60320_2pin" H 3950 4300 50  0001 C CNN
 F 3 "~" H 3950 4300 50  0001 C CNN
 	1    3950 4300
