File: KiCAD files/PSU/PSU.kicad_pcb (KiCad board)
At the start: 2 copper layers, 99.7 x 69.8 mm, 7 parts, among them J1 Ext power on, J2 Power switch, J3 Mains, J4 Power bus, K1 SRD-05VDC-SL-C

Commit message: HOME
Connections:
- K1 pad 1: LINE -> Net-(F1-Pad1)
- K1 pad 5: Net-(F1-Pad1) -> LINE
Routing:
- net LINE: track 0.00 -> 73.0 mm
- net NEUT: track 0.00 -> 71.4 mm
- net Net-(J1-Pad2): track 0.00 -> 50.4 mm
- net Net-(J4-Pad1): track 0.00 -> 43.6 mm
- net Net-(F1-Pad2): track 0.00 -> 41.4 mm
- net Net-(J1-Pad1): track 0.00 -> 41.3 mm
- net Net-(J4-Pad3): track 0.00 -> 32.6 mm
- net Net-(F1-Pad1): track 0.00 -> 24.3 mm
- net (no net): vias 0 -> 2
- added copper zone on B.Cu, net Net-(J4-Pad1)
Changed lines of the file:
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@@
     (thickness 1.6)
     (drawings 4)
-    (tracks 0)
+    (tracks 48)
     (zones 0)
     (modules 7)
@@
       (effects (font (size 1 1) (thickness 0.15)))
     )
+    (fp_text user +5V (at 17.78 -58.166) (layer F.SilkS)
+      (effects (font (size 1 1) (thickness 0.15)))
+    )
+    (fp_text user gnd (at 11.176 -58.166) (layer F.SilkS)
+      (effects (font (size 1 1) (thickness 0.15)))
+    )
+    (fp_text user line (at 8.89 -8.636) (layer F.SilkS)
+      (effects (font (size 1 1) (thickness 0.15)))
+    )
+    (fp_text user neutral (at 10.16 -15.24) (layer F.SilkS)
+      (effects (font (size 1 1) (thickness 0.15)))
+    )
+    (fp_line (start 32.512 -64.516) (end 0 -64.516) (layer F.SilkS) (width 0.12))
+    (fp_line (start 0 0) (end 32.512 0) (layer F.SilkS) (width 0.12))
+    (fp_line (start 32.512 -64.516) (end 32.512 0) (layer F.SilkS) (width 0.12))
+    (fp_line (start 0 -64.516) (end 0 0) (layer F.SilkS) (width 0.12))
+    (fp_line (start 32.4 0) (end 32.4 -64.65) (layer F.CrtYd) (width 0.12))
+    (fp_line (start 0 0) (end 0 -64.65) (layer F.CrtYd) (width 0.12))
+    (fp_line (start 0 -64.65) (end 32.4 -64.65) (layer F.CrtYd) (width 0.12))
     (fp_line (start 0 0) (end 32.4 0) (layer F.CrtYd) (width 0.12))
-    (fp_line (start 0 -65) (end 32.4 -65) (layer F.CrtYd) (width 0.12))
-    (fp_line (start 0 0) (end 0 -65) (layer F.CrtYd) (width 0.12))
-    (fp_line (start 32.4 0) (end 32.4 -65) (layer F.CrtYd) (width 0.12))
-    (fp_line (start -0.254 -65.278) (end -0.254 0.254) (layer F.SilkS) (width 0.12))
-    (fp_line (start 32.512 -65.278) (end 32.512 0.254) (layer F.SilkS) (width 0.12))
-    (fp_line (start -0.254 0.254) (end 32.512 0.254) (layer F.SilkS) (width 0.12))
-    (fp_line (start 32.512 -65.278) (end -0.254 -65.278) (layer F.SilkS) (width 0.12))
-    (fp_text user neutral (at 10.16 -15.24) (layer F.SilkS)
-      (effects (font (size 1 1) (thickness 0.15)))
-    )
-    (fp_text user line (at 8.89 -8.636) (layer F.SilkS)
-      (effects (font (size 1 1) (thickness 0.15)))
-    )
-    (fp_text user gnd (at 11.176 -58.166) (layer F.SilkS)
-      (effects (font (size 1 1) (thickness 0.15)))
-    )
-    (fp_text user +5V (at 17.78 -58.166) (layer F.SilkS)
-      (effects (font (size 1 1) (thickness 0.15)))
-    )
-    (pad 2 thru_hole circle (at 5 -8.6) (size 2 2) (drill 1) (layers *.Cu *.Mask)
+    (pad "" thru_hole circle (at 29 -62) (size 4 4) (drill 3) (layers *.Cu *.Mask))
+    (pad "" thru_hole circle (at 29 -2.5) (size 4 4) (drill 3) (layers *.Cu *.Mask))
+    (pad "" thru_hole circle (at 3.8 -62) (size 4 4) (drill 3) (layers *.Cu *.Mask))
+    (pad "" thru_hole circle (at 3.8 -2.5) (size 4 4) (drill 3) (layers *.Cu *.Mask))
+    (pad 4 thru_hole circle (at 15.7 -59.7) (size 2 2) (drill 1) (layers *.Cu *.Mask)
+      (net 8 "Net-(J4-Pad3)"))
+    (pad 3 thru_hole circle (at 13.2 -59.7) (size 2 2) (drill 1) (layers *.Cu *.Mask)
+      (net 7 "Net-(J4-Pad1)"))
+    (pad 1 thru_hole circle (at 3.1 -14.3) (size 2 2) (drill 1) (layers *.Cu *.Mask)
+      (net 6 NEUT))
+    (pad 2 thru_hole circle (at 3.1 -9.3) (size 2 2) (drill 1) (layers *.Cu *.Mask)
       (net 2 "Net-(F1-Pad2)"))
-    (pad 1 thru_hole circle (at 5 -15) (size 2 2) (drill 1) (layers *.Cu *.Mask)
-      (net 6 NEUT))
-    (pad 3 thru_hole circle (at 11.4 -61) (size 2 2) (drill 1) (layers *.Cu *.Mask)
-      (net 7 "Net-(J4-Pad1)"))
-    (pad 4 thru_hole circle (at 18 -61) (size 2 2) (drill 1) (layers *.Cu *.Mask)
-      (net 8 "Net-(J4-Pad3)"))
-    (pad "" thru_hole circle (at 2.7 -2.5) (size 4 4) (drill 3) (layers *.Cu *.Mask))
-    (pad "" thru_hole circle (at 2.7 -62.5) (size 4 4) (drill 3) (layers *.Cu *.Mask))
-    (pad "" thru_hole circle (at 29.9 -2.5) (size 4 4) (drill 3) (layers *.Cu *.Mask))
-    (pad "" thru_hole circle (at 29.9 -62.5) (size 4 4) (drill 3) (layers *.Cu *.Mask))
   )
   (module MyStuff:Relay_SPDT_Songel-15x19mm (layer F.Cu)
@@
     (fp_line (start -2.032 2.54) (end -2.032 -17.018) (layer F.Fab) (width 0.12))
     (pad 1 thru_hole circle (at 0 0) (size 2.5 2.5) (drill 0.762) (layers *.Cu *.Mask)
-      (net 5 LINE))
+      (net 1 "Net-(F1-Pad1)"))
     (pad 2 thru_hole circle (at 11.43 0) (size 2.5 2.5) (drill 0.762) (layers *.Cu *.Mask)
       (net 13 "Net-(K1-Pad2)"))
@@
       (net 4 "Net-(J1-Pad1)"))
     (pad 5 thru_hole circle (at 5.715 -14.605) (size 2.5 2.5) (drill 0.762) (layers *.Cu *.Mask)
-      (net 1 "Net-(F1-Pad1)"))
+      (net 5 LINE))
   )
   (module Connector_PinHeader_2.54mm:PinHeader_2x05_P2.54mm_Vertical (layer F.Cu)
@@
       (effects (font (size 1 1) (thickness 0.15)))
     )
-    (fp_text value Mains (at 5.08 9.2 90) (layer F.Fab)
+    (fp_text value Mains (at 5.08 6.35 90) (layer F.Fab)
       (effects (font (size 1 1) (thickness 0.15)))
     )
@@
   (gr_line (start 97.79 121.92) (end 197.485 121.92) (layer Edge.Cuts) (width 0.05))
   (gr_line (start 97.79 52.07) (end 197.485 52.07) (layer Edge.Cuts) (width 0.05))
+  (via (at 192.405 57.15) (size 5.08) (drill 3.048) (layers F.Cu B.Cu) (net 0))
+  (via (at 192.405 116.84) (size 5.08) (drill 3.048) (layers F.Cu B.Cu) (net 0))
+  (segment (start 156.21 86.36) (end 156.845 86.995) (width 1.016) (layer B.Cu) (net 1))
+  (segment (start 156.21 71.755) (end 156.21 86.36) (width 1.016) (layer B.Cu) (net 1))
+  (segment (start 156.845 93.98) (end 158.115 95.25) (width 1.016) (layer B.Cu) (net 1))
+  (segment (start 156.845 86.995) (end 156.845 93.98) (width 1.016) (layer B.Cu) (net 1))
+  (segment (start 151.945 110.08) (end 158.115 116.25) (width 1.016) (layer B.Cu) (net 2))
+  (segment (start 119.305 110.08) (end 151.945 110.08) (width 1.016) (layer B.Cu) (net 2))
+  (segment (start 189.297919 88.9) (end 190.5 88.9) (width 1.016) (layer B.Cu) (net 3))
+  (segment (start 186.69 86.292081) (end 189.297919 88.9) (width 1.016) (layer B.Cu) (net 3))
+  (segment (start 186.69 79.375) (end 186.69 86.292081) (width 1.016) (layer B.Cu) (net 3))
+  (segment (start 173.355 66.04) (end 186.69 79.375) (width 1.016) (layer B.Cu) (net 3))
+  (segment (start 162.56 66.04) (end 173.355 66.04) (width 1.016) (layer B.Cu) (net 3))
+  (segment (start 156.21 59.69) (end 162.56 66.04) (width 1.016) (layer B.Cu) (net 3))
+  (segment (start 167.64 59.69) (end 176.53 59.69) (width 1.016) (layer B.Cu) (net 4))
+  (segment (start 190.5 73.66) (end 190.5 86.36) (width 1.016) (layer B.Cu) (net 4))
+  (segment (start 176.53 59.69) (end 190.5 73.66) (width 1.016) (layer B.Cu) (net 4))
+  (segment (start 168.91 96.52) (end 159.385 86.995) (width 1.016) (layer B.Cu) (net 5))
+  (segment (start 189.23 96.52) (end 168.91 96.52) (width 1.016) (layer B.Cu) (net 5))
+  (segment (start 159.385 85.792919) (end 159.385 86.995) (width 1.016) (layer B.Cu) (net 5))
+  (segment (start 159.385 71.576318) (end 159.385 85.792919) (width 1.016) (layer B.Cu) (net 5))
+  (segment (start 153.943999 66.135317) (end 159.385 71.576318) (width 1.016) (layer B.Cu) (net 5))
+  (segment (start 153.943999 58.602319) (end 153.943999 66.135317) (width 1.016) (layer B.Cu) (net 5))
+  (segment (start 155.396318 57.15) (end 153.943999 58.602319) (width 1.016) (layer B.Cu) (net 5))
+  (segment (start 161.925 57.15) (end 155.396318 57.15) (width 1.016) (layer B.Cu) (net 5))
+  (segment (start 122.785 101.6) (end 119.305 105.08) (width 1.016) (layer B.Cu) (net 6))
+  (segment (start 189.23 101.6) (end 122.785 101.6) (width 1.016) (layer B.Cu) (net 6))
+  (segment (start 105.977081 56.515) (end 104.775 56.515) (width 1.016) (layer B.Cu) (net 7))
+  (segment (start 109.858082 60.396001) (end 105.977081 56.515) (width 1.016) (layer B.Cu) (net 7))
+  (segment (start 127.274786 60.396001) (end 109.858082 60.396001) (width 1.016) (layer B.Cu) (net 7))
+  (segment (start 127.990787 59.68) (end 127.274786 60.396001) (width 1.016) (layer B.Cu) (net 7))
+  (segment (start 129.405 59.68) (end 127.990787 59.68) (width 1.016) (layer B.Cu) (net 7))
+  (segment (start 101.385001 65.825001) (end 102.235 66.675) (width 1.016) (layer B.Cu) (net 7))
+  (segment (start 101.163319 65.825001) (end 101.385001 65.825001) (width 1.016) (layer B.Cu) (net 7))
+  (segment (start 100.368999 65.030681) (end 101.163319 65.825001) (width 1.016) (layer B.Cu) (net 7))
+  (segment (start 100.368999 58.159319) (end 100.368999 65.030681) (width 1.016) (layer B.Cu) (net 7))
+  (segment (start 101.339319 57.188999) (end 100.368999 58.159319) (width 1.016) (layer B.Cu) (net 7))
+  (segment (start 101.561001 57.188999) (end 101.339319 57.188999) (width 1.016) (layer B.Cu) (net 7))
+  (segment (start 102.235 56.515) (end 101.561001 57.188999) (width 1.016) (layer B.Cu) (net 7))
+  (segment (start 104.775 56.515) (end 102.235 56.515) (width 1.016) (layer B.Cu) (net 7))
+  (segment (start 104.775 66.675) (end 102.235 66.675) (width 1.016) (layer B.Cu) (net 7))
+  (segment (start 105.977081 59.055) (end 104.775 59.055) (width 1.016) (layer B.Cu) (net 8))
+  (segment (start 106.361807 59.055) (end 105.977081 59.055) (width 1.016) (layer B.Cu) (net 8))
+  (segment (start 109.226818 61.920011) (end 106.361807 59.055) (width 1.016) (layer B.Cu) (net 8))
+  (segment (start 131.079202 61.920011) (end 109.226818 61.920011) (width 1.016) (layer B.Cu) (net 8))
+  (segment (start 131.905 61.094213) (end 131.079202 61.920011) (width 1.016) (layer B.Cu) (net 8))
+  (segment (start 131.905 59.68) (end 131.905 61.094213) (width 1.016) (layer B.Cu) (net 8))
+  (segment (start 104.775 59.055) (end 102.235 59.055) (width 1.016) (layer B.Cu) (net 8))
+  (zone (net 7) (net_name "Net-(J4-Pad1)") (layer B.Cu) (hatch edge 0.508)
+    (connect_pads (clearance 1.016))
+    (min_thickness 0.254)
+    (fill yes (arc_segments 32) (thermal_gap 0.508) (thermal_bridge_width 0.508))
+    (polygon
+      (pts
+        (xy 97.79 52.07) (xy 197.485 52.07) (xy 197.485 121.92) (xy 97.79 121.92)
+      )
+    )
+  )
 )

Commit message: home
Parts:
- removed F1: 100mA, MyStuff:FuseHolder_Cylinder-27x8.5mm_Horizontal
- added J5: Mech support, Connector_PinHeader_2.54mm:PinHeader_2x05_P2.54mm_Vertical, F.Cu at (102.2, 108.6)
- J3: footprint Connector_Phoenix_MC_HighVoltage:PhoenixContact_MC_1,5_3-G-5.08_1x03_P5.08mm_Horizontal -> MyStuff:IEC60320_2pin
- moved PS1 61.8 mm to (177.8, 114.8), turned to 90 degrees
- moved J2 26.3 mm to (136.4, 70.5)
- moved J3 19.9 mm to (187.1, 86.9), turned to 270 degrees
- moved J1 7.62 mm to (195.1, 80.3)
- moved J4 1.27 mm to (102.2, 55.2)
Connections:
- J2 pad 1: Net-(F1-Pad1) -> Net-(J2-Pad1)
- J3 pad 1: Net-(J3-Pad1) -> LINE
- K1 pad 1: Net-(F1-Pad1) -> Net-(J2-Pad1)
- PS1 pad 2: Net-(F1-Pad2) -> Net-(J2-Pad1)
Routing:
- net LINE: track 73.0 -> 0.00 mm
- net NEUT: track 71.4 -> 0.00 mm
- net Net-(J1-Pad2): track 50.4 -> 0.00 mm
- net Net-(J4-Pad1): track 43.6 -> 0.00 mm
- net Net-(F1-Pad2): track 41.4 -> 0.00 mm
- net Net-(J1-Pad1): track 41.3 -> 0.00 mm
- net Net-(J4-Pad3): track 32.6 -> 0.00 mm
- net Net-(F1-Pad1): track 24.3 -> 0.00 mm
- removed copper zone on B.Cu, net Net-(J4-Pad1)

Commit message: home
Parts:
- moved J2 45.1 mm to (166.4, 104.1), turned to 0 degrees
- moved K1 36.7 mm to (132.5, 99.7), turned to -90 degrees
- moved J1 28.1 mm to (190.5, 108.0), turned to 90 degrees
- moved PS1 27.5 mm to (177.0, 87.3)
- moved J3 7.64 mm to (187.6, 79.2)
Connections:
- net Net-(J4-Pad1) renamed GNDREF
- J3 pad 1: LINE -> NEUT
- J3 pad 2: NEUT -> LINE
- J4 pad 5: Net-(J4-Pad5) -> unconnected-(J4-Pad5)
- J4 pad 6: Net-(J4-Pad6) -> unconnected-(J4-Pad6)
- J4 pad 7: Net-(J4-Pad7) -> unconnected-(J4-Pad7)
- J4 pad 8: Net-(J4-Pad8) -> unconnected-(J4-Pad8)
- J5 pad 1: Net-(J5-Pad1) -> unconnected-(J5-Pad1)
- J5 pad 10: Net-(J5-Pad10) -> unconnected-(J5-Pad10)
- J5 pad 2: Net-(J5-Pad2) -> unconnected-(J5-Pad2)
- J5 pad 3: Net-(J5-Pad3) -> unconnected-(J5-Pad3)
- J5 pad 4: Net-(J5-Pad4) -> unconnected-(J5-Pad4)
- J5 pad 5: Net-(J5-Pad5) -> unconnected-(J5-Pad5)
- J5 pad 6: Net-(J5-Pad6) -> unconnected-(J5-Pad6)
- J5 pad 7: Net-(J5-Pad7) -> unconnected-(J5-Pad7)
- J5 pad 8: Net-(J5-Pad8) -> unconnected-(J5-Pad8)
- J5 pad 9: Net-(J5-Pad9) -> unconnected-(J5-Pad9)
- K1 pad 2: Net-(K1-Pad2) -> unconnected-(K1-Pad2)
Routing:
- net Net-(J1-Pad2): track 0.00 -> 69.0 mm
- net Net-(J2-Pad1): track 0.00 -> 57.6 mm
- net Net-(J1-Pad1): track 0.00 -> 47.3 mm
- net LINE: track 0.00 -> 46.6 mm
- net GNDREF: track 0.00 -> 33.0 mm
- net NEUT: track 0.00 -> 29.2 mm
- net Net-(J4-Pad3): track 0.00 -> 22.2 mm
- added copper zone on F.Cu, net (none)
- added copper zone on F.Cu, net GNDREF
Other:
- net class Default removed
