File: KiCAD files/4051prog/4051prog.kicad_sch (KiCad schematic)
At the start: 14 parts

Commit message: office
Parts:
- added PS1: 5_to_12V, Converter_DCDC:Converter_DCDC_Murata_MEE1SxxxxSC_THT, symbol Converter_DCDC:MEE1S0303SC
- gave numbers to parts that had none: 14
Connections:
- net +5V: now also PS1.2 (+Vin)
- net GND: now also PS1.1 (-Vin), PS1.3 (-Vout)
- net 12V: now reaches Q2.3 (E)
- net 12V: now also PS1.4 (+Vout)
- net ENABLE_14V renamed ENABLE_12V
