File: KiCAD files/PX051/Px051_frontal/Px051_frontal.kicad_pcb (KiCad board)
At the start: 2 copper layers, 3 parts, among them J1 Conn_01x20_Male, U1 AT89C4051-24P

Commit message: office
Parts:
- added J7: fixing bolt, Connector_PinHeader_2.54mm:PinHeader_1x01_P2.54mm_Vertical, F.Cu at (264.2, 49.5)
- added J8: fixing bolt, Connector_PinHeader_2.54mm:PinHeader_1x01_P2.54mm_Vertical, F.Cu at (264.2, 109.2)
- moved U1 132.9 mm to (258.0, 68.0)
- moved J1 127.8 mm to (272.7, 55.2)
- moved C1 109.0 mm to (268.6, 68.7), turned to 90 degrees
Connections:
- C1 pad 2: Net-(C1-Pad2) -> GND
- J1 pad 18: Net-(J1-Pad18) -> GND
- J1 pad 20: Net-(C1-Pad2) -> Net-(J1-Pad20)
- U1 pad 10: Net-(J1-Pad18) -> GND
- U1 pad 8: Net-(C1-Pad2) -> Net-(J1-Pad20)
Routing:
- net GND: track 0.00 -> 75.5 mm, vias 0 -> 4
- net Net-(C1-Pad2): track 37.7 -> 0.00 mm
- net Net-(J1-Pad20): track 0.00 -> 34.3 mm
- net Net-(J1-Pad18): track 22.9 -> 0.00 mm
- net Net-(J1-Pad9): track 12.2 -> 7.08 mm
- net Net-(J1-Pad7): track 12.2 -> 7.08 mm
- net Net-(J1-Pad14): track 12.2 -> 7.08 mm
- net Net-(J1-Pad12): track 12.2 -> 7.08 mm
- net Net-(J1-Pad10): track 12.2 -> 7.08 mm
- net Net-(J1-Pad8): track 12.2 -> 7.08 mm
- net Net-(J1-Pad15): track 12.2 -> 7.08 mm
- net Net-(J1-Pad17): track 29.5 -> 24.4 mm
- net Net-(J1-Pad13): track 12.2 -> 7.08 mm
- net Net-(J1-Pad11): track 12.2 -> 7.08 mm
- net Net-(J1-Pad16): track 30.2 -> 25.1 mm
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- added copper zone on B.Cu, net GND
Other:
- board outline added: 24.8 x 80 mm
- board text added: "ADDR"
- board text added: "Design by Kaltchuk 2021"
- board text added: "PX051"
