File: KiCAD files/PX051/Px051_frontal/Px051_frontal.kicad_sch (KiCad schematic)
At the start: 3 parts, among them J1 Conn_01x20_Male, U1 AT89C4051-24P

Commit message: office
Connections:
- net GND: now reaches J1.18 (Pin_18), U1.10 (GND)
- net GND: now also C1.2
- net at J1.20 (Pin_20), U1.8 (P3.4): no longer C1.2
Changed lines of the file:
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@@
 (kicad_sch (version 20211123) (generator eeschema)
   (paper "A4")
-  (junction (at 193.04 118.11) (diameter 0) (color 0 0 0 0)
-  )
   (junction (at 165.1 52.07) (diameter 0) (color 0 0 0 0)
   )
+  (junction (at 187.96 113.03) (diameter 0) (color 0 0 0 0)
+  )
   (wire (pts (xy 134.62 115.57) (xy 190.5 115.57))
     (stroke (width 0) (type default) (color 0 0 0 0))
@@
     (stroke (width 0) (type default) (color 0 0 0 0))
   )
-  (wire (pts (xy 209.55 52.07) (xy 209.55 118.11))
+  (wire (pts (xy 209.55 52.07) (xy 209.55 113.03))
     (stroke (width 0) (type default) (color 0 0 0 0))
   )
@@
     (stroke (width 0) (type default) (color 0 0 0 0))
   )
+  (wire (pts (xy 187.96 113.03) (xy 209.55 113.03))
+    (stroke (width 0) (type default) (color 0 0 0 0))
+  )
   (wire (pts (xy 182.88 107.95) (xy 182.88 100.33))
     (stroke (width 0) (type default) (color 0 0 0 0))
@@
   )
   (wire (pts (xy 185.42 102.87) (xy 193.04 102.87))
-    (stroke (width 0) (type default) (color 0 0 0 0))
-  )
-  (wire (pts (xy 209.55 118.11) (xy 193.04 118.11))
     (stroke (width 0) (type default) (color 0 0 0 0))
   )
@@
     (pin "2")
   )
+  (symbol (lib_id "power:GND") (at 114.3 113.03 0) (unit 1)
+    (in_bom yes) (on_board yes) (fields_autoplaced)
+    (property "Reference" "#PWR?" (id 0) (at 114.3 119.38 0)
+      (effects (font (size 1.27 1.27)) hide)
+    )
+    (property "Value" "GND" (id 1) (at 114.3 118.11 0))
+    (property "Footprint" "" (id 2) (at 114.3 113.03 0)
+      (effects (font (size 1.27 1.27)) hide)
+    )
+    (property "Datasheet" "" (id 3) (at 114.3 113.03 0)
+      (effects (font (size 1.27 1.27)) hide)
+    )
+    (pin "1")
+  )
   (symbol (lib_id "Connector:Conn_01x20_Male") (at 198.12 85.09 0) (mirror y) (unit 1)
     (in_bom yes) (on_board yes) (fields_autoplaced)
@@
   )
   (symbol_instances
+    (path "/84c6ade4-472b-49ab-bf5d-7989d8cac908"
+      (reference "#PWR?") (unit 1) (value "GND") (footprint "")
+    )
     (path "/3b5cbb6d-677b-4641-88bd-7044bfd6bfae"
       (reference "C1") (unit 1) (value "10nF") (footprint "Capacitor_THT:C_Disc_D3.0mm_W2.0mm_P2.50mm")
