File: KiCAD files/stickers/stickers.kicad_pcb (KiCad board)
At the start: 2 copper layers, 0 parts

Commit message: HOME
Routing:
- net (no net): vias 902 -> 1132
Other:
- board text added: "ARDUINO NANO"
- board text added: "USB"

Commit message: home
Routing:
- net (no net): vias 1132 -> 956
Other:
- net class Default removed
- board text removed: "+12V"
- board text removed: "+5V"
- board text removed: "0"
- board text removed: "A"
- board text removed: "BSAK"
- board text removed: "BSRQ"
- board text removed: "BUSAK"
- board text removed: "BUSRQ"
- board text removed: "CLK"
- board text removed: "D"
- board text removed: "GND"
- board text removed: "HALT"
- board text removed: "INT"
- board text removed: "IORQ"
- board text removed: "M1"
- board text removed: "MREQ"
- board text removed: "NMI"
- board text removed: "R"
- board text removed: "RD"
- board text removed: "RESET"
- board text removed: "RFSH"
- board text removed: "S0"
- board text removed: "S1"
- board text removed: "T"
- board text removed: "V1"
- board text removed: "WAIT"
- board text removed: "WR"

Commit message: home
Routing:
- net (no net): vias 956 -> 1024
Other:
- board text added: "0"
