File: KiCAD files/I2C/I2C.kicad_sch (KiCad schematic)
At the start: 25 parts, among them J1 card addr, J2 Power Bus, J3 Signal Bus, U1 74LS85, U3 AT89C4051-24P, U4 74LS74, U5 DS1307+, U6 FM24C64B

Commit message: HOME
Parts:
- removed U2: (no value), symbol 74xx:74LS00
- added C1: 10nF, symbol Device:C
- added C?: 10nF, Capacitor_THT:C_Disc_D3.8mm_W2.6mm_P2.50mm, symbol Device:C
- added U? (x4): (no value), symbol 74xx:74LS04
- added U? (x2): (no value), symbol 74xx:74LS08
- added U?: 74LS245, Package_DIP:DIP-20_W7.62mm_Socket_LongPads, symbol 74xx:74LS245
- BT1: renamed from BT?; value (none) -> 3V
- C8: renamed from C7; value (none) -> 33pF
- C9: renamed from C8; value (none) -> 33pF
- J4: value (none) -> I2C ext
- R1, R2: value (none) -> 4k7
- Y1: value (none) -> 24MHz
- Y2: value (none) -> 32.768kHz
- renumbered C1 to C2, C2 to C3, C3 to C4, C4 to C5, C5 to C6, C6 to C7
Connections:
- net +5V: now also C1.1, C?.1, U?.14 (VCC), U?.14 (VCC), U?.20 (VCC)
- net GND: now also C1.2, C?.2, U?.10 (GND), U?.7 (GND), U?.7 (GND)
- net d00: now also U?.2 (A0); no longer RN2.2 (R1), U3.12 (P1.0)
- net d01: now also U?.3 (A1); no longer RN2.3 (R2), U3.13 (P1.1)
- net d02: now also U?.4 (A2); no longer U3.14 (P1.2)
- net d03: now also U?.5 (A3); no longer U3.15 (P1.3)
- net d04: now also U?.6 (A4); no longer U3.16 (P1.4)
- net d05: now also U?.7 (A5); no longer U3.17 (P1.5)
- net d06: now also U?.8 (A6); no longer U3.18 (P1.6)
- net d07: now also U?.9 (A7); no longer U3.19 (P1.7)
- net iorq: now also U?.3
- net rd: now also U?.1 (A->B)
- net reset: now also U?.1, U?.1
- net at RN2.4 (R3), U3.2 (P3.0): now also U?.2
- net at U1.3 (Ia=b): now also U?.4
- net at U1.6 (Oa=b), U3.3 (P3.1), U4.3 (C): now also U?.5
- net at U4.1 (~{R}): now also U?.3
- net at U3.1 (RST/VPP): now also U?.2
- new net: U?.19 (CE), U?.6
- new net B00: RN2.2 (R1), U3.12 (P1.0), U?.18 (B0)
- new net B01: RN2.3 (R2), U3.13 (P1.1), U?.17 (B1)
- new net B02: U3.14 (P1.2), U?.16 (B2)
- new net B03: U3.15 (P1.3), U?.15 (B3)
- new net B04: U3.16 (P1.4), U?.14 (B4)
- new net B05: U3.17 (P1.5), U?.13 (B5)
- new net B06: U3.18 (P1.6), U?.12 (B6)
- new net B07: U3.19 (P1.7), U?.11 (B7)
Other:
- moved on the sheet: C2, C3, C5, C6, C7

Commit message: office
Parts:
- removed C?: 10nF, Capacitor_THT:C_Disc_D3.8mm_W2.6mm_P2.50mm, symbol Device:C
- added C2: 10nF, symbol Device:C
- U2: renamed from U?; value (none) -> 74LS04
- U3: renamed from U?; value (none) -> 74LS08
- gave numbers to parts that had none: 1
- renumbered C9 to C10, C2 to C3, C5 to C4, C3 to C5, C4 to C8, C8 to C9, U3 to U5, U4 to U6, U5 to U7, U6 to U8
Connections:
- net +5V: now also J4.2 (Pin_2), C2.1; no longer J4.1 (Pin_1)
- net GND: now also J4.4 (Pin_4), C2.2; no longer J4.3 (Pin_3)
- net at R2.1, U5.8 (P3.4), U7.5 (SDA)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: now also J4.1 (Pin_1); no longer J4.2 (Pin_2)
- net at R1.1, U5.9 (P3.5), U7.6 (SCL)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: now also J4.3 (Pin_3); no longer J4.4 (Pin_4)
Other:
- moved on the sheet: C1, C3, C4, C5, C6, C7

Commit message: office
Parts:
- added C7: 10nF, symbol Device:C
- renumbered C9 to C10, C10 to C11, C7 to C8, C8 to C9
Connections:
- net +5V: now also C7.1
- net GND: now also C7.2

Commit message: home
Parts:
- added unit 3 of U2
- renumbered U6 to U2, U2 to U3, U3 to U4, U4 to U5, U5 to U6
Connections:
- net +5V: now also U2.14 (VCC)
- net GND: now also U2.7 (GND)
- net +BATT: now reaches BT1.1 (+), U7.3 (VBAT)
Other:
- moved on the sheet: BT1, U3G, U4E

Commit message: office
Parts:
- U2: value (none) -> 74LS74
Connections:
- net rd: no longer U6.6 (P3.2)
- net wr: now also U6.3 (P3.1); no longer U6.7 (P3.3)
- net card_sel: now reaches U1.6 (Oa=b), U2.3 (C), U3.5
- net card_sel: no longer U6.3 (P3.1)
- net at U3.6, U5.19 (CE): now also U6.6 (P3.2)
- no-connect marks 5 -> 6
Other:
- moved on the sheet: U3C

Commit message: updates i2c card
Parts:
- U2, U3, U4: footprint (none) -> Package_DIP:DIP-14_W7.62mm_Socket_LongPads
- U6: footprint Package_DIP:DIP-20_W7.62mm -> Package_DIP:DIP-20_W7.62mm_LongPads
- U7: footprint Package_DIP:DIP-8_W7.62mm -> Package_DIP:DIP-8-16_W7.62mm_Socket_LongPads
- U8: footprint Package_SO:SOIC-8_3.9x4.9mm_P1.27mm -> Package_DIP:DIP-8-16_W7.62mm_Socket_LongPads
Changed lines of the file:
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@@
       (effects (font (size 1.27 1.27)) (justify left))
     )
-    (property "Footprint" "" (id 2) (at 88.9 172.72 0)
+    (property "Footprint" "Package_DIP:DIP-14_W7.62mm_Socket_LongPads" (id 2) (at 88.9 172.72 0)
       (effects (font (size 1.27 1.27)) hide)
     )
@@
     (property "Reference" "U3" (id 0) (at 142.24 29.21 0))
     (property "Value" "74LS04" (id 1) (at 142.24 31.75 0))
-    (property "Footprint" "" (id 2) (at 142.24 38.1 0)
+    (property "Footprint" "Package_DIP:DIP-14_W7.62mm_Socket_LongPads" (id 2) (at 142.24 38.1 0)
       (effects (font (size 1.27 1.27)) hide)
     )
@@
       (effects (font (size 1.27 1.27)) (justify right))
     )
-    (property "Footprint" "Package_SO:SOIC-8_3.9x4.9mm_P1.27mm" (id 2) (at 248.92 135.89 0)
+    (property "Footprint" "Package_DIP:DIP-8-16_W7.62mm_Socket_LongPads" (id 2) (at 248.92 135.89 0)
       (effects (font (size 1.27 1.27)) hide)
     )
@@
       (effects (font (size 1.27 1.27)) (justify left))
     )
-    (property "Footprint" "" (id 2) (at 142.24 172.72 0)
+    (property "Footprint" "Package_DIP:DIP-14_W7.62mm_Socket_LongPads" (id 2) (at 142.24 172.72 0)
       (effects (font (size 1.27 1.27)) hide)
     )
@@
     (property "Reference" "U3" (id 0) (at 121.92 130.81 0))
     (property "Value" "74LS04" (id 1) (at 123.19 138.43 0))
-    (property "Footprint" "" (id 2) (at 119.38 134.62 0)
+    (property "Footprint" "Package_DIP:DIP-14_W7.62mm_Socket_LongPads" (id 2) (at 119.38 134.62 0)
       (effects (font (size 1.27 1.27)) hide)
     )
@@
       (effects (font (size 1.27 1.27)) (justify left))
     )
-    (property "Footprint" "" (id 2) (at 115.57 172.72 0)
+    (property "Footprint" "Package_DIP:DIP-14_W7.62mm_Socket_LongPads" (id 2) (at 115.57 172.72 0)
       (effects (font (size 1.27 1.27)) hide)
     )
@@
     (property "Reference" "U3" (id 0) (at 119.38 114.3 0))
     (property "Value" "74LS04" (id 1) (at 119.38 116.84 0))
-    (property "Footprint" "" (id 2) (at 119.38 123.19 0)
+    (property "Footprint" "Package_DIP:DIP-14_W7.62mm_Socket_LongPads" (id 2) (at 119.38 123.19 0)
       (effects (font (size 1.27 1.27)) hide)
     )
@@
       (effects (font (size 1.27 1.27)) (justify left))
     )
-    (property "Footprint" "Package_DIP:DIP-20_W7.62mm" (id 2) (at 179.07 58.42 0)
+    (property "Footprint" "Package_DIP:DIP-20_W7.62mm_LongPads" (id 2) (at 179.07 58.42 0)
       (effects (font (size 1.27 1.27) italic) hide)
     )
@@
     (property "Reference" "U4" (id 0) (at 222.25 49.53 0))
     (property "Value" "74LS08" (id 1) (at 222.25 52.07 0))
-    (property "Footprint" "" (id 2) (at 222.25 58.42 0)
+    (property "Footprint" "Package_DIP:DIP-14_W7.62mm_Socket_LongPads" (id 2) (at 222.25 58.42 0)
       (effects (font (size 1.27 1.27)) hide)
     )
@@
     (property "Reference" "U7" (id 0) (at 265.43 94.7293 0))
     (property "Value" "DS1307+" (id 1) (at 265.43 97.2693 0))
-    (property "Footprint" "Package_DIP:DIP-8_W7.62mm" (id 2) (at 248.92 111.76 0)
+    (property "Footprint" "Package_DIP:DIP-8-16_W7.62mm_Socket_LongPads" (id 2) (at 248.92 111.76 0)
       (effects (font (size 1.27 1.27)) hide)
     )
@@
     )
     (path "/1b77c8f9-b0fa-45ba-a726-522a68924cf1"
-      (reference "U2") (unit 3) (value "74LS74") (footprint "")
+      (reference "U2") (unit 3) (value "74LS74") (footprint "Package_DIP:DIP-14_W7.62mm_Socket_LongPads")
     )
     (path "/1c4ac060-9b7c-464c-89d2-0f5fc60c549c"
-      (reference "U3") (unit 1) (value "74LS04") (footprint "")
+      (reference "U3") (unit 1) (value "74LS04") (footprint "Package_DIP:DIP-14_W7.62mm_Socket_LongPads")
     )
     (path "/aafc2e46-7f62-46ec-bcbf-65d78307e655"
-      (reference "U3") (unit 2) (value "74LS04") (footprint "")
+      (reference "U3") (unit 2) (value "74LS04") (footprint "Package_DIP:DIP-14_W7.62mm_Socket_LongPads")
     )
     (path "/4c6e3e1a-9c98-4aaf-845f-eaa1c889def3"
-      (reference "U3") (unit 3) (value "74LS04") (footprint "")
+      (reference "U3") (unit 3) (value "74LS04") (footprint "Package_DIP:DIP-14_W7.62mm_Socket_LongPads")
     )
     (path "/a546fa6d-0a9e-4d6e-9625-024ec2fb5616"
-      (reference "U3") (unit 7) (value "74LS04") (footprint "")
+      (reference "U3") (unit 7) (value "74LS04") (footprint "Package_DIP:DIP-14_W7.62mm_Socket_LongPads")
     )
     (path "/de1dbb83-7195-47d7-b2ab-8db8131a53e5"
-      (reference "U4") (unit 1) (value "74LS08") (footprint "")
+      (reference "U4") (unit 1) (value "74LS08") (footprint "Package_DIP:DIP-14_W7.62mm_Socket_LongPads")
     )
     (path "/3d23d636-1fd4-4656-9a01-402e61a0136f"
-      (reference "U4") (unit 5) (value "74LS08") (footprint "")
+      (reference "U4") (unit 5) (value "74LS08") (footprint "Package_DIP:DIP-14_W7.62mm_Socket_LongPads")
     )
     (path "/b127cdd2-34c3-48a5-b6b1-4554e51b506e"
@@
     )
     (path "/d5c459c9-9d6e-4eae-816f-63a1560a1c47"
-      (reference "U6") (unit 1) (value "AT89C4051-24P") (footprint "Package_DIP:DIP-20_W7.62mm")
+      (reference "U6") (unit 1) (value "AT89C4051-24P") (footprint "Package_DIP:DIP-20_W7.62mm_LongPads")
     )
     (path "/f26c481d-d67e-4482-a7d9-6f79748d485a"
-      (reference "U7") (unit 1) (value "DS1307+") (footprint "Package_DIP:DIP-8_W7.62mm")
+      (reference "U7") (unit 1) (value "DS1307+") (footprint "Package_DIP:DIP-8-16_W7.62mm_Socket_LongPads")
     )
     (path "/28ced857-2be2-4629-b12a-4bdeab4d4ff1"
-      (reference "U8") (unit 1) (value "FM24C64B") (footprint "Package_SO:SOIC-8_3.9x4.9mm_P1.27mm")
+      (reference "U8") (unit 1) (value "FM24C64B") (footprint "Package_DIP:DIP-8-16_W7.62mm_Socket_LongPads")
     )
     (path "/29af8fa6-318a-4068-993d-88e7a24f7791"

Commit message: `pcbsm
Parts:
- added J5: I2C ext, symbol Connector_Generic:Conn_02x02_Top_Bottom
- J4: value I2C ext -> I2C int
- R1, R2: value 4k7 -> 6k8
Connections:
- net +5V: now also J5.3 (Pin_3)
- net GND: now also J5.4 (Pin_4)
- net SDA: now reaches J4.1 (Pin_1), R2.1, U6.8 (P3.4), U7.5 (SDA), U8.5 (SDA)
- net SDA: now also J5.1 (Pin_1)
- net SCL: now reaches J4.3 (Pin_3), R1.1, U6.9 (P3.5), U7.6 (SCL), U8.6 (SCL)
- net SCL: now also J5.2 (Pin_2)
Other:
- moved on the sheet: J4

Commit message: PCBs
Parts:
- added H1, H2: (no value), symbol Mechanical:MountingHole
- BT1: footprint (none) -> MyStuff:Battery-Holder_CR2032
- C1, C10, C11, C2, C3, C4, C5, C6, C7, C8: footprint (none) -> Capacitor_THT:C_Disc_D3.8mm_W2.6mm_P2.50mm
- J4: footprint (none) -> Connector_PinHeader_2.54mm:PinHeader_1x04_P2.54mm_Vertical
- J5: footprint (none) -> Connector_PinHeader_2.54mm:PinHeader_2x02_P2.54mm_Vertical
- R1, R2: footprint (none) -> Resistor_THT:R_Axial_DIN0207_L6.3mm_D2.5mm_P10.16mm_Horizontal
- U6: footprint Package_DIP:DIP-20_W7.62mm_LongPads -> Package_DIP:DIP-20_W7.62mm_Socket_LongPads
- U7, U8: footprint Package_DIP:DIP-8-16_W7.62mm_Socket_LongPads -> Package_DIP:DIP-8_W7.62mm_Socket_LongPads
- Y1: footprint (none) -> Crystal:Crystal_HC49-U_Vertical
- Y2: footprint (none) -> Crystal:Crystal_Round_D1.5mm_Vertical
Changed lines of the file:
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@@
     (property "Reference" "J5" (id 0) (at 264.16 66.04 0))
     (property "Value" "I2C ext" (id 1) (at 264.16 68.58 0))
-    (property "Footprint" "" (id 2) (at 262.89 72.39 0)
+    (property "Footprint" "Connector_PinHeader_2.54mm:PinHeader_2x02_P2.54mm_Vertical" (id 2) (at 262.89 72.39 0)
       (effects (font (size 1.27 1.27)) hide)
     )
@@
       (effects (font (size 1.27 1.27)) (justify left))
     )
-    (property "Footprint" "" (id 2) (at 150.8252 60.96 0)
+    (property "Footprint" "Capacitor_THT:C_Disc_D3.8mm_W2.6mm_P2.50mm" (id 2) (at 150.8252 60.96 0)
       (effects (font (size 1.27 1.27)) hide)
     )
@@
       (effects (font (size 1.27 1.27)) (justify left))
     )
-    (property "Footprint" "" (id 2) (at 162.2552 60.96 0)
+    (property "Footprint" "Capacitor_THT:C_Disc_D3.8mm_W2.6mm_P2.50mm" (id 2) (at 162.2552 60.96 0)
       (effects (font (size 1.27 1.27)) hide)
     )
@@
     )
     (pin "1")
+  )
+  (symbol (lib_id "Mechanical:MountingHole") (at 195.58 160.02 0) (unit 1)
+    (in_bom yes) (on_board yes) (fields_autoplaced)
+    (property "Reference" "H1" (id 0) (at 198.12 160.0199 0)
+      (effects (font (size 1.27 1.27)) (justify left))
+    )
+    (property "Value" "" (id 1) (at 198.12 161.2899 0)
+      (effects (font (size 1.27 1.27)) (justify left) hide)
+    )
+    (property "Footprint" "" (id 2) (at 195.58 160.02 0)
+      (effects (font (size 1.27 1.27)) hide)
+    )
+    (property "Datasheet" "~" (id 3) (at 195.58 160.02 0)
+      (effects (font (size 1.27 1.27)) hide)
+    )
   )
   (symbol (lib_id "74xx:74LS74") (at 88.9 172.72 0) (unit 3)
@@
       (effects (font (size 1.27 1.27)) (justify right))
     )
-    (property "Footprint" "" (id 2) (at 240.03 71.12 0)
+    (property "Footprint" "Connector_PinHeader_2.54mm:PinHeader_1x04_P2.54mm_Vertical" (id 2) (at 240.03 71.12 0)
       (effects (font (size 1.27 1.27)) hide)
     )
@@
       (effects (font (size 1.27 1.27)) (justify right))
     )
-    (property "Footprint" "Package_DIP:DIP-8-16_W7.62mm_Socket_LongPads" (id 2) (at 248.92 135.89 0)
+    (property "Footprint" "Package_DIP:DIP-8_W7.62mm_Socket_LongPads" (id 2) (at 248.92 135.89 0)
       (effects (font (size 1.27 1.27)) hide)
     )
@@
     (property "Reference" "Y1" (id 0) (at 156.21 44.45 0))
     (property "Value" "24MHz" (id 1) (at 156.21 52.07 0))
-    (property "Footprint" "" (id 2) (at 156.21 48.26 0)
+    (property "Footprint" "Crystal:Crystal_HC49-U_Vertical" (id 2) (at 156.21 48.26 0)
       (effects (font (size 1.27 1.27)) hide)
     )
@@
       (effects (font (size 1.27 1.27)) (justify right))
     )
-    (property "Footprint" "" (id 2) (at 231.14 104.14 0)
+    (property "Footprint" "Crystal:Crystal_Round_D1.5mm_Vertical" (id 2) (at 231.14 104.14 0)
       (effects (font (size 1.27 1.27)) hide)
     )
@@
       (effects (font (size 1.27 1.27)) (justify left))
     )
-    (property "Footprint" "" (id 2) (at 26.3652 180.34 0)
+    (property "Footprint" "Capacitor_THT:C_Disc_D3.8mm_W2.6mm_P2.50mm" (id 2) (at 26.3652 180.34 0)
       (effects (font (size 1.27 1.27)) hide)
     )
@@
     (property "Reference" "R2" (id 0) (at 208.28 128.27 90))
     (property "Value" "6k8" (id 1) (at 208.28 130.81 90))
-    (property "Footprint" "" (id 2) (at 208.28 135.128 90)
+    (property "Footprint" "Resistor_THT:R_Axial_DIN0207_L6.3mm_D2.5mm_P10.16mm_Horizontal" (id 2) (at 208.28 135.128 90)
       (effects (font (size 1.27 1.27)) hide)
     )
@@
       (effects (font (size 1.27 1.27)) (justify left))
     )
-    (property "Footprint" "" (id 2) (at 60.6552 180.34 0)
+    (property "Footprint" "Capacitor_THT:C_Disc_D3.8mm_W2.6mm_P2.50mm" (id 2) (at 60.6552 180.34 0)
       (effects (font (size 1.27 1.27)) hide)
     )
@@
       (effects (font (size 1.27 1.27)) (justify left))
     )
-    (property "Footprint" "" (id 2) (at 37.7952 180.34 0)
+    (property "Footprint" "Capacitor_THT:C_Disc_D3.8mm_W2.6mm_P2.50mm" (id 2) (at 37.7952 180.34 0)
       (effects (font (size 1.27 1.27)) hide)
     )
@@
       (effects (font (size 1.27 1.27)) (justify left))
     )
-    (property "Footprint" "" (id 2) (at 26.3652 153.67 0)
+    (property "Footprint" "Capacitor_THT:C_Disc_D3.8mm_W2.6mm_P2.50mm" (id 2) (at 26.3652 153.67 0)
       (effects (font (size 1.27 1.27)) hide)
     )
@@
     (property "Reference" "R1" (id 0) (at 199.39 140.97 90))
     (property "Value" "6k8" (id 1) (at 199.39 143.51 90))
-    (property "Footprint" "" (id 2) (at 199.39 140.208 90)
+    (property "Footprint" "Resistor_THT:R_Axial_DIN0207_L6.3mm_D2.5mm_P10.16mm_Horizontal" (id 2) (at 199.39 140.208 90)
       (effects (font (size 1.27 1.27)) hide)
     )
@@
     (pin "1")
   )
+  (symbol (lib_id "Mechanical:MountingHole") (at 203.2 160.02 0) (unit 1)
+    (in_bom yes) (on_board yes) (fields_autoplaced)
+    (property "Reference" "H2" (id 0) (at 205.74 160.0199 0)
+      (effects (font (size 1.27 1.27)) (justify left))
+    )
+    (property "Value" "" (id 1) (at 205.74 161.2899 0)
+      (effects (font (size 1.27 1.27)) (justify left) hide)
+    )
+    (property "Footprint" "" (id 2) (at 203.2 160.02 0)
+      (effects (font (size 1.27 1.27)) hide)
+    )
+    (property "Datasheet" "~" (id 3) (at 203.2 160.02 0)
+      (effects (font (size 1.27 1.27)) hide)
+    )
+  )
   (symbol (lib_id "power:GND") (at 261.62 143.51 0) (unit 1)
     (in_bom yes) (on_board yes) (fields_autoplaced)
@@
       (effects (font (size 1.27 1.27)) (justify left))
     )
-    (property "Footprint" "" (id 2) (at 37.7952 153.67 0)
+    (property "Footprint" "Capacitor_THT:C_Disc_D3.8mm_W2.6mm_P2.50mm" (id 2) (at 37.7952 153.67 0)
       (effects (font (size 1.27 1.27)) hide)
     )
@@
       (effects (font (size 1.27 1.27)) (justify left))
     )
-    (property "Footprint" "" (id 2) (at 60.6552 153.67 0)
+    (property "Footprint" "Capacitor_THT:C_Disc_D3.8mm_W2.6mm_P2.50mm" (id 2) (at 60.6552 153.67 0)
       (effects (font (size 1.27 1.27)) hide)
     )
@@
       (effects (font (size 1.27 1.27)) (justify left))
     )
-    (property "Footprint" "" (id 2) (at 49.2252 153.67 0)
+    (property "Footprint" "Capacitor_THT:C_Disc_D3.8mm_W2.6mm_P2.50mm" (id 2) (at 49.2252 153.67 0)
       (effects (font (size 1.27 1.27)) hide)
     )
@@
       (effects (font (size 1.27 1.27)) (justify left))
     )
-    (property "Footprint" "" (id 2) (at 49.2252 180.34 0)
+    (property "Footprint" "Capacitor_THT:C_Disc_D3.8mm_W2.6mm_P2.50mm" (id 2) (at 49.2252 180.34 0)
       (effects (font (size 1.27 1.27)) hide)
     )
@@
     (property "Reference" "BT1" (id 0) (at 40.64 87.63 0))
     (property "Value" "3V" (id 1) (at 35.56 87.63 0))
-    (property "Footprint" "" (id 2) (at 38.1 84.836 90)
+    (property "Footprint" "MyStuff:Battery-Holder_CR2032" (id 2) (at 38.1 84.836 90)
       (effects (font (size 1.27 1.27)) hide)
     )
@@
       (effects (font (size 1.27 1.27)) (justify left))
     )
-    (property "Footprint" "Package_DIP:DIP-20_W7.62mm_LongPads" (id 2) (at 179.07 58.42 0)
+    (property "Footprint" "Package_DIP:DIP-20_W7.62mm_Socket_LongPads" (id 2) (at 179.07 58.42 0)
       (effects (font (size 1.27 1.27) italic) hide)
     )
@@
     (property "Reference" "U7" (id 0) (at 265.43 94.7293 0))
     (property "Value" "DS1307+" (id 1) (at 265.43 97.2693 0))
-    (property "Footprint" "Package_DIP:DIP-8-16_W7.62mm_Socket_LongPads" (id 2) (at 248.92 111.76 0)
+    (property "Footprint" "Package_DIP:DIP-8_W7.62mm_Socket_LongPads" (id 2) (at 248.92 111.76 0)
       (effects (font (size 1.27 1.27)) hide)
     )
@@
     )
     (path "/c5efa317-c6ad-413e-90a3-f14d4c9780e5"
-      (reference "BT1") (unit 1) (value "3V") (footprint "Battery:Battery_Panasonic_CR2032-VS1N_Vertical_CircularHoles")
+      (reference "BT1") (unit 1) (value "3V") (footprint "MyStuff:Battery-Holder_CR2032")
     )
     (path "/8b14e97f-a7f6-455f-85ae-a0954b928855"
@@
       (reference "C11") (unit 1) (value "33pF") (footprint "Capacitor_THT:C_Disc_D3.8mm_W2.6mm_P2.50mm")
     )
+    (path "/1ad7167c-d842-43e1-aa03-616956653f99"
+      (reference "H1") (unit 1) (value "MountingHole") (footprint "MountingHole:MountingHole_3mm_Pad_TopBottom")
+    )
+    (path "/94cbfc13-d61a-4fdd-b97d-9f86f3a34f14"
+      (reference "H2") (unit 1) (value "MountingHole") (footprint "MountingHole:MountingHole_3mm_Pad_TopBottom")
+    )
     (path "/fff0ffa5-782c-4d4c-b7ca-701e7c5864bd"
       (reference "J1") (unit 1) (value "card addr") (footprint "Connector_PinHeader_2.54mm:PinHeader_2x04_P2.54mm_Vertical")
@@
     )
     (path "/d5c459c9-9d6e-4eae-816f-63a1560a1c47"
-      (reference "U6") (unit 1) (value "AT89C4051-24P") (footprint "Package_DIP:DIP-20_W7.62mm_LongPads")
+      (reference "U6") (unit 1) (value "AT89C4051-24P") (footprint "Package_DIP:DIP-20_W7.62mm_Socket_LongPads")
     )
     (path "/f26c481d-d67e-4482-a7d9-6f79748d485a"
-      (reference "U7") (unit 1) (value "DS1307+") (footprint "Package_DIP:DIP-8-16_W7.62mm_Socket_LongPads")
+      (reference "U7") (unit 1) (value "DS1307+") (footprint "Package_DIP:DIP-8_W7.62mm_Socket_LongPads")
     )
     (path "/28ced857-2be2-4629-b12a-4bdeab4d4ff1"
-      (reference "U8") (unit 1) (value "FM24C64B") (footprint "Package_DIP:DIP-8-16_W7.62mm_Socket_LongPads")
+      (reference "U8") (unit 1) (value "FM24C64B") (footprint "Package_DIP:DIP-8_W7.62mm_Socket_LongPads")
     )
     (path "/29af8fa6-318a-4068-993d-88e7a24f7791"
