File: KiCAD files/I2C/I2C.kicad_pcb (KiCad board)
At the start: 2 copper layers, 99.7 x 69.8 mm, 31 parts, among them J1 card addr, J2 Power Bus, J3 Signal Bus, J4 I2C int, J5 I2C ext, U1 74LS85, U2 74LS74, U3 74LS04, U4 74LS08, U5 74LS245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

Commit message: PCBs
Parts:
- added ?: , , F.Cu at (106.7, 106.2)
- added ?: , , F.Cu at (109.2, 106.2)
- added ?: , , F.Cu at (96.5, 106.2)
- added ?: , , F.Cu at (106.7, 113.8)
- added ?: , , F.Cu at (104.1, 113.8)
- added ?: , , F.Cu at (134.6, 101.1)
- added ?: , , F.Cu at (132.1, 116.3)
- added ?: , , F.Cu at (96.5, 116.3)
- added ?: , , F.Cu at (106.7, 118.9)
- added ?: , , F.Cu at (101.6, 103.6)
- added ?: , , F.Cu at (132.1, 118.9)
- added ?: , , F.Cu at (99.1, 116.3)
- added ?: , , F.Cu at (101.6, 113.8)
- added ?: , , F.Cu at (129.5, 103.6)
- added ?: , , F.Cu at (101.6, 101.1)
- added ?: , , F.Cu at (101.6, 116.3)
- added ?: , , F.Cu at (124.5, 106.2)
- added ?: , , F.Cu at (127.0, 116.3)
- added ?: , , F.Cu at (106.7, 103.6)
- added ?: , , F.Cu at (116.8, 116.3)
- added ?: , , F.Cu at (111.8, 118.9)
- added ?: , , F.Cu at (127.0, 118.9)
- added ?: , , F.Cu at (104.1, 116.3)
- added ?: , , F.Cu at (116.8, 113.8)
- added ?: , , F.Cu at (129.5, 113.8)
- added ?: , , F.Cu at (99.1, 101.1)
- added ?: , , F.Cu at (96.5, 113.8)
- added ?: , , F.Cu at (101.6, 106.2)
- added ?: , , F.Cu at (124.5, 118.9)
- added ?: , , F.Cu at (116.8, 106.2)
- added ?: , , F.Cu at (109.2, 116.3)
- added ?: , , F.Cu at (124.5, 113.8)
- added ?: , , F.Cu at (129.5, 101.1)
- added ?: , , F.Cu at (99.1, 103.6)
- added ?: , , F.Cu at (134.6, 103.6)
- added ?: , , F.Cu at (121.9, 118.9)
- added ?: , , F.Cu at (114.3, 106.2)
- added ?: , , F.Cu at (119.4, 116.3)
- added ?: , , F.Cu at (119.4, 113.8)
- added ?: , , F.Cu at (121.9, 106.2)
- added ?: , , F.Cu at (104.1, 106.2)
- added ?: , , F.Cu at (134.6, 106.2)
- added ?: , , F.Cu at (111.8, 113.8)
- added ?: , , F.Cu at (101.6, 118.9)
- added ?: , , F.Cu at (111.8, 101.1)
- added ?: , , F.Cu at (134.6, 116.3)
- added ?: , , F.Cu at (109.2, 118.9)
- added ?: , , F.Cu at (109.2, 101.1)
- added ?: , , F.Cu at (99.1, 106.2)
- added ?: , , F.Cu at (134.6, 113.8)
- added ?: , , F.Cu at (104.1, 103.6)
- added ?: , , F.Cu at (134.6, 118.9)
- added ?: , , F.Cu at (119.4, 101.1)
- added ?: , , F.Cu at (104.1, 118.9)
- added ?: , , F.Cu at (132.1, 113.8)
- added ?: , , F.Cu at (127.0, 106.2)
- added ?: , , F.Cu at (111.8, 103.6)
- added ?: , , F.Cu at (124.5, 116.3)
- added ?: , , F.Cu at (106.7, 116.3)
- added ?: , , F.Cu at (121.9, 113.8)
- added ?: , , F.Cu at (99.1, 118.9)
- added ?: , , F.Cu at (124.5, 103.6)
- added ?: , , F.Cu at (104.1, 101.1)
- added ?: , , F.Cu at (116.8, 103.6)
- added ?: , , F.Cu at (114.3, 103.6)
- added ?: , , F.Cu at (106.7, 101.1)
- added ?: , , F.Cu at (116.8, 118.9)
- added ?: , , F.Cu at (109.2, 103.6)
- added ?: , , F.Cu at (96.5, 101.1)
- added ?: , , F.Cu at (127.0, 103.6)
- added ?: , , F.Cu at (119.4, 106.2)
- added ?: , , F.Cu at (132.1, 106.2)
- added ?: , , F.Cu at (119.4, 103.6)
- added ?: , , F.Cu at (96.5, 103.6)
- added ?: , , F.Cu at (109.2, 113.8)
- added ?: , , F.Cu at (121.9, 103.6)
- added ?: , , F.Cu at (129.5, 116.3)
- added ?: , , F.Cu at (132.1, 101.1)
- added ?: , , F.Cu at (114.3, 116.3)
- added ?: , , F.Cu at (127.0, 113.8)
- added ?: , , F.Cu at (114.3, 101.1)
- added ?: , , F.Cu at (121.9, 101.1)
- added ?: , , F.Cu at (121.9, 116.3)
- added ?: , , F.Cu at (127.0, 101.1)
- added ?: , , F.Cu at (111.8, 106.2)
- added ?: , , F.Cu at (96.5, 118.9)
- added ?: , , F.Cu at (124.5, 101.1)
- added ?: , , F.Cu at (116.8, 101.1)
- added ?: , , F.Cu at (114.3, 118.9)
- added ?: , , F.Cu at (129.5, 106.2)
- added ?: , , F.Cu at (99.1, 113.8)
- added ?: , , F.Cu at (132.1, 103.6)
- added ?: , , F.Cu at (119.4, 118.9)
- added ?: , , F.Cu at (129.5, 118.9)
- added ?: , , F.Cu at (114.3, 113.8)
- added ?: , , F.Cu at (111.8, 116.3)
- added H1: MountingHole, MountingHole:MountingHole_3mm_Pad_TopBottom, F.Cu at (134.6, 94.6)
- added H2: MountingHole, MountingHole:MountingHole_3mm_Pad_TopBottom, F.Cu at (134.6, 154.3)
- BT1: footprint Battery:Battery_Panasonic_CR2032-VS1N_Vertical_CircularHoles -> MyStuff:Battery-Holder_CR2032
- U6: footprint Package_DIP:DIP-20_W7.62mm_LongPads -> Package_DIP:DIP-20_W7.62mm_Socket_LongPads
- U7, U8: footprint Package_DIP:DIP-8-16_W7.62mm_Socket_LongPads -> Package_DIP:DIP-8_W7.62mm_Socket_LongPads
- moved C4 209.7 mm to (56.9, 129.0), turned to 180 degrees
- moved C5 207.6 mm to (69.0, 129.5), turned to 180 degrees
- moved J2 197.4 mm to (44.4, 92.7)
- moved RN2 195.2 mm to (83.8, 153.4), turned to 90 degrees
- moved J1 191.2 mm to (57.9, 96.5), turned to 90 degrees
- moved C2 172.1 mm to (70.1, 107.2), turned to -90 degrees
- moved U3 171.7 mm to (73.7, 124.2), turned to 90 degrees
- moved C7 162.4 mm to (70.1, 119.1), turned to -90 degrees
- moved C1 160.4 mm to (56.6, 102.6), turned to 180 degrees
- moved C6 158.3 mm to (94.2, 144.3), turned to 180 degrees
- moved C3 157.6 mm to (70.1, 97.8), turned to 90 degrees
- moved U5 155.8 mm to (51.6, 132.6)
- moved U6 155.5 mm to (63.8, 132.7)
- moved U8 153.5 mm to (88.9, 147.6)
- moved Y1 153.1 mm to (76.7, 140.7), turned to -90 degrees
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Routing:
- net GND: track 0.00 -> 321.4 mm
- net +5V: track 0.00 -> 244.0 mm
- net /SCL: track 0.00 -> 106.0 mm
- net /SDA: track 0.00 -> 103.5 mm
- net /reset: track 0.00 -> 87.3 mm
- net /a00: track 0.00 -> 73.2 mm
- net Net-(RN2-Pad4): track 0.00 -> 63.2 mm
- net /wait: track 0.00 -> 63.1 mm
- net /iorq: track 0.00 -> 53.7 mm
- net /card_sel: track 0.00 -> 51.4 mm
- net /B00: track 0.00 -> 48.6 mm
- net Net-(U3-Pad6): track 0.00 -> 45.7 mm
- net /B01: track 0.00 -> 40.4 mm
- net Net-(U1-Pad3): track 0.00 -> 36.1 mm
- net Net-(J1-Pad8): track 0.00 -> 34.3 mm
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- added copper zone on B.Cu, net GND
Other:
- board text added: "+5V"
- board text added: "3 2 1 0"
- board text added: "GND"
- board text added: "Prototyping Area"
- board text added: "SCL"
- board text added: "SDA"
- board text added: "Z80 Modular Computer I2C Card version 1.0 Design by Kaltchuk, 06/2022"
- board text added: "card addr"
