File: KiCAD files/PSU2/PSU2.kicad_pcb (KiCad board)
At the start: 2 copper layers, 18 parts, among them J1 Enable 12V, J2 To switch, J3 Mains, J4 Ext switch, J5 Enable 3V3, J6 Power bus, J7 Mech support, U1 LM317_TO-220

Commit message: home
Parts:
- removed J7: Mech support, Connector_PinHeader_2.54mm:PinHeader_2x05_P2.54mm_Vertical
- added H1: MountingHole, MyStuff:Mounting_Hole_0.2in, F.Cu at (197.7, 87.0)
- added H2: MountingHole, MyStuff:Mounting_Hole_0.2in, F.Cu at (197.7, 146.7)
- PS1: value MEE1S0512SC -> MT3608_2-24V_2A; footprint Converter_DCDC:Converter_DCDC_Murata_MEE1SxxxxSC_THT -> MyStuff:MT3608_2-24V_2A
- R1, R3, R5: footprint Resistor_THT:R_Axial_DIN0204_L3.6mm_D1.6mm_P1.90mm_Vertical -> Resistor_THT:R_Axial_DIN0207_L6.3mm_D2.5mm_P7.62mm_Horizontal
- moved PS2 170.8 mm to (184.0, 149.9), turned to 90 degrees
- moved J3 153.7 mm to (188.6, 117.9), turned to -90 degrees
- moved D3 142.8 mm to (200.5, 102.0), turned to -90 degrees
- moved D2 141.7 mm to (200.5, 96.8), turned to -90 degrees
- moved R1 138.8 mm to (195.8, 92.6), turned to 180 degrees
- moved D1 133.0 mm to (200.5, 91.6), turned to -90 degrees
- moved R5 127.0 mm to (195.8, 102.2), turned to 180 degrees
- moved R3 123.4 mm to (195.8, 97.3), turned to 180 degrees
- moved J2 122.3 mm to (167.1, 113.9), turned to 180 degrees
- moved PS1 119.4 mm to (172.0, 85.0), turned to 180 degrees
- moved J4 115.9 mm to (170.7, 113.9), turned to 180 degrees
- moved R4 113.8 mm to (112.1, 132.8), turned to 180 degrees
- moved R2 103.1 mm to (112.1, 129.2), turned to 180 degrees
- moved J1 95.3 mm to (136.5, 105.9), turned to 90 degrees
- moved J5 83.4 mm to (113.0, 111.8), turned to -90 degrees
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Connections:
- J3 pad 1: NEUT -> LINE
- J3 pad 2: LINE -> NEUT
Routing:
- net GND: track 0.00 -> 179.3 mm, vias 0 -> 4
- net /+3.3V: track 0.00 -> 174.5 mm, vias 0 -> 4
- net /+5V: track 0.00 -> 170.6 mm
- net /+12V: track 0.00 -> 104.4 mm, vias 0 -> 2
- net Net-(J2-Pad1): track 0.00 -> 38.1 mm
- net NEUT: track 0.00 -> 33.1 mm
- net LINE: track 0.00 -> 27.7 mm
- net Net-(R2-Pad1): track 0.00 -> 9.49 mm
- net Net-(J1-Pad2): track 0.00 -> 8.95 mm
- net Net-(J5-Pad2): track 0.00 -> 7.20 mm
- net Net-(D1-Pad1): track 0.00 -> 5.12 mm
- net Net-(D2-Pad1): track 0.00 -> 4.91 mm
- net Net-(D3-Pad1): track 0.00 -> 4.81 mm
- added copper zone on B.Cu, net (none)
- added copper zone on B.Cu, net GND
Other:
- board outline added: 99.7 x 69.8 mm

Commit message: PCBs
Parts:
- removed the J1 at (136.5, 105.9)
- removed the J5 at (113.0, 111.8)
- added J4: Vo enable, Connector_PinHeader_2.54mm:PinHeader_2x02_P2.54mm_Vertical, F.Cu at (125.1, 107.7)
- added J6: Mech support, Connector_PinHeader_2.54mm:PinHeader_2x05_P2.54mm_Vertical, F.Cu at (107.6, 138.4)
- added K1: SRD-05VDC-SL-C, MyStuff:Relay_SPDT_Songel-15x19mm, F.Cu at (168.7, 86.0)
- J1: renamed from J4; footprint Connector_PinSocket_2.54mm:PinSocket_1x02_P2.54mm_Vertical -> Connector_PinHeader_2.54mm:PinHeader_1x02_P2.54mm_Vertical
- R2: value 400 -> 390; footprint Resistor_THT:R_Axial_DIN0204_L3.6mm_D1.6mm_P1.90mm_Vertical -> Resistor_THT:R_Axial_DIN0207_L6.3mm_D2.5mm_P7.62mm_Horizontal
- R4: footprint Resistor_THT:R_Axial_DIN0204_L3.6mm_D1.6mm_P1.90mm_Vertical -> Resistor_THT:R_Axial_DIN0207_L6.3mm_D2.5mm_P7.62mm_Horizontal
- moved J1 25.5 mm to (195.8, 110.0), turned to 0 degrees
- moved R2 22.3 mm to (111.5, 106.8), turned to 0 degrees
- moved R4 22.0 mm to (111.5, 110.9), turned to 0 degrees
- moved PS1 21.1 mm to (150.9, 83.6)
- moved U1 3.57 mm to (112.2, 119.9), turned to -90 degrees
- moved R3 3.19 mm to (192.7, 97.5)
- moved R1 3.18 mm to (192.7, 92.7)
- moved R5 3.18 mm to (192.7, 102.2)
- moved J2 2.91 mm to (168.8, 111.5)
- moved D3 2.85 mm to (197.9, 101.0)
- moved D2 2.71 mm to (197.9, 96.3)
- moved D1 2.67 mm to (197.9, 91.6)
- renumbered J6 to J5
Connections:
- J1 pad 1: Net-(J2-Pad1) -> Net-(J1-Pad1)
- J1 pad 2: LINE -> Net-(J1-Pad2)
- R4 pad 1: Net-(R2-Pad1) -> /+3.3V
- R4 pad 2: /+3.3V -> Net-(R2-Pad1)
Routing:
- net Net-(J1-Pad1): track 0.00 -> 65.0 mm
- net /+3.3V: track 174.5 -> 127.6 mm, vias 4 -> 0
- net Net-(J1-Pad2): track 0.00 -> 33.2 mm
- net /+5V: track 170.6 -> 143.0 mm
- net LINE: track 27.7 -> 51.4 mm
- net Net-(J4-Pad3): track 7.20 -> 21.2 mm
- net Net-(J2-Pad1): track 38.1 -> 52.2 mm
- net GND: track 179.3 -> 166.2 mm, vias 4 -> 0
- net Net-(R2-Pad1): track 9.49 -> 19.9 mm
- net /+12V: track 104.4 -> 94.5 mm, vias 2 -> 0
- net NEUT: track 33.1 -> 24.1 mm
- net Net-(J4-Pad1): track 8.95 -> 15.2 mm
- net Net-(D2-Pad1): track 4.91 -> 5.74 mm
- net Net-(D3-Pad1): track 4.81 -> 5.38 mm
- net Net-(D1-Pad1): track 5.12 -> 5.68 mm
- removed copper zone on B.Cu, net (none)
- removed copper zone on B.Cu, net GND
Other:
- board text added: "Enable 12V"
- board text added: "Enable 3.3V"
- board text added: "Z80 Modular Computer PSU Card version 2.0 Design by Kaltchuk, 08/2021"

Commit message: PCBs
Parts:
- moved K1 13.6 mm to (171.3, 99.3), turned to 90 degrees
- moved R2 7.64 mm to (119.1, 107.3), turned to 180 degrees
- moved U1 5.62 mm to (110.9, 125.3), turned to 90 degrees
- moved R4 0.25 mm to (111.5, 110.6)
Routing:
- net /+3.3V: track 127.6 -> 165.3 mm
- net Net-(J1-Pad2): track 33.2 -> 59.5 mm
- net Net-(J1-Pad1): track 65.0 -> 45.7 mm
- net Net-(J2-Pad1): track 52.2 -> 68.9 mm
- net LINE: track 51.4 -> 39.8 mm
- net GND: track 166.2 -> 154.6 mm
- net /+5V: track 143.0 -> 133.9 mm
- net /+12V: track 94.5 -> 101.8 mm
- net NEUT: track 24.1 -> 30.6 mm
- net Net-(R2-Pad1): track 19.9 -> 25.4 mm
- net Net-(J4-Pad3): track 21.2 -> 18.4 mm
- net Net-(J4-Pad1): track 15.2 -> 16.4 mm
- added copper zone on B.Cu, net GND
