File: KiCAD files/PSU2/PSU2.kicad_sch (KiCad schematic)
At the start: 15 parts, among them J1 Power switch, J2 Mains, J3 Power bus, J4 Mech support, U1 LM317_TO-220

Commit message: office
Parts:
- added J1: Enable 12V, Connector_PinHeader_2.54mm:PinHeader_1x02_P2.54mm_Vertical, symbol Connector_Generic:Conn_01x02
- added J4: Ext switch, Connector_PinSocket_2.54mm:PinSocket_1x02_P2.54mm_Vertical, symbol Connector_Generic:Conn_01x02
- added J5: Enable 3V3, Connector_PinHeader_2.54mm:PinHeader_1x02_P2.54mm_Vertical, symbol Connector_Generic:Conn_01x02
- D1, D2, D3: footprint (none) -> LED_THT:LED_D3.0mm
- J2: renamed from J1; value Power switch -> To switch
- PS1: value MEE1S0512SC -> MT3608_2-24V_2A; footprint Converter_DCDC:Converter_DCDC_Murata_MEE1SxxxxSC_THT -> (none)
- R1, R2, R3, R4, R5: footprint (none) -> Resistor_THT:R_Axial_DIN0204_L3.6mm_D1.6mm_P1.90mm_Vertical
- renumbered J2 to J3, J3 to J6, J4 to J7
Connections:
- net +5V: now also J1.1 (Pin_1), J5.1 (Pin_1); no longer PS1.2 (+Vin), U1.3 (VI)
- net LINE: now also J4.2 (Pin_2)
- net at J2.1 (Pin_1), PS2.2 (AC/L): now also J4.1 (Pin_1)
- new net: J1.2 (Pin_2), PS1.2 (+Vin)
- new net: J5.2 (Pin_2), U1.3 (VI)
Other:
- note removed: "Power on Switch"
- moved on the sheet: J7

Commit message: home
Parts:
- added H1, H2: MountingHole, MyStuff:Mounting_Hole_0.2in, symbol Mechanical:MountingHole
- PS1: footprint (none) -> MyStuff:MT3608_2-24V_2A
- R1, R3, R5: footprint Resistor_THT:R_Axial_DIN0204_L3.6mm_D1.6mm_P1.90mm_Vertical -> Resistor_THT:R_Axial_DIN0207_L6.3mm_D2.5mm_P7.62mm_Horizontal
Connections:
- net LINE: now also J3.1 (Pin_1); no longer J3.2 (Pin_2)
- net NEUT: now also J3.2 (Pin_2); no longer J3.1 (Pin_1)
Other:
- moved on the sheet: J3
Changed lines of the file:
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@@
       (effects (font (size 1.27 1.27)) (justify left))
     )
-    (property "Footprint" "Resistor_THT:R_Axial_DIN0204_L3.6mm_D1.6mm_P1.90mm_Vertical" (id 2) (at 94.742 135.89 90)
+    (property "Footprint" "Resistor_THT:R_Axial_DIN0207_L6.3mm_D2.5mm_P7.62mm_Horizontal" (id 2) (at 94.742 135.89 90)
       (effects (font (size 1.27 1.27)) hide)
     )
@@
     (property "Reference" "PS1" (id 0) (at 77.47 116.84 0))
     (property "Value" "MT3608_2-24V_2A" (id 1) (at 77.47 119.38 0))
-    (property "Footprint" "" (id 2) (at 50.8 133.35 0)
+    (property "Footprint" "MyStuff:MT3608_2-24V_2A" (id 2) (at 50.8 133.35 0)
       (effects (font (size 1.27 1.27)) (justify left) hide)
     )
@@
     )
     (pin "1")
+  )
+  (symbol (lib_id "Mechanical:MountingHole") (at 255.27 86.36 0) (unit 1)
+    (in_bom yes) (on_board yes) (fields_autoplaced)
+    (property "Reference" "H2" (id 0) (at 257.81 85.5253 0)
+      (effects (font (size 1.27 1.27)) (justify left))
+    )
+    (property "Value" "MountingHole" (id 1) (at 257.81 88.0622 0)
+      (effects (font (size 1.27 1.27)) (justify left))
+    )
+    (property "Footprint" "MyStuff:Mounting_Hole_0.2in" (id 2) (at 255.27 86.36 0)
+      (effects (font (size 1.27 1.27)) hide)
+    )
+    (property "Datasheet" "~" (id 3) (at 255.27 86.36 0)
+      (effects (font (size 1.27 1.27)) hide)
+    )
   )
   (symbol (lib_id "Device:R") (at 138.43 142.24 0) (unit 1)
@@
     (pin "4")
   )
-  (symbol (lib_id "Connector_Generic:Conn_01x02") (at 68.58 76.2 180) (unit 1)
-    (in_bom yes) (on_board yes)
-    (property "Reference" "J3" (id 0) (at 68.58 71.12 0))
-    (property "Value" "Mains" (id 1) (at 68.58 78.74 0))
-    (property "Footprint" "MyStuff:IEC60320_2pin" (id 2) (at 68.58 76.2 0)
-      (effects (font (size 1.27 1.27)) hide)
-    )
-    (property "Datasheet" "~" (id 3) (at 68.58 76.2 0)
+  (symbol (lib_id "Connector_Generic:Conn_01x02") (at 68.58 73.66 0) (mirror y) (unit 1)
+    (in_bom yes) (on_board yes)
+    (property "Reference" "J3" (id 0) (at 68.58 78.74 0))
+    (property "Value" "Mains" (id 1) (at 68.58 71.12 0))
+    (property "Footprint" "MyStuff:IEC60320_2pin" (id 2) (at 68.58 73.66 0)
+      (effects (font (size 1.27 1.27)) hide)
+    )
+    (property "Datasheet" "~" (id 3) (at 68.58 73.66 0)
       (effects (font (size 1.27 1.27)) hide)
     )
@@
       (effects (font (size 1.27 1.27)) (justify left))
     )
-    (property "Footprint" "Resistor_THT:R_Axial_DIN0204_L3.6mm_D1.6mm_P1.90mm_Vertical" (id 2) (at 155.702 137.16 90)
+    (property "Footprint" "Resistor_THT:R_Axial_DIN0207_L6.3mm_D2.5mm_P7.62mm_Horizontal" (id 2) (at 155.702 137.16 90)
       (effects (font (size 1.27 1.27)) hide)
     )
@@
       (effects (font (size 1.27 1.27)) (justify left))
     )
-    (property "Footprint" "Resistor_THT:R_Axial_DIN0204_L3.6mm_D1.6mm_P1.90mm_Vertical" (id 2) (at 140.462 82.55 90)
+    (property "Footprint" "Resistor_THT:R_Axial_DIN0207_L6.3mm_D2.5mm_P7.62mm_Horizontal" (id 2) (at 140.462 82.55 90)
       (effects (font (size 1.27 1.27)) hide)
     )
@@
     (pin "2")
   )
+  (symbol (lib_id "Mechanical:MountingHole") (at 255.27 72.39 0) (unit 1)
+    (in_bom yes) (on_board yes) (fields_autoplaced)
+    (property "Reference" "H1" (id 0) (at 257.81 71.5553 0)
+      (effects (font (size 1.27 1.27)) (justify left))
+    )
+    (property "Value" "MountingHole" (id 1) (at 257.81 74.0922 0)
+      (effects (font (size 1.27 1.27)) (justify left))
+    )
+    (property "Footprint" "MyStuff:Mounting_Hole_0.2in" (id 2) (at 255.27 72.39 0)
+      (effects (font (size 1.27 1.27)) hide)
+    )
+    (property "Datasheet" "~" (id 3) (at 255.27 72.39 0)
+      (effects (font (size 1.27 1.27)) hide)
+    )
+  )
   (symbol (lib_id "power:GND") (at 90.17 132.08 0) (unit 1)
     (in_bom yes) (on_board yes) (fields_autoplaced)
@@
       (reference "D3") (unit 1) (value "LED") (footprint "LED_THT:LED_D3.0mm")
     )
+    (path "/f602d291-6480-4ea1-9db6-21a52cb0f66b"
+      (reference "H1") (unit 1) (value "MountingHole") (footprint "MyStuff:Mounting_Hole_0.2in")
+    )
+    (path "/b5352702-8529-4bc9-91ca-7bc458f6c534"
+      (reference "H2") (unit 1) (value "MountingHole") (footprint "MyStuff:Mounting_Hole_0.2in")
+    )
     (path "/3bced514-7c6a-4929-a2f4-97c9dfd34def"
       (reference "J1") (unit 1) (value "Enable 12V") (footprint "Connector_PinHeader_2.54mm:PinHeader_1x02_P2.54mm_Vertical")
@@
     )
     (path "/aeee7a19-a484-49a2-8dd1-3304e6bdcff4"
-      (reference "PS1") (unit 1) (value "MT3608_2-24V_2A") (footprint "")
+      (reference "PS1") (unit 1) (value "MT3608_2-24V_2A") (footprint "MyStuff:MT3608_2-24V_2A")
     )
     (path "/cd472c07-49b0-43d1-9768-94dd38b72eb4"
@@
     )
     (path "/93e73584-d592-4726-92d2-a9567055e651"
-      (reference "R1") (unit 1) (value "1k2") (footprint "Resistor_THT:R_Axial_DIN0204_L3.6mm_D1.6mm_P1.90mm_Vertical")
+      (reference "R1") (unit 1) (value "1k2") (footprint "Resistor_THT:R_Axial_DIN0207_L6.3mm_D2.5mm_P7.62mm_Horizontal")
     )
     (path "/be48cf36-6613-45b4-9256-7e2c3d708f91"
@@
     )
     (path "/e29dca74-8ecf-4cc1-872a-e8938e9b5b29"
-      (reference "R3") (unit 1) (value "330") (footprint "Resistor_THT:R_Axial_DIN0204_L3.6mm_D1.6mm_P1.90mm_Vertical")
+      (reference "R3") (unit 1) (value "330") (footprint "Resistor_THT:R_Axial_DIN0207_L6.3mm_D2.5mm_P7.62mm_Horizontal")
     )
     (path "/f42a5b60-5d96-4544-a9dd-5a8d4e2bd6a3"
@@
     )
     (path "/e20e5fe9-9617-43f9-9479-6c61d12dff91"
-      (reference "R5") (unit 1) (value "150") (footprint "Resistor_THT:R_Axial_DIN0204_L3.6mm_D1.6mm_P1.90mm_Vertical")
+      (reference "R5") (unit 1) (value "150") (footprint "Resistor_THT:R_Axial_DIN0207_L6.3mm_D2.5mm_P7.62mm_Horizontal")
     )
     (path "/c5bfbfb0-e048-4c9d-9481-ac0596d198ce"

Commit message: PCBs
Parts:
- removed J1: Enable 12V, Connector_PinHeader_2.54mm:PinHeader_1x02_P2.54mm_Vertical, symbol Connector_Generic:Conn_01x02
- removed J5: Enable 3V3, Connector_PinHeader_2.54mm:PinHeader_1x02_P2.54mm_Vertical, symbol Connector_Generic:Conn_01x02
- added J4: Vo enable, Connector_PinHeader_2.54mm:PinHeader_2x02_P2.54mm_Vertical, symbol Connector_Generic:Conn_02x02_Odd_Even
- added K1: SRD-05VDC-SL-C, MyStuff:Relay_SPDT_Songel-15x19mm, symbol Relay:Y14x-1C-xxDS
- J1: renamed from J4; footprint Connector_PinSocket_2.54mm:PinSocket_1x02_P2.54mm_Vertical -> (none)
- R2: value 400 -> 390; footprint Resistor_THT:R_Axial_DIN0204_L3.6mm_D1.6mm_P1.90mm_Vertical -> Resistor_THT:R_Axial_DIN0207_L6.3mm_D2.5mm_P7.62mm_Horizontal
- R4: footprint Resistor_THT:R_Axial_DIN0204_L3.6mm_D1.6mm_P1.90mm_Vertical -> Resistor_THT:R_Axial_DIN0207_L6.3mm_D2.5mm_P7.62mm_Horizontal
- renumbered J6 to J5, J7 to J6
Connections:
- net +3.3V: now also R4.1; no longer R4.2
- net +5V: now also J4.2 (Pin_2), J4.4 (Pin_4)
- net LINE: now also K1.1; no longer J1.2 (Pin_2)
- net at PS1.2 (+Vin): now also J4.1 (Pin_1)
- net at R2.1, U1.1 (ADJ): now also R4.2; no longer R4.1
- net at J2.1 (Pin_1), PS2.2 (AC/L): now also K1.5, K1.6; no longer J1.1 (Pin_1)
- net at U1.3 (VI): now also J4.3 (Pin_3)
- new net: J1.2 (Pin_2), K1.3
- new net: J1.1 (Pin_1), K1.4
- no-connect marks 10 -> 12
Other:
- moved on the sheet: D3, J1, R5

Commit message: manual update
Parts:
- J1: footprint (none) -> Connector_PinHeader_2.54mm:PinHeader_1x02_P2.54mm_Vertical
Other:
- note added: "Enable 12V"
- note added: "Enable 3.3V"
Changed lines of the file:
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@@
     (stroke (width 0) (type default) (color 0 0 0 0))
+  )
+  (text "Enable 3.3V" (at 81.28 106.68 0)
+    (effects (font (size 1.27 1.27)) (justify left bottom))
+  )
+  (text "Enable 12V" (at 81.28 102.87 0)
+    (effects (font (size 1.27 1.27)) (justify left bottom))
   )
   (text "220Vac\n\nLine\nNeutral" (at 66.04 76.2 180)
@@
     (property "Reference" "J1" (id 0) (at 68.58 30.48 0))
     (property "Value" "Ext switch" (id 1) (at 68.58 38.1 0))
-    (property "Footprint" "" (id 2) (at 68.58 33.02 0)
-      (effects (font (size 1.27 1.27)) hide)
-    )
+    (property "Footprint" "Connector_PinHeader_2.54mm:PinHeader_1x02_P2.54mm_Vertical" (id 2) (at 68.58 33.02 0)
+      (effects (font (size 1.27 1.27)) hide)
+    )
