File: KiCAD files/I2C/I2C_frontal/I2C_frontal.kicad_pcb (KiCad board)
At the start: 2 copper layers, 24.6 x 80 mm, 2 parts, among them J7 fixing bolt, J8 fixing bolt

Commit message: PCBs
Other:
- outline, holes or cut-outs redrawn
- board text added: "I2C Bus"
- board text removed: "I2C bus"
Changed lines of the file:
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@@
     (pad_to_mask_clearance 0)
     (pcbplotparams
-      (layerselection 0x00010fc_ffffffff)
+      (layerselection 0x00010f0_ffffffff)
       (disableapertmacros false)
       (usegerberextensions false)
@@
       (outputformat 1)
       (mirror false)
-      (drillshape 1)
+      (drillshape 0)
       (scaleselection 1)
       (outputdirectory "")
@@
       (xy 192.786 122.936)
     ) (layer "F.SilkS") (width 0.1) (fill solid))
-  (gr_arc (start 178.181 63.881) (mid 178.552974 62.982974) (end 179.451 62.611) (layer "Edge.Cuts") (width 0.05))
+  (gr_arc (start 184.531 91.567) (mid 184.902974 90.668974) (end 185.801 90.297) (layer "Edge.Cuts") (width 0.05))
   (gr_line (start 195.961 128.651) (end 195.961 48.641) (layer "Edge.Cuts") (width 0.05))
-  (gr_arc (start 179.451 94.361) (mid 178.552974 93.989026) (end 178.181 93.091) (layer "Edge.Cuts") (width 0.05))
-  (gr_arc (start 185.801 114.681) (mid 184.902974 114.309026) (end 184.531 113.411) (layer "Edge.Cuts") (width 0.05))
-  (gr_line (start 189.611 62.611) (end 179.451 62.611) (layer "Edge.Cuts") (width 0.05))
-  (gr_line (start 179.451 94.361) (end 183.261 94.361) (layer "Edge.Cuts") (width 0.05))
-  (gr_line (start 178.181 63.881) (end 178.181 93.091) (layer "Edge.Cuts") (width 0.05))
-  (gr_arc (start 183.261 94.361) (mid 184.159026 94.732974) (end 184.531 95.631) (layer "Edge.Cuts") (width 0.05))
-  (gr_line (start 185.801 114.681) (end 189.611 114.681) (layer "Edge.Cuts") (width 0.05))
+  (gr_arc (start 185.791974 97.907974) (mid 184.893948 97.536) (end 184.521974 96.637974) (layer "Edge.Cuts") (width 0.05))
+  (gr_arc (start 189.601974 90.306026) (mid 190.5 90.678) (end 190.871974 91.576026) (layer "Edge.Cuts") (width 0.05))
+  (gr_line (start 185.791974 97.907974) (end 189.601974 97.907974) (layer "Edge.Cuts") (width 0.05))
   (gr_line (start 171.323 128.651) (end 195.961 128.651) (layer "Edge.Cuts") (width 0.05))
-  (gr_line (start 184.531 95.631) (end 184.531 113.411) (layer "Edge.Cuts") (width 0.05))
+  (gr_line (start 189.601974 90.306026) (end 185.810026 90.306026) (layer "Edge.Cuts") (width 0.05))
+  (gr_line (start 184.521974 91.576026) (end 184.521974 96.637974) (layer "Edge.Cuts") (width 0.05))
   (gr_line (start 171.323 48.641) (end 195.961 48.641) (layer "Edge.Cuts") (width 0.05))
-  (gr_line (start 190.881 113.411) (end 190.881 63.881) (layer "Edge.Cuts") (width 0.05))
-  (gr_arc (start 189.611 62.611) (mid 190.509026 62.982974) (end 190.881 63.881) (layer "Edge.Cuts") (width 0.05))
-  (gr_arc (start 190.881 113.411) (mid 190.509026 114.309026) (end 189.611 114.681) (layer "Edge.Cuts") (width 0.05))
+  (gr_line (start 190.871974 96.637974) (end 190.871974 91.576026) (layer "Edge.Cuts") (width 0.05))
+  (gr_arc (start 190.871974 96.637974) (mid 190.5 97.536) (end 189.601974 97.907974) (layer "Edge.Cuts") (width 0.05))
   (gr_line (start 171.323 48.641) (end 171.323 128.651) (layer "Edge.Cuts") (width 0.1))
-  (gr_text "I2C\nbus" (at 212.979 81.28) (layer "F.SilkS")
+  (gr_text "I2C\nBus" (at 184.912 85.852) (layer "F.SilkS")
     (effects (font (size 2.0828 2.0828) (thickness 0.3302)) (justify left))
   )

Commit message: update PCBs
Changed lines of the file:
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@@
     (fp_line (start -1.27 1.27) (end -1.27 -0.635) (layer "F.Fab") (width 0.1))
     (fp_line (start -1.27 -0.635) (end -0.635 -1.27) (layer "F.Fab") (width 0.1))
-    (pad "1" thru_hole circle locked (at 0 0) (size 5.08 5.08) (drill 3.048) (layers *.Cu *.Mask))
+    (pad "" thru_hole circle locked (at 0 0) (size 5.08 5.08) (drill 3.048) (layers *.Cu *.Mask))
     (model "${KISYS3DMOD}/Connector_PinHeader_2.54mm.3dshapes/PinHeader_1x01_P2.54mm_Vertical.wrl"
       (offset (xyz 0 0 0))
@@
     (fp_line (start -1.27 -0.635) (end -0.635 -1.27) (layer "F.Fab") (width 0.1))
     (fp_line (start -1.27 1.27) (end -1.27 -0.635) (layer "F.Fab") (width 0.1))
-    (pad "1" thru_hole circle locked (at 0 0) (size 5.08 5.08) (drill 3.048) (layers *.Cu *.Mask))
+    (pad "" thru_hole circle locked (at 0 0) (size 5.08 5.08) (drill 3.048) (layers *.Cu *.Mask))
     (model "${KISYS3DMOD}/Connector_PinHeader_2.54mm.3dshapes/PinHeader_1x01_P2.54mm_Vertical.wrl"
       (offset (xyz 0 0 0))
@@
   (gr_arc (start 190.871974 96.637974) (mid 190.5 97.536) (end 189.601974 97.907974) (layer "Edge.Cuts") (width 0.05))
   (gr_line (start 171.323 48.641) (end 171.323 128.651) (layer "Edge.Cuts") (width 0.1))
-  (gr_text "I2C\nBus" (at 184.912 85.852) (layer "F.SilkS")
+  (gr_text "I2C\nBus" (at 175.387 93.853) (layer "F.SilkS")
     (effects (font (size 2.0828 2.0828) (thickness 0.3302)) (justify left))
   )
