File: KiCAD files/PSU2/PSU2_frontal/PSU2_frontal.kicad_pcb (KiCad board)
At the start: 2 copper layers, 24.6 x 80 mm, 6 parts, among them J1 fixing bolt, J10 led, J17 led, J2 fixing bolt, J9 reset button

Commit message: PCBs
Parts:
- moved J9 1.52 mm to (115.6, 86.5)
Other:
- outline, holes or cut-outs redrawn
- board text added: "100~265Vac"
- board text added: "5V relay"
- board text added: "I"
- board text added: "Mains"
- board text added: "O"
- board text removed: "Mains 100~265Vac"
- board text removed: "On/Off"
- board text removed: "on/off (5V)"
Changed lines of the file:
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@@
     (pad_to_mask_clearance 0)
     (pcbplotparams
-      (layerselection 0x00010fc_ffffffff)
+      (layerselection 0x00010f0_ffffffff)
       (disableapertmacros false)
       (usegerberextensions false)
@@
       (outputformat 1)
       (mirror false)
-      (drillshape 1)
+      (drillshape 0)
       (scaleselection 1)
       (outputdirectory "")
@@
   )
   (footprint "Connector_PinHeader_2.54mm:PinHeader_1x01_P2.54mm_Vertical" (layer "F.Cu")
-    (at 117.094 86.487)
+    (at 115.57 86.487)
     (descr "Through hole straight pin header, 1x01, 2.54mm pitch, single row")
     (tags "Through hole pin header THT 1x01 2.54mm single row")
@@
     (fp_line (start -1.27 -0.635) (end -0.635 -1.27) (layer "F.Fab") (width 0.1))
     (fp_line (start -1.27 1.27) (end -1.27 -0.635) (layer "F.Fab") (width 0.1))
-    (pad "1" thru_hole circle locked (at 0 0) (size 9.144 9.144) (drill 7.112) (layers *.Cu *.Mask))
+    (pad "1" thru_hole circle locked (at 0 0) (size 8 8) (drill 6) (layers *.Cu *.Mask))
     (model "${KISYS3DMOD}/Connector_PinHeader_2.54mm.3dshapes/PinHeader_1x01_P2.54mm_Vertical.wrl"
       (offset (xyz 0 0 0))
@@
     )
   )
+  (gr_line (start 126.374026 83.956026) (end 125.739026 83.956026) (layer "Edge.Cuts") (width 0.05))
   (gr_line (start 120.015 93.726) (end 126.365 93.726) (layer "Edge.Cuts") (width 0.05))
   (gr_arc (start 120.005974 115.941974) (mid 119.107948 115.57) (end 118.735974 114.671974) (layer "Edge.Cuts") (width 0.05))
   (gr_arc (start 127.625974 114.671974) (mid 127.254 115.57) (end 126.355974 115.941974) (layer "Edge.Cuts") (width 0.05))
+  (gr_line (start 124.469026 85.226026) (end 124.469025 89.163025) (layer "Edge.Cuts") (width 0.05))
   (gr_line (start 127.635 94.996) (end 127.625974 104.775) (layer "Edge.Cuts") (width 0.05))
   (gr_line (start 132.588 52.832) (end 132.588 132.842) (layer "Edge.Cuts") (width 0.1))
@@
   (gr_line (start 127.625974 104.775) (end 127.625974 114.671974) (layer "Edge.Cuts") (width 0.05))
   (gr_line (start 126.355974 115.941974) (end 120.005974 115.941974) (layer "Edge.Cuts") (width 0.05))
+  (gr_arc (start 127.644025 89.163025) (mid 127.272051 90.061051) (end 126.374025 90.433025) (layer "Edge.Cuts") (width 0.05))
   (gr_line (start 107.95 52.832) (end 132.588 52.832) (layer "Edge.Cuts") (width 0.05))
+  (gr_line (start 125.739025 90.433025) (end 126.374025 90.433025) (layer "Edge.Cuts") (width 0.05))
+  (gr_arc (start 126.374026 83.956026) (mid 127.272051 84.328001) (end 127.644026 85.226026) (layer "Edge.Cuts") (width 0.05))
+  (gr_line (start 127.644025 89.163025) (end 127.644026 85.226026) (layer "Edge.Cuts") (width 0.05))
   (gr_line (start 107.95 52.832) (end 107.95 132.842) (layer "Edge.Cuts") (width 0.05))
   (gr_arc (start 118.745 94.996) (mid 119.116974 94.097974) (end 120.015 93.726) (layer "Edge.Cuts") (width 0.05))
+  (gr_arc (start 125.739025 90.433025) (mid 124.840999 90.061051) (end 124.469025 89.163025) (layer "Edge.Cuts") (width 0.05))
+  (gr_arc (start 124.469026 85.226026) (mid 124.841 84.328) (end 125.739026 83.956026) (layer "Edge.Cuts") (width 0.05))
   (gr_line (start 107.95 132.842) (end 132.588 132.842) (layer "Edge.Cuts") (width 0.05))
   (gr_text "5V\n" (at 119.634 73.152) (layer "F.SilkS")
@@
     (effects (font (size 2.0828 2.0828) (thickness 0.3302)) (justify right))
   )
-  (gr_text "on/off (5V)" (at 129.667 81.534 90) (layer "F.SilkS")
-    (effects (font (size 2.0828 2.0828) (thickness 0.3302)) (justify left))
-  )
-  (gr_text "Mains\n100~265Vac" (at 113.665 105.029 90) (layer "F.SilkS")
+  (gr_text "5V relay" (at 129.921 90.424 90) (layer "F.SilkS")
+    (effects (font (size 1 1) (thickness 0.15)) (justify left))
+  )
+  (gr_text "100~265Vac" (at 115.189 105.156 90) (layer "F.SilkS")
+    (effects (font (size 1 1) (thickness 0.15)))
+  )
+  (gr_text "Mains" (at 112.649 105.029 90) (layer "F.SilkS")
     (effects (font (size 2.0828 2.0828) (thickness 0.3302)))
   )
@@
     (effects (font (size 2.0828 2.0828) (thickness 0.3302)) (justify right))
   )
+  (gr_text "I" (at 111.125 80.645) (layer "F.SilkS")
+    (effects (font (size 2.0828 2.0828) (thickness 0.3302)) (justify right))
+  )
   (gr_text "12V\n" (at 119.634 68.707) (layer "F.SilkS")
     (effects (font (size 2.0828 2.0828) (thickness 0.3302)) (justify right))
   )
-  (gr_text "On/Off" (at 110.236 80.899 90) (layer "F.SilkS")
-    (effects (font (size 2.0828 2.0828) (thickness 0.3302)) (justify right))
-  )
+  (gr_text "O" (at 111.633 92.583) (layer "F.SilkS")
+    (effects (font (size 2.0828 2.0828) (thickness 0.3302)) (justify right))
+  )

Commit message: update PCBs
Other:
- board text added: "On/Off"
Changed lines of the file:
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@@
     (fp_line (start -1.33 -1.33) (end 0 -1.33) (layer "F.SilkS") (width 0.12))
     (fp_line (start 1.33 1.27) (end 1.33 1.33) (layer "F.SilkS") (width 0.12))
-    (fp_line (start -1.8 -1.8) (end -1.8 1.8) (layer "F.CrtYd") (width 0.05))
-    (fp_line (start 1.8 1.8) (end 1.8 -1.8) (layer "F.CrtYd") (width 0.05))
-    (fp_line (start 1.8 -1.8) (end -1.8 -1.8) (layer "F.CrtYd") (width 0.05))
-    (fp_line (start -1.8 1.8) (end 1.8 1.8) (layer "F.CrtYd") (width 0.05))
-    (fp_line (start -0.635 -1.27) (end 1.27 -1.27) (layer "F.Fab") (width 0.1))
-    (fp_line (start 1.27 -1.27) (end 1.27 1.27) (layer "F.Fab") (width 0.1))
-    (fp_line (start -1.27 -0.635) (end -0.635 -1.27) (layer "F.Fab") (width 0.1))
-    (fp_line (start -1.27 1.27) (end -1.27 -0.635) (layer "F.Fab") (width 0.1))
-    (fp_line (start 1.27 1.27) (end -1.27 1.27) (layer "F.Fab") (width 0.1))
-    (pad "1" thru_hole circle locked (at 0 0) (size 4.064 4.064) (drill 3.048) (layers *.Cu *.Mask))
+    (fp_line (start -0.635 -1.27) (end 1.27 -1.27) (layer "F.Fab") (width 0.1))
+    (fp_line (start 1.27 -1.27) (end 1.27 1.27) (layer "F.Fab") (width 0.1))
+    (fp_line (start -1.27 -0.635) (end -0.635 -1.27) (layer "F.Fab") (width 0.1))
+    (fp_line (start -1.27 1.27) (end -1.27 -0.635) (layer "F.Fab") (width 0.1))
+    (fp_line (start 1.27 1.27) (end -1.27 1.27) (layer "F.Fab") (width 0.1))
+    (pad "" thru_hole circle (at 0 0) (size 4.064 4.064) (drill 3.048) (layers *.Cu *.Mask))
     (model "${KISYS3DMOD}/Connector_PinHeader_2.54mm.3dshapes/PinHeader_1x01_P2.54mm_Vertical.wrl"
       (offset (xyz 0 0 0))
@@
     (fp_line (start -1.27 -0.635) (end -0.635 -1.27) (layer "F.Fab") (width 0.1))
     (fp_line (start -1.27 1.27) (end -1.27 -0.635) (layer "F.Fab") (width 0.1))
-    (pad "1" thru_hole circle locked (at 0 0) (size 8 8) (drill 6) (layers *.Cu *.Mask))
+    (pad "" thru_hole circle locked (at 0 0) (size 8 8) (drill 6) (layers *.Cu *.Mask))
     (model "${KISYS3DMOD}/Connector_PinHeader_2.54mm.3dshapes/PinHeader_1x01_P2.54mm_Vertical.wrl"
       (offset (xyz 0 0 0))
@@
     (fp_line (start -1.33 1.27) (end 1.33 1.27) (layer "F.SilkS") (width 0.12))
     (fp_line (start 1.33 1.27) (end 1.33 1.33) (layer "F.SilkS") (width 0.12))
-    (fp_line (start 1.8 -1.8) (end -1.8 -1.8) (layer "F.CrtYd") (width 0.05))
-    (fp_line (start 1.8 1.8) (end 1.8 -1.8) (layer "F.CrtYd") (width 0.05))
-    (fp_line (start -1.8 1.8) (end 1.8 1.8) (layer "F.CrtYd") (width 0.05))
-    (fp_line (start -1.8 -1.8) (end -1.8 1.8) (layer "F.CrtYd") (width 0.05))
-    (fp_line (start 1.27 -1.27) (end 1.27 1.27) (layer "F.Fab") (width 0.1))
-    (fp_line (start -0.635 -1.27) (end 1.27 -1.27) (layer "F.Fab") (width 0.1))
-    (fp_line (start 1.27 1.27) (end -1.27 1.27) (layer "F.Fab") (width 0.1))
-    (fp_line (start -1.27 -0.635) (end -0.635 -1.27) (layer "F.Fab") (width 0.1))
-    (fp_line (start -1.27 1.27) (end -1.27 -0.635) (layer "F.Fab") (width 0.1))
-    (pad "1" thru_hole circle locked (at 0 0) (size 4.064 4.064) (drill 3.048) (layers *.Cu *.Mask))
+    (fp_line (start 1.27 -1.27) (end 1.27 1.27) (layer "F.Fab") (width 0.1))
+    (fp_line (start -0.635 -1.27) (end 1.27 -1.27) (layer "F.Fab") (width 0.1))
+    (fp_line (start 1.27 1.27) (end -1.27 1.27) (layer "F.Fab") (width 0.1))
+    (fp_line (start -1.27 -0.635) (end -0.635 -1.27) (layer "F.Fab") (width 0.1))
+    (fp_line (start -1.27 1.27) (end -1.27 -0.635) (layer "F.Fab") (width 0.1))
+    (pad "" thru_hole circle (at 0 0) (size 4.064 4.064) (drill 3.048) (layers *.Cu *.Mask))
     (model "${KISYS3DMOD}/Connector_PinHeader_2.54mm.3dshapes/PinHeader_1x01_P2.54mm_Vertical.wrl"
       (offset (xyz 0 0 0))
@@
     (fp_line (start -1.33 1.33) (end 1.33 1.33) (layer "F.SilkS") (width 0.12))
     (fp_line (start -1.33 1.27) (end 1.33 1.27) (layer "F.SilkS") (width 0.12))
-    (fp_line (start -1.8 -1.8) (end -1.8 1.8) (layer "F.CrtYd") (width 0.05))
-    (fp_line (start 1.8 -1.8) (end -1.8 -1.8) (layer "F.CrtYd") (width 0.05))
-    (fp_line (start 1.8 1.8) (end 1.8 -1.8) (layer "F.CrtYd") (width 0.05))
-    (fp_line (start -1.8 1.8) (end 1.8 1.8) (layer "F.CrtYd") (width 0.05))
-    (fp_line (start -1.27 1.27) (end -1.27 -0.635) (layer "F.Fab") (width 0.1))
-    (fp_line (start 1.27 1.27) (end -1.27 1.27) (layer "F.Fab") (width 0.1))
-    (fp_line (start 1.27 -1.27) (end 1.27 1.27) (layer "F.Fab") (width 0.1))
-    (fp_line (start -0.635 -1.27) (end 1.27 -1.27) (layer "F.Fab") (width 0.1))
-    (fp_line (start -1.27 -0.635) (end -0.635 -1.27) (layer "F.Fab") (width 0.1))
-    (pad "1" thru_hole circle locked (at 0 0) (size 4.064 4.064) (drill 3.048) (layers *.Cu *.Mask))
+    (fp_line (start -1.27 1.27) (end -1.27 -0.635) (layer "F.Fab") (width 0.1))
+    (fp_line (start 1.27 1.27) (end -1.27 1.27) (layer "F.Fab") (width 0.1))
+    (fp_line (start 1.27 -1.27) (end 1.27 1.27) (layer "F.Fab") (width 0.1))
+    (fp_line (start -0.635 -1.27) (end 1.27 -1.27) (layer "F.Fab") (width 0.1))
+    (fp_line (start -1.27 -0.635) (end -0.635 -1.27) (layer "F.Fab") (width 0.1))
+    (pad "" thru_hole circle (at 0 0) (size 4.064 4.064) (drill 3.048) (layers *.Cu *.Mask))
     (model "${KISYS3DMOD}/Connector_PinHeader_2.54mm.3dshapes/PinHeader_1x01_P2.54mm_Vertical.wrl"
       (offset (xyz 0 0 0))
@@
     (fp_line (start -1.27 1.27) (end -1.27 -0.635) (layer "F.Fab") (width 0.1))
     (fp_line (start 1.27 -1.27) (end 1.27 1.27) (layer "F.Fab") (width 0.1))
-    (pad "1" thru_hole circle locked (at 0 0) (size 5.08 5.08) (drill 3.048) (layers *.Cu *.Mask))
+    (pad "" thru_hole circle locked (at 0 0) (size 5.08 5.08) (drill 3.048) (layers *.Cu *.Mask))
     (model "${KISYS3DMOD}/Connector_PinHeader_2.54mm.3dshapes/PinHeader_1x01_P2.54mm_Vertical.wrl"
       (offset (xyz 0 0 0))
@@
     (fp_line (start -1.27 -0.635) (end -0.635 -1.27) (layer "F.Fab") (width 0.1))
     (fp_line (start -1.27 1.27) (end -1.27 -0.635) (layer "F.Fab") (width 0.1))
-    (pad "1" thru_hole circle locked (at 0 0) (size 5.08 5.08) (drill 3.048) (layers *.Cu *.Mask))
+    (pad "" thru_hole circle locked (at 0 0) (size 5.08 5.08) (drill 3.048) (layers *.Cu *.Mask))
     (model "${KISYS3DMOD}/Connector_PinHeader_2.54mm.3dshapes/PinHeader_1x01_P2.54mm_Vertical.wrl"
       (offset (xyz 0 0 0))
@@
     (effects (font (size 2.0828 2.0828) (thickness 0.3302)) (justify right))
   )
-  (gr_text "5V relay" (at 129.921 90.424 90) (layer "F.SilkS")
+  (gr_text "5V relay" (at 129.413 90.424 90) (layer "F.SilkS")
     (effects (font (size 1 1) (thickness 0.15)) (justify left))
   )
@@
     (effects (font (size 2.0828 2.0828) (thickness 0.3302)) (justify right))
   )
+  (gr_text "On/Off" (at 121.793 81.28 90) (layer "F.SilkS")
+    (effects (font (size 2.0828 2.0828) (thickness 0.3302)) (justify right))
+  )
   (gr_text "12V\n" (at 119.634 68.707) (layer "F.SilkS")
     (effects (font (size 2.0828 2.0828) (thickness 0.3302)) (justify right))
   )
-  (gr_text "O" (at 111.633 92.583) (layer "F.SilkS")
-    (effects (font (size 2.0828 2.0828) (thickness 0.3302)) (justify right))
-  )
+  (gr_text "O" (at 111.76 92.456) (layer "F.SilkS")
+    (effects (font (size 2.0828 2.0828) (thickness 0.3302)) (justify right))
+  )
