File: KiCAD files/PX051/PX051.kicad_sch (KiCad schematic)
At the start: 23 parts, among them J1 card addr, J2 Power Bus, J3 Signal Bus, Q1 BC547, Q2 BC328, Q3 BC547, Q4 BC328, U1 74LS85, U2 74LS04, U3 8255A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

Commit message: office
Parts:
- added U? (x2): 74LS04, symbol 74xx:74LS04
Connections:
- net GND: now also U?.11, U?.13
- no-connect marks 11 -> 13
Changed lines of the file:
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@@
   (junction (at 267.97 123.19) (diameter 0) (color 0 0 0 0)
   )
+  (no_connect (at 157.48 161.29))
+  (no_connect (at 157.48 177.8))
   (no_connect (at 250.19 41.91))
   (no_connect (at 219.71 54.61))
@@
     (pin "1")
   )
+  (symbol (lib_id "power:GND") (at 142.24 161.29 0) (unit 1)
+    (in_bom yes) (on_board yes) (fields_autoplaced)
+    (property "Reference" "#PWR?" (id 0) (at 142.24 167.64 0)
+      (effects (font (size 1.27 1.27)) hide)
+    )
+    (property "Value" "GND" (id 1) (at 142.24 166.37 0))
+    (property "Footprint" "" (id 2) (at 142.24 161.29 0)
+      (effects (font (size 1.27 1.27)) hide)
+    )
+    (property "Datasheet" "" (id 3) (at 142.24 161.29 0)
+      (effects (font (size 1.27 1.27)) hide)
+    )
+    (pin "1")
+  )
+  (symbol (lib_id "74xx:74LS04") (at 149.86 161.29 0) (unit 5)
+    (in_bom yes) (on_board yes) (fields_autoplaced)
+    (property "Reference" "U?" (id 0) (at 149.86 152.4 0))
+    (property "Value" "74LS04" (id 1) (at 149.86 154.94 0))
+    (property "Footprint" "" (id 2) (at 149.86 161.29 0)
+      (effects (font (size 1.27 1.27)) hide)
+    )
+    (property "Datasheet" "http://www.ti.com/lit/gpn/sn74LS04" (id 3) (at 149.86 161.29 0)
+      (effects (font (size 1.27 1.27)) hide)
+    )
+    (pin "10")
+    (pin "11")
+  )
   (symbol (lib_id "power:+5V") (at 54.61 167.64 0) (unit 1)
     (in_bom yes) (on_board yes) (fields_autoplaced)
@@
     )
     (property "Datasheet" "" (id 3) (at 62.23 54.61 0)
+      (effects (font (size 1.27 1.27)) hide)
+    )
+    (pin "1")
+  )
+  (symbol (lib_id "power:GND") (at 142.24 177.8 0) (unit 1)
+    (in_bom yes) (on_board yes) (fields_autoplaced)
+    (property "Reference" "#PWR?" (id 0) (at 142.24 184.15 0)
+      (effects (font (size 1.27 1.27)) hide)
+    )
+    (property "Value" "GND" (id 1) (at 142.24 182.88 0))
+    (property "Footprint" "" (id 2) (at 142.24 177.8 0)
+      (effects (font (size 1.27 1.27)) hide)
+    )
+    (property "Datasheet" "" (id 3) (at 142.24 177.8 0)
       (effects (font (size 1.27 1.27)) hide)
     )
@@
     (pin "3")
   )
+  (symbol (lib_id "74xx:74LS04") (at 149.86 177.8 0) (unit 6)
+    (in_bom yes) (on_board yes) (fields_autoplaced)
+    (property "Reference" "U?" (id 0) (at 149.86 168.91 0))
+    (property "Value" "74LS04" (id 1) (at 149.86 171.45 0))
+    (property "Footprint" "" (id 2) (at 149.86 177.8 0)
+      (effects (font (size 1.27 1.27)) hide)
+    )
+    (property "Datasheet" "http://www.ti.com/lit/gpn/sn74LS04" (id 3) (at 149.86 177.8 0)
+      (effects (font (size 1.27 1.27)) hide)
+    )
+    (pin "12")
+    (pin "13")
+  )
   (symbol (lib_id "power:GND") (at 62.23 69.85 0) (unit 1)
     (in_bom yes) (on_board yes)
@@
       (reference "#PWR031") (unit 1) (value "GND") (footprint "")
     )
+    (path "/2a67836a-a519-4ab4-8b9f-f34934c8fe15"
+      (reference "#PWR?") (unit 1) (value "GND") (footprint "")
+    )
+    (path "/4b5893ab-254a-408e-a775-ee4775099eb0"
+      (reference "#PWR?") (unit 1) (value "GND") (footprint "")
+    )
     (path "/3b434176-5f57-4fd6-998d-219d1cbb5dbc"
       (reference "C1") (unit 1) (value "10nF") (footprint "")
@@
       (reference "U4") (unit 1) (value "AT89C4051-24P") (footprint "Package_DIP:DIP-20_W7.62mm")
     )
-  )
+    (path "/31661a0e-1491-413b-954a-1bcd23432c00"
+      (reference "U?") (unit 5) (value "74LS04") (footprint "")
+    )
+    (path "/cfa82190-a0ae-430f-bfc8-4113205faaf4"
+      (reference "U?") (unit 6) (value "74LS04") (footprint "")
+    )
+  )

Commit message: office
Parts:
- added R? (x2): 10k, symbol Device:R
Connections:
- net +5V: now also R?.1, R?.1
- net at U3.3 (PA1), U4.13 (P1.1): now also R?.2
- net at U3.4 (PA0), U4.12 (P1.0): now also R?.2
Changed lines of the file:
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@@
   (junction (at 54.61 116.84) (diameter 0) (color 0 0 0 0)
   )
+  (junction (at 196.85 31.75) (diameter 0) (color 0 0 0 0)
+  )
   (junction (at 35.56 119.38) (diameter 0) (color 0 0 0 0)
   )
   (junction (at 96.52 116.84) (diameter 0) (color 0 0 0 0)
   )
+  (junction (at 204.47 22.86) (diameter 0) (color 0 0 0 0)
+  )
   (junction (at 57.15 119.38) (diameter 0) (color 0 0 0 0)
+  )
+  (junction (at 204.47 34.29) (diameter 0) (color 0 0 0 0)
   )
   (junction (at 267.97 115.57) (diameter 0) (color 0 0 0 0)
@@
     (stroke (width 0) (type default) (color 0 0 0 0))
   )
-  (wire (pts (xy 189.23 31.75) (xy 219.71 31.75))
+  (wire (pts (xy 204.47 34.29) (xy 219.71 34.29))
     (stroke (width 0) (type default) (color 0 0 0 0))
   )
@@
     (stroke (width 0) (type default) (color 0 0 0 0))
   )
+  (wire (pts (xy 189.23 34.29) (xy 204.47 34.29))
+    (stroke (width 0) (type default) (color 0 0 0 0))
+  )
   (wire (pts (xy 96.52 116.84) (xy 96.52 119.38))
     (stroke (width 0) (type default) (color 0 0 0 0))
@@
     (stroke (width 0) (type default) (color 0 0 0 0))
   )
+  (wire (pts (xy 196.85 22.86) (xy 204.47 22.86))
+    (stroke (width 0) (type default) (color 0 0 0 0))
+  )
   (wire (pts (xy 143.51 137.16) (xy 119.38 137.16))
     (stroke (width 0) (type default) (color 0 0 0 0))
@@
     (stroke (width 0) (type default) (color 0 0 0 0))
   )
+  (wire (pts (xy 204.47 30.48) (xy 204.47 34.29))
+    (stroke (width 0) (type default) (color 0 0 0 0))
+  )
   (wire (pts (xy 57.15 113.03) (xy 57.15 119.38))
     (stroke (width 0) (type default) (color 0 0 0 0))
   )
+  (wire (pts (xy 196.85 30.48) (xy 196.85 31.75))
+    (stroke (width 0) (type default) (color 0 0 0 0))
+  )
   (wire (pts (xy 261.62 36.83) (xy 261.62 90.17))
     (stroke (width 0) (type default) (color 0 0 0 0))
@@
     (stroke (width 0) (type default) (color 0 0 0 0))
   )
+  (wire (pts (xy 189.23 31.75) (xy 196.85 31.75))
+    (stroke (width 0) (type default) (color 0 0 0 0))
+  )
   (wire (pts (xy 31.75 33.02) (xy 31.75 36.83))
     (stroke (width 0) (type default) (color 0 0 0 0))
@@
     (stroke (width 0) (type default) (color 0 0 0 0))
   )
-  (wire (pts (xy 189.23 34.29) (xy 219.71 34.29))
-    (stroke (width 0) (type default) (color 0 0 0 0))
-  )
   (wire (pts (xy 130.81 31.75) (xy 130.81 82.55))
     (stroke (width 0) (type default) (color 0 0 0 0))
@@
   )
   (wire (pts (xy 52.07 59.69) (xy 73.66 59.69))
+    (stroke (width 0) (type default) (color 0 0 0 0))
+  )
+  (wire (pts (xy 196.85 31.75) (xy 219.71 31.75))
     (stroke (width 0) (type default) (color 0 0 0 0))
   )
@@
     )
     (pin "1")
+  )
+  (symbol (lib_id "power:+5V") (at 204.47 22.86 0) (unit 1)
+    (in_bom yes) (on_board yes) (fields_autoplaced)
+    (property "Reference" "#PWR?" (id 0) (at 204.47 26.67 0)
+      (effects (font (size 1.27 1.27)) hide)
+    )
+    (property "Value" "+5V" (id 1) (at 204.47 17.78 0))
+    (property "Footprint" "" (id 2) (at 204.47 22.86 0)
+      (effects (font (size 1.27 1.27)) hide)
+    )
+    (property "Datasheet" "" (id 3) (at 204.47 22.86 0)
+      (effects (font (size 1.27 1.27)) hide)
+    )
+    (pin "1")
+  )
+  (symbol (lib_id "Device:R") (at 196.85 26.67 0) (unit 1)
+    (in_bom yes) (on_board yes)
+    (property "Reference" "R?" (id 0) (at 198.12 25.4 0)
+      (effects (font (size 1.27 1.27)) (justify left))
+    )
+    (property "Value" "10k" (id 1) (at 198.12 27.94 0)
+      (effects (font (size 1.27 1.27)) (justify left))
+    )
+    (property "Footprint" "" (id 2) (at 195.072 26.67 90)
+      (effects (font (size 1.27 1.27)) hide)
+    )
+    (property "Datasheet" "~" (id 3) (at 196.85 26.67 0)
+      (effects (font (size 1.27 1.27)) hide)
+    )
+    (pin "1")
+    (pin "2")
   )
   (symbol (lib_id "power:GND") (at 142.24 177.8 0) (unit 1)
@@
     (pin "9")
   )
+  (symbol (lib_id "Device:R") (at 204.47 26.67 0) (unit 1)
+    (in_bom yes) (on_board yes)
+    (property "Reference" "R?" (id 0) (at 205.74 25.4 0)
+      (effects (font (size 1.27 1.27)) (justify left))
+    )
+    (property "Value" "10k" (id 1) (at 205.74 27.94 0)
+      (effects (font (size 1.27 1.27)) (justify left))
+    )
+    (property "Footprint" "" (id 2) (at 202.692 26.67 90)
+      (effects (font (size 1.27 1.27)) hide)
+    )
+    (property "Datasheet" "~" (id 3) (at 204.47 26.67 0)
+      (effects (font (size 1.27 1.27)) hide)
+    )
+    (pin "1")
+    (pin "2")
+  )
   (symbol (lib_id "Transistor_BJT:BC328") (at 255.27 125.73 270) (mirror x) (unit 1)
     (in_bom yes) (on_board yes)
@@
       (reference "#PWR?") (unit 1) (value "GND") (footprint "")
     )
+    (path "/49efb0be-60b6-44b1-8fc9-baffb4405f8d"
+      (reference "#PWR?") (unit 1) (value "+5V") (footprint "")
+    )
     (path "/4b5893ab-254a-408e-a775-ee4775099eb0"
       (reference "#PWR?") (unit 1) (value "GND") (footprint "")
@@
       (reference "R5") (unit 1) (value "10k") (footprint "Resistor_THT:R_Axial_DIN0207_L6.3mm_D2.5mm_P7.62mm_Horizontal")
     )
+    (path "/4a075904-512b-4037-94e6-7684d38257fa"
+      (reference "R?") (unit 1) (value "10k") (footprint "")
+    )
+    (path "/be356eb4-ff45-49c8-8d6a-27c498cf79f0"
+      (reference "R?") (unit 1) (value "10k") (footprint "")
+    )
     (path "/19c97e1b-f7b7-42cd-a358-3bfa194d1c62"

Commit message: updates
Parts:
- gave numbers to parts that had none: 3
Changed lines of the file:
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@@
       (effects (font (size 1.27 1.27)) hide)
     )
+    (pin "1")
+    (pin "2")
+    (pin "3")
+    (pin "4")
     (pin "5")
     (pin "6")
+    (pin "8")
+    (pin "9")
+    (pin "10")
+    (pin "11")
+    (pin "12")
+    (pin "13")
+    (pin "14")
+    (pin "7")
   )
   (symbol (lib_id "power:GND") (at 83.82 144.78 0) (unit 1)
@@
   (symbol (lib_id "power:GND") (at 142.24 161.29 0) (unit 1)
     (in_bom yes) (on_board yes) (fields_autoplaced)
-    (property "Reference" "#PWR?" (id 0) (at 142.24 167.64 0)
+    (property "Reference" "#PWR0103" (id 0) (at 142.24 167.64 0)
       (effects (font (size 1.27 1.27)) hide)
     )
@@
   (symbol (lib_id "74xx:74LS04") (at 149.86 161.29 0) (unit 5)
     (in_bom yes) (on_board yes) (fields_autoplaced)
-    (property "Reference" "U?" (id 0) (at 149.86 152.4 0))
+    (property "Reference" "U5" (id 0) (at 149.86 152.4 0))
     (property "Value" "74LS04" (id 1) (at 149.86 154.94 0))
     (property "Footprint" "" (id 2) (at 149.86 161.29 0)
@@
       (effects (font (size 1.27 1.27)) hide)
     )
+    (pin "1")
+    (pin "2")
+    (pin "3")
+    (pin "4")
+    (pin "5")
+    (pin "6")
+    (pin "8")
+    (pin "9")
     (pin "10")
     (pin "11")
+    (pin "12")
+    (pin "13")
+    (pin "14")
+    (pin "7")
   )
   (symbol (lib_id "power:+5V") (at 54.61 167.64 0) (unit 1)
@@
   (symbol (lib_id "power:+5V") (at 204.47 22.86 0) (unit 1)
     (in_bom yes) (on_board yes) (fields_autoplaced)
-    (property "Reference" "#PWR?" (id 0) (at 204.47 26.67 0)
+    (property "Reference" "#PWR0101" (id 0) (at 204.47 26.67 0)
       (effects (font (size 1.27 1.27)) hide)
     )
@@
   (symbol (lib_id "Device:R") (at 196.85 26.67 0) (unit 1)
     (in_bom yes) (on_board yes)
-    (property "Reference" "R?" (id 0) (at 198.12 25.4 0)
+    (property "Reference" "R6" (id 0) (at 198.12 25.4 0)
       (effects (font (size 1.27 1.27)) (justify left))
     )
@@
   (symbol (lib_id "power:GND") (at 142.24 177.8 0) (unit 1)
     (in_bom yes) (on_board yes) (fields_autoplaced)
-    (property "Reference" "#PWR?" (id 0) (at 142.24 184.15 0)
+    (property "Reference" "#PWR0102" (id 0) (at 142.24 184.15 0)
       (effects (font (size 1.27 1.27)) hide)
     )
@@
       (effects (font (size 1.27 1.27)) hide)
     )
+    (pin "1")
+    (pin "2")
     (pin "3")
     (pin "4")
+    (pin "5")
+    (pin "6")
+    (pin "8")
+    (pin "9")
+    (pin "10")
+    (pin "11")
+    (pin "12")
+    (pin "13")
+    (pin "14")
+    (pin "7")
   )
   (symbol (lib_id "power:PWR_FLAG") (at 73.66 33.02 0) (unit 1)
@@
     (pin "1")
     (pin "2")
+    (pin "3")
+    (pin "4")
+    (pin "5")
+    (pin "6")
+    (pin "8")
+    (pin "9")
+    (pin "10")
+    (pin "11")
+    (pin "12")
+    (pin "13")
+    (pin "14")
+    (pin "7")
   )
   (symbol (lib_id "power:GND") (at 106.68 182.88 0) (unit 1)
@@
   (symbol (lib_id "Device:R") (at 204.47 26.67 0) (unit 1)
     (in_bom yes) (on_board yes)
-    (property "Reference" "R?" (id 0) (at 205.74 25.4 0)
+    (property "Reference" "R7" (id 0) (at 205.74 25.4 0)
       (effects (font (size 1.27 1.27)) (justify left))
     )
@@
   (symbol (lib_id "74xx:74LS04") (at 149.86 177.8 0) (unit 6)
     (in_bom yes) (on_board yes) (fields_autoplaced)
-    (property "Reference" "U?" (id 0) (at 149.86 168.91 0))
+    (property "Reference" "U5" (id 0) (at 149.86 168.91 0))
     (property "Value" "74LS04" (id 1) (at 149.86 171.45 0))
     (property "Footprint" "" (id 2) (at 149.86 177.8 0)
@@
       (effects (font (size 1.27 1.27)) hide)
     )
+    (pin "1")
+    (pin "2")
+    (pin "3")
+    (pin "4")
+    (pin "5")
+    (pin "6")
+    (pin "8")
+    (pin "9")
+    (pin "10")
+    (pin "11")
     (pin "12")
     (pin "13")
+    (pin "14")
+    (pin "7")
   )
   (symbol (lib_id "power:GND") (at 62.23 69.85 0) (unit 1)
@@
       (effects (font (size 1.27 1.27)) hide)
     )
+    (pin "1")
+    (pin "2")
+    (pin "3")
+    (pin "4")
+    (pin "5")
+    (pin "6")
+    (pin "8")
+    (pin "9")
+    (pin "10")
+    (pin "11")
+    (pin "12")
+    (pin "13")
     (pin "14")
     (pin "7")
@@
       (effects (font (size 1.27 1.27)) hide)
     )
+    (pin "1")
+    (pin "2")
+    (pin "3")
+    (pin "4")
+    (pin "5")
+    (pin "6")
     (pin "8")
     (pin "9")
+    (pin "10")
+    (pin "11")
+    (pin "12")
+    (pin "13")
+    (pin "14")
+    (pin "7")
   )
   (symbol (lib_id "power:GND") (at 255.27 149.86 0) (unit 1)
@@
       (reference "#PWR031") (unit 1) (value "GND") (footprint "")
     )
+    (path "/49efb0be-60b6-44b1-8fc9-baffb4405f8d"
+      (reference "#PWR0101") (unit 1) (value "+5V") (footprint "")
+    )
+    (path "/4b5893ab-254a-408e-a775-ee4775099eb0"
+      (reference "#PWR0102") (unit 1) (value "GND") (footprint "")
+    )
     (path "/2a67836a-a519-4ab4-8b9f-f34934c8fe15"
-      (reference "#PWR?") (unit 1) (value "GND") (footprint "")
-    )
-    (path "/49efb0be-60b6-44b1-8fc9-baffb4405f8d"
-      (reference "#PWR?") (unit 1) (value "+5V") (footprint "")
-    )
-    (path "/4b5893ab-254a-408e-a775-ee4775099eb0"
-      (reference "#PWR?") (unit 1) (value "GND") (footprint "")
+      (reference "#PWR0103") (unit 1) (value "GND") (footprint "")
     )
     (path "/3b434176-5f57-4fd6-998d-219d1cbb5dbc"
@@
     )
     (path "/4a075904-512b-4037-94e6-7684d38257fa"
-      (reference "R?") (unit 1) (value "10k") (footprint "")
+      (reference "R6") (unit 1) (value "10k") (footprint "")
     )
     (path "/be356eb4-ff45-49c8-8d6a-27c498cf79f0"
-      (reference "R?") (unit 1) (value "10k") (footprint "")
+      (reference "R7") (unit 1) (value "10k") (footprint "")
     )
     (path "/19c97e1b-f7b7-42cd-a358-3bfa194d1c62"
@@
     )
     (path "/31661a0e-1491-413b-954a-1bcd23432c00"
-      (reference "U?") (unit 5) (value "74LS04") (footprint "")
+      (reference "U5") (unit 5) (value "74LS04") (footprint "")
     )
     (path "/cfa82190-a0ae-430f-bfc8-4113205faaf4"
-      (reference "U?") (unit 6) (value "74LS04") (footprint "")
-    )
-  )
+      (reference "U5") (unit 6) (value "74LS04") (footprint "")
+    )
+  )
