File: KiCAD files/Protoboard v2/Protoboardv2.kicad_pcb (KiCad board)
At the start: 2 copper layers, 99.7 x 69.8 mm, 250 parts, among them J1 Conn_02x05, J2 Conn_02x20, J3 Conn_01x04, J4 Conn_01x08, J5 Conn_01x08, J6 Conn_01x08, J7 Conn_01x06, J8 Conn_01x04, J9 Conn_01x06

Commit message: updates
Other:
- net class Default removed
- net class Power removed
