File: KiCAD files/Telnet_Server/Telnet_Server.kicad_sch (KiCad schematic)
At the start: 20 parts, among them J1 USB_B_Mini, J2 To PSU, J3 DB9_Male_MountingHoles, M1 ESP-01S_ESP8266, U1 LM317_TO-220, U3 ADM3022AN

Commit message: telnet server
Connections:
- net at R3.1: now also M1.6 (GPIO0); no longer M1.4 (GPIO2)
Changed lines of the file:
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@@
   (no_connect (at 166.37 83.82))
   (no_connect (at 194.31 83.82))
-  (no_connect (at 129.54 78.74))
+  (no_connect (at 129.54 81.28))
   (wire (pts (xy 204.47 92.71) (xy 213.36 92.71))
     (stroke (width 0) (type default) (color 0 0 0 0))
@@
     (stroke (width 0) (type default) (color 0 0 0 0))
   )
+  (wire (pts (xy 129.54 78.74) (xy 134.62 78.74))
+    (stroke (width 0) (type default) (color 0 0 0 0))
+  )
   (wire (pts (xy 161.29 57.15) (xy 161.29 72.39))
     (stroke (width 0) (type default) (color 0 0 0 0))
@@
   )
   (wire (pts (xy 194.31 57.15) (xy 204.47 57.15))
-    (stroke (width 0) (type default) (color 0 0 0 0))
-  )
-  (wire (pts (xy 129.54 81.28) (xy 134.62 81.28))
     (stroke (width 0) (type default) (color 0 0 0 0))
   )
@@
     (stroke (width 0) (type default) (color 0 0 0 0))
   )
-  (wire (pts (xy 134.62 81.28) (xy 134.62 111.76))
+  (wire (pts (xy 134.62 78.74) (xy 134.62 111.76))
     (stroke (width 0) (type default) (color 0 0 0 0))
   )

Commit message: telnet server update
Parts:
- added D1, D3: (no value), symbol Device:LED_Small
- added R1: (no value), symbol Device:R
- added R6: 330, symbol Device:R
- D2: renamed from D1; value (none) -> 1N4001; footprint (none) -> Diode_THT:D_DO-41_SOD81_P10.16mm_Horizontal
- Q1: value (none) -> BC547; footprint (none) -> Package_TO_SOT_THT:TO-92_Inline
- R4: renamed from R3; value (none) -> 270
- R5: renamed from R4; value (none) -> 10K
- U2: value (none) -> 4N25; footprint (none) -> Package_DIP:DIP-6_W7.62mm
- renumbered R1 to R2, R2 to R3
Connections:
- net +5V: now also R1.2, R6.2
- net GND: now also D1.1 (K)
- net at D2.2 (A), J2.2 (Pin_2), Q1.1 (C): now also D3.1 (K)
- new net: D1.2 (A), R1.1
- new net: D3.2 (A), R6.1
Other:
- moved on the sheet: J2
