File: KiCAD files/PLC cards/DO-8/DO-8.kicad_sch (KiCad schematic)
At the start: 40 parts

Commit message: do8 and rs485
Parts:
- added D?: (no value), symbol Diode:1N4001
Changed lines of the file:
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@@
     (pin "3")
+  )
+  (symbol (lib_id "Diode:1N4001") (at 250.19 106.68 0) (unit 1)
+    (in_bom yes) (on_board yes) (fields_autoplaced)
+    (property "Reference" "D?" (id 0) (at 250.19 100.33 0))
+    (property "Value" "" (id 1) (at 250.19 102.87 0))
+    (property "Footprint" "" (id 2) (at 250.19 111.125 0)
+      (effects (font (size 1.27 1.27)) hide)
+    )
+    (property "Datasheet" "http://www.vishay.com/docs/88503/1n4001.pdf" (id 3) (at 250.19 106.68 0)
+      (effects (font (size 1.27 1.27)) hide)
+    )
+    (pin "1")
+    (pin "2")
   )
   (symbol (lib_id "Device:LED_Small") (at 165.1 99.06 0) (mirror y) (unit 1)
@@
       (reference "D?") (unit 1) (value "LED_Small") (footprint "")
     )
+    (path "/bb9a7083-9ca4-4483-aa95-8301b4c105d2"
+      (reference "D?") (unit 1) (value "1N4001") (footprint "Diode_THT:D_DO-41_SOD81_P10.16mm_Horizontal")
+    )
     (path "/bdb7f7cf-e09e-4da7-935b-ec4e6268cca9"
