File: KiCAD files/PLC cards/DO-8/DO-8.kicad_sch (KiCad schematic)
At the start: 40 parts

Commit message: do-8
Parts:
- removed D? (x7): LED_Small, symbol Device:LED_Small
- removed D?: (no value), symbol Device:LED_Small
- removed J? (x8): (no value), symbol Connector:Conn_01x03_Female
- removed RN?: 220, Resistor_THT:R_Array_SIP5, symbol Device:R_Network04
- removed RN?: (no value), Resistor_THT:R_Array_SIP5, symbol Device:R_Network04
- removed U? (x7): 4N25, Package_DIP:DIP-6_W7.62mm, symbol Isolator:4N25
- removed U?: (no value), symbol Isolator:4N25
- added D? (x8): LED_Small, symbol Device:LED_Small
- added D? (x8): 1N4001, Diode_THT:D_DO-41_SOD81_P10.16mm_Horizontal, symbol Diode:1N4001
- added J? (x2): Conn_01x16_Female, symbol Connector:Conn_01x16_Female
- added K? (x8): SRD-05VDC-SL-C, MyStuff:Relay_SPDT_Songel-15x19mm, symbol Relay:Y14x-1C-xxDS
- C? (x2): value (none) -> 10nF
- C? (x2): value (none) -> 33pF
- J?: value (none) -> RS485
- J?: value (none) -> end
- J?: value (none) -> FS
- R?: value (none) -> 220
- RN?: value (none) -> 10k; footprint (none) -> Resistor_THT:R_Array_SIP5
- U?: value (none) -> SN75176AP; footprint (none) -> Package_DIP:DIP-8_W7.62mm
- U?: value (none) -> FM24C64B; footprint (none) -> Package_SO:SOIC-8_3.9x4.9mm_P1.27mm
- U?: value (none) -> AT89C4051-24P; footprint (none) -> Package_DIP:DIP-20_W7.62mm
- Y?: value (none) -> 11.059MHz
Connections:
- net +5V: now also D?.2 (A), D?.2 (A), D?.2 (A), D?.2 (A), D?.2 (A), D?.2 (A), D?.2 (A), D?.2 (A), K?.3, K?.3, K?.3, K?.3, K?.3, K?.3, K?.3, K?.3
- net Earth_Protective: now also J?.12 (Pin_12), J?.12 (Pin_12), J?.16 (Pin_16), J?.16 (Pin_16), J?.4 (Pin_4), J?.4 (Pin_4), J?.8 (Pin_8), J?.8 (Pin_8)
- net at U?.15 (P1.3): now also D?.1 (K)
- net at U?.16 (P1.4): now also D?.1 (K)
- net at U?.19 (P1.7): now also D?.1 (K)
- net at RN?.4 (R3), U?.12 (P1.0): now also D?.1 (K)
- net at RN?.5 (R4), U?.13 (P1.1): now also D?.1 (K)
- net at U?.14 (P1.2): now also D?.1 (K)
- net at U?.17 (P1.5): now also D?.1 (K)
- net at U?.18 (P1.6): now also D?.1 (K)
- new net: D?.1 (K), D?.2 (A), K?.4 (x8)
- new net: J?.2 (Pin_2), K?.1 (x2)
- new net: J?.1 (Pin_1), K?.2 (x2)
- new net: J?.3 (Pin_3), K?.5 (x2)
- new net: J?.14 (Pin_14), K?.1 (x2)
- new net: J?.13 (Pin_13), K?.2 (x2)
- new net: J?.15 (Pin_15), K?.5 (x2)
- new net: J?.10 (Pin_10), K?.1 (x2)
- new net: J?.9 (Pin_9), K?.2 (x2)
- new net: J?.11 (Pin_11), K?.5 (x2)
- new net: J?.6 (Pin_6), K?.1 (x2)
- new net: J?.5 (Pin_5), K?.2 (x2)
- new net: J?.7 (Pin_7), K?.5 (x2)
- no-connect marks 10 -> 2
Other:
- moved on the sheet: C?, J?, R?, RN?, U?, Y?
