File: KiCAD files/PLC cards/DI-16/DI-16/DI-16.kicad_sch (KiCad schematic)
At the start: 19 parts

Commit message: pcbs
Parts:
- U3: renamed from U?; value (none) -> 74LS241
- gave numbers to parts that had none: 18
Connections:
- net SCL: now also RN1.2 (R1); no longer RN1.3 (R2)
- net SDA: now also RN1.3 (R2); no longer RN1.2 (R1)
Other:
- moved on the sheet: C1, C2, C3, C4, C5, C6, C7, J1, J2, J3, J4, R1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

Commit message: pcbs
Parts:
- RN1: value R_Network04 -> (none)
Changed lines of the file:
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@@
       (effects (font (size 1.27 1.27)) (justify left))
     )
-    (property "Value" "R_Network04" (id 1) (at 106.68 34.2899 0)
+    (property "Value" "" (id 1) (at 106.68 34.2899 0)
       (effects (font (size 1.27 1.27)) (justify left))
     )
@@
       (effects (font (size 1.27 1.27)) hide)
     )
-    (property "Value" "" (id 1) (at 238.76 129.54 0))
+    (property "Value" "PWR_FLAG" (id 1) (at 238.76 129.54 0))
     (property "Footprint" "" (id 2) (at 238.76 134.62 0)
       (effects (font (size 1.27 1.27)) hide)
@@
     )
     (path "/7756fa9b-0668-423f-8c55-701a1a1b7d1b/6d905af8-fdc3-480f-b23d-c850c4760595"
-      (reference "R2") (unit 1) (value "R_Small") (footprint "")
+      (reference "R2") (unit 1) (value "3k") (footprint "")
     )
     (path "/7756fa9b-0668-423f-8c55-701a1a1b7d1b/afd5b057-559a-4a5f-b3f1-1584a8e14682"
-      (reference "R3") (unit 1) (value "R_Small") (footprint "")
+      (reference "R3") (unit 1) (value "3k") (footprint "")
     )
     (path "/7756fa9b-0668-423f-8c55-701a1a1b7d1b/ad297e62-78ee-4605-860b-e7900137ef2a"
-      (reference "R4") (unit 1) (value "R_Small") (footprint "")
+      (reference "R4") (unit 1) (value "3k") (footprint "")
     )
     (path "/7756fa9b-0668-423f-8c55-701a1a1b7d1b/500b8de0-a5e3-4d03-a680-9979014a4d42"
-      (reference "R5") (unit 1) (value "R_Small") (footprint "")
+      (reference "R5") (unit 1) (value "3k") (footprint "")
     )
     (path "/7756fa9b-0668-423f-8c55-701a1a1b7d1b/c100734c-6507-4449-b15b-7fc2d8cfd81f"
-      (reference "R6") (unit 1) (value "R_Small") (footprint "")
+      (reference "R6") (unit 1) (value "3k") (footprint "")
     )
     (path "/7756fa9b-0668-423f-8c55-701a1a1b7d1b/f1ce561f-1489-4028-90fc-b22a58ee5112"
-      (reference "R7") (unit 1) (value "R_Small") (footprint "")
+      (reference "R7") (unit 1) (value "3k") (footprint "")
     )
     (path "/7756fa9b-0668-423f-8c55-701a1a1b7d1b/355460e6-380a-4454-93f2-9b4830d944ec"
-      (reference "R8") (unit 1) (value "R_Small") (footprint "")
+      (reference "R8") (unit 1) (value "3k") (footprint "")
     )
     (path "/7756fa9b-0668-423f-8c55-701a1a1b7d1b/8a45ff39-b1ad-4bf3-ad61-b9e718d2317e"
-      (reference "R9") (unit 1) (value "R_Small") (footprint "")
+      (reference "R9") (unit 1) (value "3k") (footprint "")
     )
     (path "/c516f7ec-34d5-48ab-b054-a8258417558c/07cc1e71-cc98-4ab2-b0ab-f3e09bbf80a0"
-      (reference "R10") (unit 1) (value "R_Small") (footprint "")
+      (reference "R10") (unit 1) (value "3k") (footprint "")
     )
     (path "/c516f7ec-34d5-48ab-b054-a8258417558c/6edb5287-a8e6-4f0c-8133-a85add57394b"
-      (reference "R11") (unit 1) (value "R_Small") (footprint "")
+      (reference "R11") (unit 1) (value "3k") (footprint "")
     )
     (path "/c516f7ec-34d5-48ab-b054-a8258417558c/632eb4ea-ff2b-4b50-9afa-4d5754b2edf3"
-      (reference "R12") (unit 1) (value "R_Small") (footprint "")
+      (reference "R12") (unit 1) (value "3k") (footprint "")
     )
     (path "/c516f7ec-34d5-48ab-b054-a8258417558c/d6334727-0221-41d3-8be7-43a77f1b8196"
-      (reference "R13") (unit 1) (value "R_Small") (footprint "")
+      (reference "R13") (unit 1) (value "3k") (footprint "")
     )
     (path "/c516f7ec-34d5-48ab-b054-a8258417558c/520a51ec-66f0-4528-898c-4f9943769291"
-      (reference "R14") (unit 1) (value "R_Small") (footprint "")
+      (reference "R14") (unit 1) (value "3k") (footprint "")
     )
     (path "/c516f7ec-34d5-48ab-b054-a8258417558c/c39a4188-7c20-47ea-8ea2-a33de9fa821c"
-      (reference "R15") (unit 1) (value "R_Small") (footprint "")
+      (reference "R15") (unit 1) (value "3k") (footprint "")
     )
     (path "/c516f7ec-34d5-48ab-b054-a8258417558c/07137f10-3978-4e42-940d-5ae2c1ff290f"
-      (reference "R16") (unit 1) (value "R_Small") (footprint "")
+      (reference "R16") (unit 1) (value "3k") (footprint "")
     )
     (path "/c516f7ec-34d5-48ab-b054-a8258417558c/2db81ea2-6ccf-49bc-8af6-82b73db1d20d"
-      (reference "R17") (unit 1) (value "R_Small") (footprint "")
+      (reference "R17") (unit 1) (value "3k") (footprint "")
     )
     (path "/46a4ea48-c711-4ba8-bcde-157460e3d207"
-      (reference "RN1") (unit 1) (value "R_Network04") (footprint "Resistor_THT:R_Array_SIP5")
+      (reference "RN1") (unit 1) (value "10k") (footprint "Resistor_THT:R_Array_SIP5")
     )
     (path "/7756fa9b-0668-423f-8c55-701a1a1b7d1b/be6350f0-a816-4d57-b657-afba9d1682e8"

Commit message: DI & DO updates
Parts:
- J1: value Conn_01x02 -> (none)
- RN1: value (none) -> 10k
Changed lines of the file:
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@@
       (effects (font (size 1.27 1.27)) (justify left))
     )
-    (property "Value" "" (id 1) (at 106.68 34.2899 0)
+    (property "Value" "10k" (id 1) (at 106.68 34.2899 0)
       (effects (font (size 1.27 1.27)) (justify left))
     )
@@
   (symbol (lib_id "Connector_Generic:Conn_01x02") (at 50.292 141.224 0) (mirror y) (unit 1)
     (in_bom yes) (on_board yes) (fields_autoplaced)
-    (property "Reference" "J1" (id 0) (at 50.292 134.874 0))
-    (property "Value" "Conn_01x02" (id 1) (at 50.292 137.414 0))
+    (property "Reference" "J1" (id 0) (at 50.292 134.62 0))
+    (property "Value" "" (id 1) (at 50.292 137.16 0))
     (property "Footprint" "" (id 2) (at 50.292 141.224 0)
       (effects (font (size 1.27 1.27)) hide)
@@
       (reference "#PWR036") (unit 1) (value "GND") (footprint "")
     )
-    (path "/7756fa9b-0668-423f-8c55-701a1a1b7d1b/9975ff27-218d-40a0-839b-08ceb6270cd4"
-      (reference "#PWR037") (unit 1) (value "Earth_Protective") (footprint "")
-    )
     (path "/c516f7ec-34d5-48ab-b054-a8258417558c/f4f1dc14-6014-458c-aa74-cfb27d95d3b6"
       (reference "#PWR038") (unit 1) (value "+5V") (footprint "")
@@
       (reference "#PWR043") (unit 1) (value "GND") (footprint "")
     )
-    (path "/c516f7ec-34d5-48ab-b054-a8258417558c/a4a76260-beaa-42d5-a380-c55c69277fe7"
-      (reference "#PWR044") (unit 1) (value "Earth_Protective") (footprint "")
-    )
     (path "/c516f7ec-34d5-48ab-b054-a8258417558c/aab3ada9-e7cd-4cb0-9101-762f9c4c6d82"
       (reference "#PWR045") (unit 1) (value "+5V") (footprint "")
@@
       (reference "#PWR050") (unit 1) (value "GND") (footprint "")
     )
-    (path "/c516f7ec-34d5-48ab-b054-a8258417558c/febc858c-4b6b-408d-94d2-7d45dff56bc4"
-      (reference "#PWR051") (unit 1) (value "Earth_Protective") (footprint "")
+    (path "/c516f7ec-34d5-48ab-b054-a8258417558c/1bb158ad-8432-4708-b927-e62bf2eaeced"
+      (reference "#PWR?") (unit 1) (value "Earth_Protective") (footprint "")
+    )
+    (path "/7756fa9b-0668-423f-8c55-701a1a1b7d1b/20e6d2d8-cc77-4536-8909-c0a4b5d338a2"
+      (reference "#PWR?") (unit 1) (value "Earth_Protective") (footprint "")
+    )
+    (path "/c516f7ec-34d5-48ab-b054-a8258417558c/276b2729-c8ba-48f7-be81-25833c3e1e23"
+      (reference "#PWR?") (unit 1) (value "Earth_Protective") (footprint "")
     )
     (path "/f53a99df-250f-4a1e-afbf-bad4642182eb"
@@
     )
     (path "/827067f8-941d-41b2-a241-7467adb8ddca"
-      (reference "J1") (unit 1) (value "Conn_01x02") (footprint "")
+      (reference "J1") (unit 1) (value "terminal") (footprint "")
     )
     (path "/b6a23e91-69f5-44fe-a673-f9196ceb2100"
@@
       (reference "J5") (unit 1) (value "Conn_02x06_Odd_Even") (footprint "")
     )
-    (path "/7756fa9b-0668-423f-8c55-701a1a1b7d1b/3699b637-1b8b-487c-8c61-2299cec6c16b"
+    (path "/7756fa9b-0668-423f-8c55-701a1a1b7d1b/887ad99a-ff2c-421c-a746-b7864028919b"
       (reference "J6") (unit 1) (value "Conn_02x06_Odd_Even") (footprint "")
     )
-    (path "/c516f7ec-34d5-48ab-b054-a8258417558c/317f957b-f55a-4770-aa19-d699a1319be0"
+    (path "/c516f7ec-34d5-48ab-b054-a8258417558c/1aa267b4-7cd6-4cc6-93fd-b11ca94f57c2"
       (reference "J7") (unit 1) (value "Conn_02x06_Odd_Even") (footprint "")
     )
-    (path "/c516f7ec-34d5-48ab-b054-a8258417558c/52e7ed00-d24b-4444-a6c4-bfea26f5951f"
+    (path "/c516f7ec-34d5-48ab-b054-a8258417558c/e695e33c-9e3d-4296-8d28-9c5c56ef9e93"
       (reference "J8") (unit 1) (value "Conn_02x06_Odd_Even") (footprint "")
     )
