File: KiCAD files/Proton cards/RS485/RS485.kicad_sch (KiCad schematic)
At the start: 26 parts

Commit message: RS485
Parts:
- removed C? (x2): 22pF, Capacitor_THT:C_Disc_D3.8mm_W2.6mm_P2.50mm, symbol Device:C
- removed C? (x6): 10nF, Capacitor_THT:C_Disc_D3.8mm_W2.6mm_P2.50mm, symbol Device:C
- removed C?: 10uF, symbol Device:C_Polarized
- removed J?: Signal Buss, Connector_PinHeader_2.54mm:PinHeader_2x20_P2.54mm_Vertical, symbol Connector_Generic:Conn_02x20_Odd_Even
- removed J?: Power Bus, Connector_PinHeader_2.54mm:PinHeader_2x05_P2.54mm_Vertical, symbol Connector_Generic:Conn_02x05_Odd_Even
- removed J?: Card addr, Connector_PinHeader_2.54mm:PinHeader_2x04_P2.54mm_Vertical, symbol Connector_Generic:Conn_02x04_Odd_Even
- removed R?: (no value), symbol Device:R
- removed RN?: 4x10k, Resistor_THT:R_Array_SIP5, symbol Device:R_Network04
- removed U?: ATmega328P-PU, Package_DIP:DIP-28_W7.62mm_Socket_LongPads, symbol TTY-rescue:ATmega328P-PU-MCU_Microchip_ATmega
- removed U? (x3): (no value), symbol 74xx:74LS00
- removed U?: 74LS85, Package_DIP:DIP-16_W7.62mm_Socket_LongPads, symbol 74xx:74LS85
- removed U?: 74LS245, Package_DIP:DIP-20_W7.62mm_Socket_LongPads, symbol 74xx:74LS245
- removed U? (x2): 74LS74, Package_DIP:DIP-14_W7.62mm_Socket_LongPads, symbol 74xx:74LS74
- removed U?: (no value), symbol Interface_UART:SN75176AP
- removed U? (x2): 74LS00, Package_DIP:DIP-14_W7.62mm_Socket_LongPads, symbol 74xx:74LS00
- removed Y?: 20MHz, Crystal:Crystal_HC49-U_Vertical, symbol Device:Crystal
- added C1, C10, C11, C12, C13, C14, C5, C6, C9: 10nF, Capacitor_THT:C_Disc_D3.8mm_W2.6mm_P2.50mm, symbol Device:C_Small
- added C2, C3, C7, C8: 22pF, Capacitor_THT:C_Disc_D3.8mm_W2.6mm_P2.50mm, symbol Device:C_Small
- added C4: 10uF, symbol Device:C_Polarized_Small
- added J1, J6: (no value), symbol Connector_Generic:Conn_01x03
- added J2: Power Bus, Connector_PinHeader_2.54mm:PinHeader_2x05_P2.54mm_Vertical, symbol Connector_Generic:Conn_02x05_Odd_Even
- added J3: (no value), symbol Connector_Generic:Conn_01x02
- added J4: Signal Buss, Connector_PinHeader_2.54mm:PinHeader_2x20_P2.54mm_Vertical, symbol Connector_Generic:Conn_02x20_Odd_Even
- added J5: Card addr, Connector_PinHeader_2.54mm:PinHeader_2x04_P2.54mm_Vertical, symbol Connector_Generic:Conn_02x04_Odd_Even
- added J7: terminal, symbol Connector_Generic:Conn_01x02
- added R1: (no value), symbol Device:R_Small
- added R2: 150, symbol Device:R_Small
- added RN1, RN2: 4x10k, Resistor_THT:R_Array_SIP5, symbol Device:R_Network04
- added U1: (no value), symbol Interface_UART:SN75176AP
- added U2, U5: ATmega328P-PU, Package_DIP:DIP-28_W7.62mm_Socket_LongPads, symbol TTY-rescue:ATmega328P-PU-MCU_Microchip_ATmega
- added U3: SN75176AP, Package_DIP:DIP-8_W7.62mm, symbol Interface_UART:SN75176AP
- added U4: 74LS85, Package_DIP:DIP-16_W7.62mm_Socket_LongPads, symbol 74xx:74LS85
- added U6: 74LS00, Package_DIP:DIP-14_W7.62mm_Socket_LongPads, symbol 74xx:74LS00
- added U7: (no value), symbol 74xx:74LS08
- added U8: 74LS74, Package_DIP:DIP-14_W7.62mm_Socket_LongPads, symbol 74xx:74LS74
- added U9: 74LS245, Package_DIP:DIP-20_W7.62mm_Socket_LongPads, symbol 74xx:74LS245
- added Y1: (no value), Crystal:Crystal_HC49-U_Vertical, symbol Device:Crystal_Small
- added Y2: 11.059MHz, Crystal:Crystal_HC49-U_Vertical, symbol Device:Crystal_Small
Connections:
- net +12V: now also J2.5 (Pin_5), J2.6 (Pin_6)
- net +5V: now also C1.2, C10.2, C11.2, C12.2, C13.2, C14.2, C4.1, C5.2, C6.2, C9.2, J2.3 (Pin_3), J2.4 (Pin_4), RN1.1 (common), RN2.1 (common), U1.8 (VCC), U2.20 (AVCC), U2.7 (VCC), U3.8 (VCC), U4.16 (VCC), U5.20 (AVCC), U5.7 (VCC), U6.14 (VCC), U7.14 (VCC), U8.10 (~{S}), U8.13 (~{R}), U8.14 (VCC), U8.2 (D), U8.4 (~{S}), U9.20 (VCC)
- net B00: now also U2.14 (PB0), U5.14 (PB0), U9.18 (B0)
- net B01: now also U2.15 (PB1), U5.15 (PB1), U9.17 (B1)
- net B02: now also U2.16 (PB2), U5.16 (PB2), U9.16 (B2)
- net B03: now also U2.5 (PD3), U5.5 (PD3), U9.15 (B3)
- net B04: now also U2.6 (PD4), U5.6 (PD4), U9.14 (B4)
- net B05: now also U2.11 (PD5), U5.11 (PD5), U9.13 (B5)
- net B06: now also U2.12 (PD6), U5.12 (PD6), U9.12 (B6)
- net B07: now also U2.13 (PD7), U5.13 (PD7), U9.11 (B7)
- net GND: now also C1.1, C10.1, C11.1, C12.1, C13.1, C14.1, C2.2, C3.2, C4.2, C5.1, C6.1, C7.2, C8.2, C9.1, J2.1 (Pin_1), J2.10 (Pin_10), J2.2 (Pin_2), J2.9 (Pin_9), J5.1 (Pin_1), J5.3 (Pin_3), J5.5 (Pin_5), J5.7 (Pin_7), U1.5 (GND), U2.22 (GND), U2.8 (GND), U3.5 (GND), U4.2 (Ia<b), U4.4 (Ia>b), U4.8 (GND), U5.22 (GND), U5.8 (GND), U6.7 (GND), U7.7 (GND), U8.11 (C), U8.12 (D), U8.7 (GND), U9.10 (GND)
- net a00: now also J4.2 (Pin_2), U6.12, U6.13, U6.5
- net a01: now also J4.1 (Pin_1), U2.23 (PC0), U5.23 (PC0)
- net a04: now also J4.6 (Pin_6), U4.10 (A0)
- net a05: now also J4.5 (Pin_5), U4.12 (A1)
- net a06: now also J4.8 (Pin_8), U4.13 (A2)
- net a07: now also J4.7 (Pin_7), U4.15 (A3)
- net d00: now also J4.18 (Pin_18), U9.2 (A0)
- net d01: now also J4.17 (Pin_17), U9.3 (A1)
- net d02: now also J4.20 (Pin_20), U9.4 (A2)
- net d03: now also J4.19 (Pin_19), U9.5 (A3)
- net d04: now also J4.22 (Pin_22), U9.6 (A4)
- net d05: now also J4.21 (Pin_21), U9.7 (A5)
- net d06: now also J4.24 (Pin_24), U9.8 (A6)
- net d07: now also J4.23 (Pin_23), U9.9 (A7)
- net iorq: now also J4.28 (Pin_28), U6.1, U6.2
- net rd: now also J4.27 (Pin_27), U2.24 (PC1), U5.24 (PC1), U9.1 (A->B)
- net reset: now also J4.40 (Pin_40), U2.1 (~{RESET}/PC6), U5.1 (~{RESET}/PC6), U7.2
- net v1: now also J2.7 (Pin_7), J2.8 (Pin_8)
- net wait: now also J4.32 (Pin_32), U8.6 (~{Q})
- net wr: now also J4.25 (Pin_25), U2.25 (PC2), U5.25 (PC2)
- new net: J6.2 (Pin_2), R2.1, U3.6 (A)
- new net: J6.1 (Pin_1), J7.2 (Pin_2), U3.7 (B)
- new net: C2.1, U2.9 (XTAL1/PB6), Y1.1
- new net: C3.1, U2.10 (XTAL2/PB7), Y1.2
- new net: J7.1 (Pin_1), R2.2
- new net: J1.2 (Pin_2), R1.1, U1.6 (A)
- new net: J1.1 (Pin_1), J3.2 (Pin_2), U1.7 (B)
- new net: U7.8, U9.19 (CE)
- new net: J3.1 (Pin_1), R1.2
- new net: C8.1, U5.10 (XTAL2/PB7), Y2.2
- new net: J5.2 (Pin_2), RN1.2 (R1), U4.1 (B3)
- new net: J5.4 (Pin_4), RN1.3 (R2), U4.14 (B2)
- new net: J5.6 (Pin_6), RN1.4 (R3), U4.11 (B1)
- new net: J5.8 (Pin_8), RN1.5 (R4), U4.9 (B0)
- new net: U7.1, U7.6
- new net: U7.3, U8.1 (~{R})
- new net: C7.1, U5.9 (XTAL1/PB6), Y2.1
- new net: U6.10, U6.11
- new net: U4.3 (Ia=b), U6.3
- new net: U4.6 (Oa=b), U6.4, U6.9, U8.3 (C)
- new net CS0: U2.4 (PD2), U6.8, U7.10
- new net CS1: U5.4 (PD2), U6.6, U7.9
- new net DE0: U1.2 (~{RE}), U1.3 (DE), U2.27 (PC4)
- new net DE1: U3.2 (~{RE}), U3.3 (DE), U5.27 (PC4)
- new net Earth_Protective: J1.3 (Pin_3), J6.3 (Pin_3)
- new net RSM0: RN2.2 (R1), U2.26 (PC3), U7.4
- new net RSM1: RN2.3 (R2), U5.26 (PC3), U7.5
- new net RX0: U1.1 (R), U2.2 (PD0)
- new net RX1: U3.1 (R), U5.2 (PD0)
- new net TX0: U1.4 (D), U2.3 (PD1)
- new net TX1: U3.4 (D), U5.3 (PD1)
- no-connect marks 30 -> 41
