File: KiCAD files/Proton cards/RS485/PiggyBackRS485/PiggyBackRS485.kicad_sch (KiCad schematic)
At the start: 10 parts

Commit message: rs485
Parts:
- U1, U2: renamed from U?; footprint Package_DIP:DIP-8_W7.62mm -> (none)
- gave numbers to parts that had none: 8
Other:
- moved on the sheet: C1, J1, J2, J3, J4, J5, R1, R2, U1, U2
