File: KiCAD files/BoilerCtrl/BoilerCtrl.kicad_sch (KiCad schematic)
At the start: 38 parts

Commit message: pt100
Parts:
- removed C? (x2): 47uF, symbol Device:C_Polarized_Small
- removed J?: I2C_bus, symbol Connector_Generic:Conn_02x02_Odd_Even
- removed U?: LM317L_TO92, Package_TO_SOT_THT:TO-92_Inline, symbol Regulator_Linear:LM317L_TO92
- added C?: 10uF, symbol Device:C_Polarized
- added C? (x2): 10nF, symbol Device:C_Small
- added J?: I2C ext, Connector_PinHeader_2.54mm:PinHeader_2x02_P2.54mm_Vertical, symbol Connector_Generic:Conn_02x02_Top_Bottom
- added R? (x2): (no value), symbol Device:R_Small
- added R?: 390, Resistor_THT:R_Axial_DIN0207_L6.3mm_D2.5mm_P10.16mm_Horizontal, symbol Device:R
- added R?: 240, Resistor_THT:R_Axial_DIN0207_L6.3mm_D2.5mm_P10.16mm_Horizontal, symbol Device:R
- added U?: LM317_TO-220, Package_TO_SOT_THT:TO-220-3_Vertical, symbol Regulator_Linear:LM317_TO-220
- R? (x2): value 10k -> 6.8k
Connections:
- net +5V: now also C?.1, J?.1 (Pin_1), C?.1, C?.1, J?.3 (Pin_3), U?.3 (VI)
- net GND: now also C?.2, J?.2 (Pin_2), J?.3 (Pin_3), C?.2, C?.2, C?.2, J?.4 (Pin_4), R?.2, R?.2
- net RX: now also J?.1 (Pin_1)
- net SCL: now also J?.2 (Pin_2)
- net SDA: now also J?.1 (Pin_1)
- net TS: no longer U?.24 (PC1)
- net TX: now also R?.1
- net +3V3: now reaches J?.3 (Pin_3)
- net +3V3: now also J?.7 (Pin_7), C?.1, R?.1, U?.2 (VO)
- net at J?.8 (Pin_8): now also R?.1, R?.2
- net HTS: now reaches J?.2 (Pin_2)
- net HTS: now also U?.24 (PC1)
- new net: R?.1, R?.2, U?.1 (ADJ)
- no-connect marks 16 -> 19
Other:
- moved on the sheet: C?, J?, U?E
