File: KiCAD files/PT100/PT100.kicad_sch (KiCad schematic)
At the start: 23 parts, among them J1 PT100, J2 Power, J3 Comm, U1 LM358, U2 ADC0804, U3 AT89C4051-24P, Y1 16MHz

Commit message: pt100
Parts:
- removed J1: PT100, symbol Connector:Conn_01x02_Male
- removed J2: Power, symbol Connector:Conn_01x03_Male
- removed J3: Comm, symbol Connector:Conn_01x04_Male
- removed U1: LM358, symbol Amplifier_Operational:LM358
- added C3: 10uF, symbol Device:C_Polarized_Small
- added J1: PT100, symbol Connector_Generic:Conn_01x02
- added J2: Power, symbol Connector_Generic:Conn_01x04
- added J3: Comm, symbol Connector_Generic:Conn_01x04
- added R6, R7, R8, R9: 24k, symbol Device:R_Small
- added RV1: 10k, symbol Device:R_Potentiometer_Trim
- added RV2: 1k, symbol Device:R_Potentiometer_Trim
- added U1: LM324, symbol Amplifier_Operational:LM324
- C1, C2: value 3.3uF -> 10uF
- R4: value 5k6 -> 24k
- R5: value 150k -> 24k
- Y1: value 16MHz -> 24MHz
- renumbered C3 to C6, C6 to C7, C7 to C8, C8 to C9, R6 to R10, R7 to R11, R8 to R12
Connections:
- net +12V: now also J2.1 (Pin_1), U1.4 (V+)
- net +5V: now also J2.2 (Pin_2), J3.4 (Pin_4), RV2.1
- net GND: now also C3.2, J1.2 (Pin_2), J2.3 (Pin_3), J3.3 (Pin_3), R8.2, RV2.3
- net RX: now also J3.1 (Pin_1)
- net TX: now also J3.2 (Pin_2)
- net at R2.2, R3.1: now also U1.10 (+); no longer R4.2
- net at R5.1: now also RV1.2, RV1.3, U1.9 (-); no longer U2.6 (VIN+)
- net at R5.2: now also R7.1, U1.8; no longer R4.1
- net at R1.2: now also J1.1 (Pin_1), U1.3 (+)
- net at U2.9 (VREF/2): now also RV2.2
- new net: R6.2, R8.1, U1.5 (+)
- new net: R7.2, R9.1, U1.6 (-)
- new net: R9.2, U1.7, U2.6 (VIN+)
- new net: R4.1, R6.1, U1.1
- new net: R4.2, RV1.1, U1.2 (-)
- new net -12V: C3.1, J2.4 (Pin_4), U1.11 (V-)
- no-connect marks 2 -> 1
Other:
- moved on the sheet: C4, C5, C6, C7, C8, C9, R10, R11, R12, U2, U3, Y1

Commit message: pt100
Parts:
- Y1: value 24MHz -> (none)
Changed lines of the file:
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@@
       (effects (font (size 1.27 1.27)) (justify left))
     )
-    (property "Value" "24MHz" (id 1) (at 238.76 87.63 90)
+    (property "Value" "" (id 1) (at 233.68 87.63 90)
       (effects (font (size 1.27 1.27)) (justify left))
     )
@@
     )
     (path "/d4425a69-7786-4067-88c4-6c450a65597a"
-      (reference "Y1") (unit 1) (value "24MHz") (footprint "")
-    )
-  )
+      (reference "Y1") (unit 1) (value "11.059MHz") (footprint "")
+    )
+  )

Commit message: PT100
Parts:
- removed C1, C2, C3: 10uF, symbol Device:C_Polarized_Small
- removed J2: Power, symbol Connector_Generic:Conn_01x04
- added R13: (no value), symbol Device:R_Small
- Y1: value (none) -> 11.059MHz
- renumbered C4 to C1, C5 to C2, C7 to C3, C6 to C4, C8 to C5, C9 to C6, J3 to J2
Connections:
- net at U3.11 (P3.7): now also R13.1
- new net AC_part/CTRL: R13.2
- no-connect marks 1 -> 0
Other:
- added sheet AC_part (untitled.kicad_sch)
- moved on the sheet: C1, C2, C3, U1E
