File: KiCAD files/PLC cards/DO-08/DO-08.kicad_sch (KiCad schematic)
At the start: 57 parts

Commit message: PCBs
Parts:
- removed D? (x8): 1N4001, Diode_THT:D_DO-41_SOD81_P10.16mm_Horizontal, symbol Diode:1N4001
- removed D?: (no value), symbol Device:LED_Small
- removed D? (x7): LED_Small, symbol Device:LED_Small
- removed K? (x8): SRD-05VDC-SL-C, MyStuff:Relay_SPDT_Songel-15x19mm, symbol Relay:Y14x-1C-xxDS
- removed Q? (x8): BC328, Package_TO_SOT_THT:TO-92_Inline, symbol Transistor_BJT:BC328
- removed R? (x7): 15k, symbol Device:R_Small
- removed R?: (no value), symbol Device:R_Small
- removed RN? (x2): (no value), Resistor_THT:R_Array_SIP5, symbol Device:R_Network04
- C1, C2: renamed from C?; value (none) -> 33pF
- C4: renamed from C?; value (none) -> 10nF
- J2: renamed from J?; value (none) -> factory setup
- J3: renamed from J?; value (none) -> RS485
- J4: renamed from J?; value (none) -> TTL comm
- Y1: renamed from Y?; value (none) -> 11.059MHz
- gave numbers to parts that had none: 8
Connections:
- net Relays/D07: now reaches U1.19 (P1.7)
- net Relays/D05: now reaches U1.17 (P1.5)
- net Relays/D02: now reaches U1.14 (P1.2)
- net Relays/D01: now reaches RN1.4 (R3), U1.13 (P1.1)
- net Relays/D06: now reaches U1.18 (P1.6)
- net Relays/D00: now reaches RN1.5 (R4), U1.12 (P1.0)
- net Relays/D03: now reaches U1.15 (P1.3)
- net Relays/D04: now reaches U1.16 (P1.4)
Other:
- added sheet Relays (untitled.kicad_sch)
- moved on the sheet: C1, C2, C3, C4, C5, J1, J2, J3, J4, R1, RN1, U1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

Commit message: pcbs
Parts:
- RN1: value R_Network04 -> (none)
- renumbered C5 to C4, C4 to C5, U3 to U2, U2 to U3
Connections:
- net SCL: now also RN1.2 (R1); no longer RN1.3 (R2)
- net SDA: now also RN1.3 (R2); no longer RN1.2 (R1)
Other:
- moved on the sheet: C1, C2, C3, C4, C5, J1, J2, J3, J4, R1, RN1, U1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

Commit message: pcbs
Parts:
- RN1: value (none) -> 10k
Changed lines of the file:
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@@
       (effects (font (size 1.27 1.27)) (justify left))
     )
-    (property "Value" "" (id 1) (at 153.67 48.2599 0)
+    (property "Value" "10k" (id 1) (at 153.67 48.2599 0)
       (effects (font (size 1.27 1.27)) (justify left))
     )
@@
     )
     (path "/63220742-c59d-4aab-99e4-fb52a628905e/4117bd78-9085-4a22-9861-944b06bea1fa"
-      (reference "RN2") (unit 1) (value "220") (footprint "Resistor_THT:R_Array_SIP5")
+      (reference "RN2") (unit 1) (value "330") (footprint "Resistor_THT:R_Array_SIP5")
     )
     (path "/63220742-c59d-4aab-99e4-fb52a628905e/2896ffab-efaa-4523-84f4-c2df3ed62417"
-      (reference "RN3") (unit 1) (value "220") (footprint "Resistor_THT:R_Array_SIP5")
+      (reference "RN3") (unit 1) (value "330") (footprint "Resistor_THT:R_Array_SIP5")
     )
     (path "/ab8b0540-9c9f-4195-88f5-7bed0b0a8ed6"

Commit message: DI & DO updates
Parts:
- J1: value Conn_01x02 -> (none)
Changed lines of the file:
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@@
   (symbol (lib_id "Connector_Generic:Conn_01x02") (at 97.282 155.194 0) (mirror y) (unit 1)
     (in_bom yes) (on_board yes) (fields_autoplaced)
-    (property "Reference" "J1" (id 0) (at 97.282 148.844 0))
-    (property "Value" "Conn_01x02" (id 1) (at 97.282 151.384 0))
+    (property "Reference" "J1" (id 0) (at 97.282 148.59 0))
+    (property "Value" "" (id 1) (at 97.282 151.13 0))
     (property "Footprint" "" (id 2) (at 97.282 155.194 0)
       (effects (font (size 1.27 1.27)) hide)
@@
     )
     (path "/daa15e48-77cb-44c9-99cc-50bca0d156eb"
-      (reference "J1") (unit 1) (value "Conn_01x02") (footprint "")
+      (reference "J1") (unit 1) (value "terminal") (footprint "")
     )
     (path "/76039f1a-afec-47d2-9df2-342db8f33034"

Commit message: PT100
Parts:
- added C?: 47uF, symbol Device:C_Polarized_Small
- added C?: (no value), symbol Device:C_Polarized_Small
- added H? (x2): (no value), symbol Mechanical:MountingHole
- added H? (x6): MountingHole, symbol Mechanical:MountingHole
- added J?: (no value), symbol Connector_Generic:Conn_01x03
- J1: value (none) -> terminal
Connections:
- net +5V: now also C?.1
- net GND: now also C?.2, C?.2, J?.2 (Pin_2)
- new net +24V: C?.1, J?.1 (Pin_1)
- new net Earth_Protective: J?.3 (Pin_3)
Other:
- note added: "buck"
