File: KiCAD files/PLC cards/DI-08/DI-08.kicad_sch (KiCad schematic)
At the start: 15 parts, among them J1 terminal, J2 factory setup, J3 RS485, J4 TTL comm, U1 AT89C4051-24P, U2 SN75176AP, U3 FM24C64B, Y1 11.059MHz

Commit message: misc.
Parts:
- added J?: I2C bus, symbol Connector_Generic:Conn_01x04
Connections:
- net +5V: now also J?.1 (Pin_1)
- net GND: now also J?.4 (Pin_4)
- net SCL: now also J?.3 (Pin_3)
- net SDA: now also J?.2 (Pin_2)
Other:
- note added: "+5V SDA SCL GND"
Changed lines of the file:
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@@
   (junction (at 146.05 83.82) (diameter 0) (color 0 0 0 0)
   )
+  (junction (at 148.59 107.95) (diameter 0) (color 0 0 0 0)
+  )
   (junction (at 99.568 63.5) (diameter 0) (color 0 0 0 0)
   )
@@
   )
   (junction (at 180.086 120.65) (diameter 0) (color 0 0 0 0)
+  )
+  (junction (at 146.05 113.03) (diameter 0) (color 0 0 0 0)
   )
   (junction (at 148.59 81.28) (diameter 0) (color 0 0 0 0)
@@
     (stroke (width 0) (type default) (color 0 0 0 0))
   )
+  (wire (pts (xy 146.05 134.62) (xy 146.05 113.03))
+    (stroke (width 0) (type default) (color 0 0 0 0))
+  )
   (wire (pts (xy 96.52 63.5) (xy 99.568 63.5))
     (stroke (width 0) (type default) (color 0 0 0 0))
@@
     (stroke (width 0) (type default) (color 0 0 0 0))
   )
+  (wire (pts (xy 160.02 125.73) (xy 160.02 129.54))
+    (stroke (width 0) (type default) (color 0 0 0 0))
+  )
   (wire (pts (xy 153.67 42.926) (xy 153.67 53.34))
     (stroke (width 0) (type default) (color 0 0 0 0))
@@
     (stroke (width 0) (type default) (color 0 0 0 0))
   )
+  (wire (pts (xy 160.02 137.16) (xy 160.02 140.97))
+    (stroke (width 0) (type default) (color 0 0 0 0))
+  )
   (wire (pts (xy 132.08 76.2) (xy 143.51 76.2))
     (stroke (width 0) (type default) (color 0 0 0 0))
@@
     (stroke (width 0) (type default) (color 0 0 0 0))
   )
+  (wire (pts (xy 160.02 134.62) (xy 146.05 134.62))
+    (stroke (width 0) (type default) (color 0 0 0 0))
+  )
   (wire (pts (xy 132.08 78.74) (xy 140.97 78.74))
     (stroke (width 0) (type default) (color 0 0 0 0))
   )
+  (wire (pts (xy 148.59 132.08) (xy 148.59 107.95))
+    (stroke (width 0) (type default) (color 0 0 0 0))
+  )
   (wire (pts (xy 143.51 76.2) (xy 143.51 148.844))
     (stroke (width 0) (type default) (color 0 0 0 0))
@@
     (stroke (width 0) (type default) (color 0 0 0 0))
   )
+  (wire (pts (xy 160.02 132.08) (xy 148.59 132.08))
+    (stroke (width 0) (type default) (color 0 0 0 0))
+  )
   (wire (pts (xy 192.786 120.65) (xy 192.786 110.49))
     (stroke (width 0) (type default) (color 0 0 0 0))
@@
   )
   (text "A  B" (at 112.014 161.798 0)
+    (effects (font (size 1.27 1.27)) (justify left bottom))
+  )
+  (text "+5V\nSDA\nSCL\nGND" (at 167.64 137.16 0)
     (effects (font (size 1.27 1.27)) (justify left bottom))
   )
@@
     (pin "1")
     (pin "2")
+  )
+  (symbol (lib_id "power:+5V") (at 160.02 125.73 0) (unit 1)
+    (in_bom yes) (on_board yes) (fields_autoplaced)
+    (property "Reference" "#PWR?" (id 0) (at 160.02 129.54 0)
+      (effects (font (size 1.27 1.27)) hide)
+    )
+    (property "Value" "+5V" (id 1) (at 160.02 120.65 0))
+    (property "Footprint" "" (id 2) (at 160.02 125.73 0)
+      (effects (font (size 1.27 1.27)) hide)
+    )
+    (property "Datasheet" "" (id 3) (at 160.02 125.73 0)
+      (effects (font (size 1.27 1.27)) hide)
+    )
+    (pin "1")
   )
   (symbol (lib_id "power:GND") (at 225.806 145.034 0) (mirror y) (unit 1)
@@
     (pin "1")
   )
+  (symbol (lib_id "Connector_Generic:Conn_01x04") (at 165.1 132.08 0) (unit 1)
+    (in_bom yes) (on_board yes)
+    (property "Reference" "J?" (id 0) (at 163.83 140.97 0)
+      (effects (font (size 1.27 1.27)) (justify left))
+    )
+    (property "Value" "I2C bus" (id 1) (at 163.83 143.51 0)
+      (effects (font (size 1.27 1.27)) (justify left))
+    )
+    (property "Footprint" "" (id 2) (at 165.1 132.08 0)
+      (effects (font (size 1.27 1.27)) hide)
+    )
+    (property "Datasheet" "~" (id 3) (at 165.1 132.08 0)
+      (effects (font (size 1.27 1.27)) hide)
+    )
+    (pin "1")
+    (pin "2")
+    (pin "3")
+    (pin "4")
+  )
   (symbol (lib_id "power:GND") (at 100.076 112.014 270) (unit 1)
     (in_bom yes) (on_board yes)
@@
     )
     (property "Datasheet" "" (id 3) (at 99.568 70.104 0)
+      (effects (font (size 1.27 1.27)) hide)
+    )
+    (pin "1")
+  )
+  (symbol (lib_id "power:GND") (at 160.02 140.97 0) (unit 1)
+    (in_bom yes) (on_board yes)
+    (property "Reference" "#PWR?" (id 0) (at 160.02 147.32 0)
+      (effects (font (size 1.27 1.27)) hide)
+    )
+    (property "Value" "GND" (id 1) (at 160.02 144.78 0))
+    (property "Footprint" "" (id 2) (at 160.02 140.97 0)
+      (effects (font (size 1.27 1.27)) hide)
+    )
+    (property "Datasheet" "" (id 3) (at 160.02 140.97 0)
       (effects (font (size 1.27 1.27)) hide)
     )
@@
       (reference "#PWR031") (unit 1) (value "Earth_Protective") (footprint "")
     )
+    (path "/8caf16fb-af01-4af9-8180-9f4e321ea159"
+      (reference "#PWR?") (unit 1) (value "+5V") (footprint "")
+    )
+    (path "/dec670f6-d381-4c6c-9aa5-171066a3c21f"
+      (reference "#PWR?") (unit 1) (value "GND") (footprint "")
+    )
     (path "/c2a7c843-0a97-4b10-ae64-475349f900c5"
       (reference "C1") (unit 1) (value "33pF") (footprint "")
@@
       (reference "J6") (unit 1) (value "Conn_02x06_Odd_Even") (footprint "")
     )
+    (path "/d043d156-05f8-4a65-9ef1-581b1290125f"
+      (reference "J?") (unit 1) (value "I2C bus") (footprint "")
+    )
     (path "/84adba40-c7b9-4527-921b-cd0b4fd0fb40"
