File: KiCAD files/RCcar/RCcar.kicad_pcb (KiCad board)
At the start: 2 copper layers, 35 parts, among them J1 Power, J2 9V Battery, J3 Test, J4 L298N, J5 HC-05, J6 ICSP, J7 Comm, Q1 BC328, Q2 BC547, SW1 on/off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

Commit message: RCבשר
Parts:
- added R10: 100, Resistor_THT:R_Axial_DIN0207_L6.3mm_D2.5mm_P7.62mm_Horizontal, F.Cu at (139.3, 116.8)
- moved J2 0.51 mm to (167.1, 122.4)
- moved R8 0.30 mm to (153.7, 105.8)
Connections:
- U2 pad 3: Net-(BZ1-Pad1) -> Net-(U2-Pad3)
Routing:
- net Net-(BZ1-Pad1): track 26.3 -> 11.1 mm
- net Net-(U2-Pad3): track 0.00 -> 10.5 mm
- net /RX: track 98.2 -> 103.8 mm
- net +5V: track 209.4 -> 212.8 mm
- net GND: track 328.4 -> 325.5 mm
- net /TX: track 75.0 -> 77.7 mm
- net /RESET: track 50.3 -> 52.0 mm
- net Net-(J4-Pad2): track 33.1 -> 34.8 mm
- net Net-(J4-Pad5): track 35.9 -> 36.6 mm
