File: KiCAD files/RCcar/RCcar.kicad_sch (KiCad schematic)
At the start: 35 parts, among them J3 Test, J4 L298N, J5 HC-05, J6 ICSP, J7 Comm, Q2 BC547, U1 ATmega328-P, Y1 16MHz

Commit message: RCבשר
Parts:
- added R10: 100, Resistor_THT:R_Axial_DIN0207_L6.3mm_D2.5mm_P7.62mm_Horizontal, symbol Device:R_Small
- BZ1: footprint (none) -> Buzzer_Beeper:Buzzer_12x9.5RM7.6
- C1: footprint (none) -> Capacitor_THT:CP_Radial_D5.0mm_P2.50mm
- C2, C3, C4, C5, C6: footprint (none) -> Capacitor_THT:C_Disc_D3.0mm_W2.0mm_P2.50mm
- D1, D2: footprint (none) -> LED_THT:LED_D3.0mm_Clear
- H1, H2, H4: footprint (none) -> MountingHole:MountingHole_3mm
- H3: value (none) -> MountingHole; footprint (none) -> MountingHole:MountingHole_3mm
- J1: value (none) -> Power; footprint (none) -> Connector_PinHeader_2.54mm:PinHeader_1x03_P2.54mm_Vertical
- J2: value (none) -> 9V Battery; footprint (none) -> Connector_PinHeader_2.54mm:PinHeader_1x02_P2.54mm_Vertical
- J3: footprint (none) -> Connector_PinHeader_2.54mm:PinHeader_1x02_P2.54mm_Vertical
- J4: footprint (none) -> Connector_PinHeader_2.54mm:PinHeader_1x06_P2.54mm_Vertical
- J5: footprint (none) -> Connector_PinSocket_2.54mm:PinSocket_1x06_P2.54mm_Vertical
- J6: footprint (none) -> Connector_PinHeader_2.54mm:PinHeader_2x03_P2.54mm_Vertical
- J7: footprint (none) -> Connector_PinHeader_2.54mm:PinHeader_1x03_P2.54mm_Vertical
- Q1: value (none) -> BC328; footprint (none) -> Package_TO_SOT_THT:TO-92_Inline
- R1, R2, R3, R4, R5, R6, R7, R8, R9: footprint (none) -> Resistor_THT:R_Axial_DIN0207_L6.3mm_D2.5mm_P7.62mm_Horizontal
- SW1: value (none) -> on/off; footprint (none) -> Button_Switch_THT:SW_CW_GPTS203211B
- U1: footprint (none) -> Package_DIP:DIP-28_W7.62mm_Socket_LongPads
- U2: value (none) -> NE555P; footprint (none) -> Package_DIP:DIP-8_W7.62mm_Socket_LongPads
- Y1: footprint (none) -> Crystal:Crystal_HC49-4H_Vertical
Connections:
- net at U2.3 (Q): now also R10.1; no longer BZ1.1 (-)
- new net: BZ1.1 (-), R10.2
